File: kicad/projects/control_unit/control_unit.sch (KiCad schematic (older format))
At the start: 4 parts, among them U1 28C256, U2 28C256, U3 28C256, U4 28C256

Commit message: Start control unit - make board slightly larger to accomodate control unit and ALU needs.
Parts:
- added J1: Conn_01x08_Male, Connector_PinHeader_2.54mm:PinHeader_1x08_P2.54mm_Horizontal, symbol Connector:Conn_01x08_Male
- added J2: Conn_01x04_Female, Connector_PinSocket_2.54mm:PinSocket_1x04_P2.54mm_Horizontal, symbol Connector:Conn_01x04_Female
- added J3, J7: Conn_01x08_Female, Connector_PinSocket_2.54mm:PinSocket_1x08_P2.54mm_Horizontal, symbol Connector:Conn_01x08_Female
- added J4: Conn_01x34_Male, Connector_PinHeader_2.54mm:PinHeader_1x34_P2.54mm_Horizontal, symbol Connector:Conn_01x34_Male
- added J5, J6: Conn_01x16_Female, Connector_PinSocket_2.54mm:PinSocket_1x16_P2.54mm_Horizontal, symbol Connector:Conn_01x16_Female
- added RN1, RN2: R_Network08_US, Resistor_THT:R_Array_SIP9, symbol Device:R_Network08_US
- added RN3: R_Network04_US, Resistor_THT:R_Array_SIP5, symbol Device:R_Network04_US
- added U5: 74HCT377, Package_DIP:DIP-20_W7.62mm_Socket, symbol eight-bit-computer:74HCT377
- added U6: 74HCT161, Package_DIP:DIP-16_W7.62mm_Socket, symbol eight-bit-computer:74HCT161
- added U7: 74HCT173, Package_DIP:DIP-16_W7.62mm_Socket, symbol eight-bit-computer:74HCT173
- added U8: 74HCT138, Package_DIP:DIP-16_W7.62mm_Socket, symbol eight-bit-computer:74HCT138
- added U9: 74HCT04, Package_DIP:DIP-14_W7.62mm_Socket, symbol 74xx:74HCT04
Connections:
- net MIR_INST_7: now reaches U1.1 (A14)
- net MIR_INST_7: now also U2.1 (A14), U3.1 (A14), U4.1 (A14), U5.19 (Q7)
- net MC_STEP_0: now reaches U1.10 (A0)
- net MC_STEP_0: now also U2.10 (A0), U3.10 (A0), U4.10 (A0), U6.14 (Q0)
- net ROM_0_0: now reaches U1.11 (D0)
- net ROM_0_0: now also J4.1 (Pin_1)
- net ROM_0_1: now reaches U1.12 (D1)
- net ROM_0_1: now also J4.2 (Pin_2)
- net ROM_0_2: now reaches U1.13 (D2)
- net ROM_0_2: now also J4.3 (Pin_3)
- net ROM_0_3: now reaches U1.15 (D3)
- net ROM_0_3: now also J4.4 (Pin_4)
- net ROM_0_4: now reaches U1.16 (D4)
- net ROM_0_4: now also J4.5 (Pin_5)
- net ROM_0_5: now reaches U1.17 (D5)
- net ROM_0_5: now also J4.6 (Pin_6)
- net ROM_0_6: now reaches U1.18 (D6)
- net ROM_0_6: now also J4.7 (Pin_7)
- net ROM_0_7: now reaches U1.19 (D7)
- net ROM_0_7: now also J4.8 (Pin_8)
- net MIR_INST_5: now reaches U1.2 (A12)
- net MIR_INST_5: now also U2.2 (A12), U3.2 (A12), U4.2 (A12), U5.15 (Q5)
- net MIR_INST_3: now reaches U1.21 (A10)
- net MIR_INST_3: now also U2.21 (A10), U3.21 (A10), U4.21 (A10), U5.9 (Q3)
- net MIR_INST_4: now reaches U1.23 (A11)
- net MIR_INST_4: now also U2.23 (A11), U3.23 (A11), U4.23 (A11), U5.12 (Q4)
- net MIR_INST_2: now reaches U1.24 (A9)
- net MIR_INST_2: now also U2.24 (A9), U3.24 (A9), U4.24 (A9), U5.6 (Q2)
- net MIR_INST_1: now reaches U1.25 (A8)
- net MIR_INST_1: now also U2.25 (A8), U3.25 (A8), U4.25 (A8), U5.5 (Q1)
- net MIR_INST_6: now reaches U1.26 (A13)
- net MIR_INST_6: now also U2.26 (A13), U3.26 (A13), U4.26 (A13), U5.16 (Q6)
- net MIR_INST_0: now reaches U1.3 (A7)
- net MIR_INST_0: now also U2.3 (A7), U3.3 (A7), U4.3 (A7), U5.2 (Q0)
- net MIR_FLAG_E: now reaches U1.4 (A6)
- net MIR_FLAG_E: now also U2.4 (A6), U3.4 (A6), U4.4 (A6), U7.6 (Q3)
- net MIR_FLAG_C: now reaches U1.5 (A5)
- net MIR_FLAG_C: now also U2.5 (A5), U3.5 (A5), U4.5 (A5), U7.5 (Q2)
- net MIR_FLAG_N: now reaches U1.6 (A4)
- net MIR_FLAG_N: now also U2.6 (A4), U3.6 (A4), U4.6 (A4), U7.4 (Q1)
- net MIR_FLAG_Z: now reaches U1.7 (A3)
- net MIR_FLAG_Z: now also U2.7 (A3), U3.7 (A3), U4.7 (A3), U7.3 (Q0)
- net MC_STEP_2: now reaches U1.8 (A2)
- net MC_STEP_2: now also U2.8 (A2), U3.8 (A2), U4.8 (A2), U6.12 (Q2)
- net MC_STEP_1: now reaches U1.9 (A1)
- net MC_STEP_1: now also U2.9 (A1), U3.9 (A1), U4.9 (A1), U6.13 (Q1)
- net ROM_1_0: now reaches U2.11 (D0)
- net ROM_1_0: now also J4.9 (Pin_9)
- net ROM_1_1: now reaches U2.12 (D1)
- net ROM_1_1: now also J4.10 (Pin_10)
- net ROM_1_2: now reaches U2.13 (D2)
- net ROM_1_2: now also J4.11 (Pin_11)
- net ROM_1_3: now reaches U2.15 (D3)
- net ROM_1_3: now also J4.12 (Pin_12)
- net ROM_1_4: now reaches U2.16 (D4)
- net ROM_1_4: now also J4.13 (Pin_13)
- net ROM_1_5: now reaches U2.17 (D5)
- net ROM_1_5: now also J4.14 (Pin_14)
- net ROM_1_6: now reaches U2.18 (D6)
- net ROM_1_6: now also J4.15 (Pin_15)
- net ROM_1_7: now reaches U2.19 (D7)
- net ROM_1_7: now also J4.16 (Pin_16)
- net ROM_2_0: now reaches U3.11 (D0)
- net ROM_2_0: now also J4.17 (Pin_17)
- net ROM_2_1: now reaches U3.12 (D1)
- net ROM_2_1: now also J4.18 (Pin_18)
- net ROM_2_2: now reaches U3.13 (D2)
- net ROM_2_2: now also J4.19 (Pin_19)
- net ROM_2_3: now reaches U3.15 (D3)
- net ROM_2_3: now also J4.20 (Pin_20)
- net ROM_2_4: now reaches U3.16 (D4)
- net ROM_2_4: now also J4.21 (Pin_21)
- net ROM_2_5: now reaches U3.17 (D5)
- net ROM_2_5: now also J4.22 (Pin_22)
- net ROM_2_6: now reaches U3.18 (D6)
- net ROM_2_6: now also J4.23 (Pin_23)
- net ROM_2_7: now reaches U3.19 (D7)
- net ROM_2_7: now also J4.24 (Pin_24)
- net ROM_3_0: now reaches U4.11 (D0)
- net ROM_3_0: now also J4.25 (Pin_25)
- net ROM_3_1: now reaches U4.12 (D1)
- net ROM_3_1: now also J4.26 (Pin_26)
- net ROM_3_2: now reaches U4.13 (D2)
- net ROM_3_2: now also J4.27 (Pin_27)
- net ROM_3_3: now reaches U4.15 (D3)
- net ROM_3_3: now also J4.28 (Pin_28)
- net ROM_3_4: now reaches U4.16 (D4)
- net ROM_3_4: now also J4.29 (Pin_29)
- net ROM_3_5: now reaches U4.17 (D5)
- net ROM_3_5: now also J4.30 (Pin_30)
- net ROM_3_6: now reaches U4.18 (D6)
- net ROM_3_6: now also J4.31 (Pin_31)
- net ROM_3_7: now reaches U4.19 (D7)
- net ROM_3_7: now also J4.32 (Pin_32)
- no-connect marks 0 -> 2
Other:
- moved on the sheet: U1, U2, U3, U4

Commit message: More work on control unit schematic.
Parts:
- removed J1: Conn_01x08_Male, Connector_PinHeader_2.54mm:PinHeader_1x08_P2.54mm_Horizontal, symbol Connector:Conn_01x08_Male
- added J1: Conn_01x11_Male, Connector_PinHeader_2.54mm:PinHeader_1x11_P2.54mm_Horizontal, symbol Connector:Conn_01x11_Male
- added J8: Conn_01x01_Female, Connector_Wire:SolderWirePad_1x01_Drill0.8mm, symbol Connector:Conn_01x01_Female
- J4: footprint Connector_PinHeader_2.54mm:PinHeader_1x34_P2.54mm_Horizontal -> eight-bit-computer:backplane-connector
Connections:
- net MC_STEP_0: now also U8.1 (A)
- net MC_STEP_1: now also U8.2 (B)
- net MC_STEP_2: now also U8.3 (C)
- net MIR_FLAG_C: now also J7.5 (Pin_5)
- net MIR_FLAG_E: now also J7.7 (Pin_7)
- net MIR_FLAG_N: now also J7.3 (Pin_3)
- net MIR_FLAG_Z: now also J7.1 (Pin_1)
- net MIR_INST_0: now also J5.1 (Pin_1)
- net MIR_INST_1: now also J5.3 (Pin_3)
- net MIR_INST_2: now also J5.5 (Pin_5)
- net MIR_INST_3: now also J5.7 (Pin_7)
- net MIR_INST_4: now also J5.9 (Pin_9)
- net MIR_INST_5: now also J5.11 (Pin_11)
- net MIR_INST_6: now also J5.13 (Pin_13)
- net MIR_INST_7: now also J5.15 (Pin_15)
- net GND: now reaches U1.14 (GND)
- net GND: now also U2.14 (GND), U2.20 (~CS), U2.22 (~OE), U3.14 (GND), U3.20 (~CS), U3.22 (~OE), U4.14 (GND), U4.20 (~CS), U4.22 (~OE), U5.1 (~E), U5.10 (GND), U6.3 (P0), U6.4 (P1), U6.5 (P2), U6.6 (P3), U7.1 (~OE), U7.10 (~E2), U7.15 (MR), U7.2 (~OE2), U7.9 (~E1)
- net at J7.2 (Pin_2): now also RN3.2 (R1)
- net at J7.4 (Pin_4): now also RN3.3 (R2)
- net at J7.6 (Pin_6): now also RN3.4 (R3)
- net at J7.8 (Pin_8): now also RN3.5 (R4)
- net at J5.10 (Pin_10): now also RN1.6 (R5)
- net at J5.12 (Pin_12): now also RN1.7 (R6)
- net at J5.14 (Pin_14): now also RN1.8 (R7)
- net at J5.16 (Pin_16): now also RN1.9 (R8)
- net at J5.2 (Pin_2): now also RN1.2 (R1)
- net at J5.4 (Pin_4): now also RN1.3 (R2)
- net at J5.6 (Pin_6): now also RN1.4 (R3)
- net at J5.8 (Pin_8): now also RN1.5 (R4)
- net at J2.1 (Pin_1): now also U7.14 (D0)
- net at J2.2 (Pin_2): now also U7.13 (D1)
- net at J2.3 (Pin_3): now also U7.12 (D2)
- net at J2.4 (Pin_4): now also U7.11 (D3)
- net at J3.1 (Pin_1): now also U5.3 (D0)
- net at J3.2 (Pin_2): now also U5.4 (D1)
- net at J3.3 (Pin_3): now also U5.7 (D2)
- net at J3.4 (Pin_4): now also U5.8 (D3)
- net at J3.5 (Pin_5): now also U5.13 (D4)
- net at J3.6 (Pin_6): now also U5.14 (D5)
- net at J3.7 (Pin_7): now also U5.17 (D6)
- net at J3.8 (Pin_8): now also U5.18 (D7)
- net at J6.1 (Pin_1): now also U8.15 (Y0)
- net at J6.10 (Pin_10): now also RN2.6 (R5)
- net at J6.11 (Pin_11): now also U8.10 (Y5)
- net at J6.12 (Pin_12): now also RN2.7 (R6)
- net at J6.13 (Pin_13): now also U8.9 (Y6)
- net at J6.14 (Pin_14): now also RN2.8 (R7)
- net at J6.15 (Pin_15): now also U8.7 (Y7)
- net at J6.16 (Pin_16): now also RN2.9 (R8)
- net at J6.2 (Pin_2): now also RN2.2 (R1)
- net at J6.3 (Pin_3): now also U8.14 (Y1)
- net at J6.4 (Pin_4): now also RN2.3 (R2)
- net at J6.5 (Pin_5): now also U8.13 (Y2)
- net at J6.6 (Pin_6): now also RN2.4 (R3)
- net at J6.7 (Pin_7): now also U8.12 (Y3)
- net at J6.8 (Pin_8): now also RN2.5 (R4)
- net at J6.9 (Pin_9): now also U8.11 (Y4)
- net CONTROL_CLOCK: now reaches J4.34 (Pin_34)
- net CONTROL_CLOCK: now also U5.11 (CP), U6.2 (CP), U7.7 (CP)
- net MASTER_RESET: now reaches U9.1
- net MASTER_RESET: now also J1.11 (Pin_11)
- net at U9.2: now also U6.1 (~MR)
- net at U9.3: now also J8.1 (Pin_1)
- net at U9.4: now also U6.9 (~SPE)
- net VCC: now reaches U6.10 (TE)
- net VCC: now also U6.7 (PE)
- no-connect marks 2 -> 3
Other:
- moved on the sheet: J2, J3, J5, J6, J7, RN1, RN2, RN3, U1, U2, U3, U4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

Commit message: Start pcblayout on cu. Fix small path messiness on register.
Parts:
- added C1, C2, C3, C4, C5, C6, C7, C8, C9: 100nF, Capacitor_THT:C_Disc_D4.7mm_W2.5mm_P5.00mm, symbol Device:C
- J1: value Conn_01x11_Male -> BUS
- J2: value Conn_01x04_Female -> FLAGS
- J3: value Conn_01x08_Female -> INSTRUCTION
- J4: value Conn_01x34_Male -> BACKPLANE
- J5: value Conn_01x16_Female -> MIR INST LEDS
- J6: value Conn_01x16_Female -> STEP LEDS
- J7: value Conn_01x08_Female -> MIR FLAG LEDS
- J8: value Conn_01x01_Female -> STEP RESET
- RN1: value R_Network08_US -> MIR INST RESISTORS
- RN2: value R_Network08_US -> STEP RESISTORS
- RN3: value R_Network04_US -> MIR FLAG RESISTORS
Connections:
- net GND: now also J1.10 (Pin_10), RN1.1 (common), RN3.1 (common), U1.20 (~CS), U1.22 (~OE), U6.8 (GND), U7.8 (GND), U8.4 (~G2A), U8.5 (~G2B), U8.8 (GND), U9.11, U9.13, U9.5, U9.7 (GND), U9.9, C1.1, C2.2, C3.1, C4.2, C5.1, C6.2, C7.2, C8.2, C9.2
- net VCC: now also J1.9 (Pin_9), RN2.1 (common), U1.27 (~WE), U1.28 (VCC), U2.27 (~WE), U2.28 (VCC), U3.27 (~WE), U3.28 (VCC), U4.27 (~WE), U4.28 (VCC), U5.20 (VCC), U6.16 (VCC), U7.16 (VCC), U8.16 (VCC), U8.6 (G1), U9.14 (VCC), C1.2, C2.1, C3.2, C4.1, C5.2, C6.1, C7.1, C8.1, C9.1
- no-connect marks 3 -> 15
Other:
- moved on the sheet: J2, J3, J5, J7, RN3, U5, U7, U9C, U9D, U9E, U9F, U9G

Commit message: Tiny bit of work - mostly re-familiarising myself with KiCad.
Parts:
- added J9: MASTER RESET, Connector_PinSocket_2.54mm:PinSocket_1x01_P2.54mm_Horizontal, symbol Connector:Conn_01x01_Female
Connections:
- net MASTER_RESET: no longer U9.1
- new net: J9.1 (Pin_1), U9.1
Changed lines of the file:
@@
 Wire Wire Line
 	1450 7450 1450 7350
-Text Label 6100 900  2    50   ~ 0
+Text Label 6000 700  2    50   ~ 0
 MASTER_RESET
-Wire Wire Line
-	6100 900  6100 1000
 $Comp
 L Connector:Conn_01x01_Female J8
@@
 	3100 4300 2000 4300
 Connection ~ 2000 4300
+$Comp
+L Connector:Conn_01x01_Female J9
+U 1 1 5F14C107
+P 6100 800
+F 0 "J9" V 6000 1450 50  0000 R CNN
+F 1 "MASTER RESET" V 6100 1450 50  0000 R CNN
+F 2 "Connector_PinSocket_2.54mm:PinSocket_1x01_P2.54mm_Horizontal" H 6100 800 50  0001 C CNN
+F 3 "~" H 6100 800 50  0001 C CNN
+	1    6100 800
+	0    -1   -1   0
+$EndComp
 Wire Bus Line
 	5250 6900 5950 6900
