File: kicad/projects/cpu_status/cpu_status.sch (KiCad schematic (older format))
At the start: 95 parts, among them J1 Control_signal_backplane, J2 Aux_connection, J3 Bus_connection, J4 MAR_content_in, U1 74HCT245, U2 74HCT245, U3 74HCT245, U4 74HCT245, U5 74HCT245, U6 74HCT245, U7 74HCT245, U8 74HCT245

Commit message: Mostly schematic work on both boards.
Parts:
- added C12: 0.1uF, Capacitor_THT:C_Disc_D4.7mm_W2.5mm_P5.00mm, symbol Device:C
- added D65, D66, D67: LED, eight-bit-computer:eight-bit-computer-LED_D5.0mm, symbol Device:LED
- added R1, R2: 2K, Resistor_THT:R_Axial_DIN0207_L6.3mm_D2.5mm_P10.16mm_Horizontal, symbol Device:R_US
- added R3: 1.3K, Resistor_THT:R_Axial_DIN0207_L6.3mm_D2.5mm_P10.16mm_Horizontal, symbol Device:R_US
- added U9: 74HCT126, Package_DIP:DIP-14_W7.62mm, symbol eight-bit-computer:74HCT126
- D1, D10, D11, D12, D13, D14, D15, D16, D17, D18, D19, D2, D20, D21, D22, D23, D24, D25, D26, D27, D28, D29, D3, D30, D31, D32, D33, D34, D35, D36, D37, D38, D39, D4, D40, D41, D42, D43, D44, D45, D46, D47, D48, D49, D5, D50, D51, D52, D53, D54, D55, D56, D57, D58, D59, D6, D60, D61, D62, D63, D64, D7, D8, D9: footprint LED_THT:LED_D5.0mm -> eight-bit-computer:eight-bit-computer-LED_D5.0mm
Connections:
- net CTL_CLK: now also U9.5
- net DATA_CLK: now also U9.2
- net GND: now also C12.2, R1.1, R2.1, R3.1, U9.12, U9.13, U9.7 (GND)
- net RESET: now also U9.9
- net VCC: now also C12.1, U9.1, U9.10, U9.14 (VCC), U9.4
- new net: D65.1 (K), R1.2
- new net: D66.1 (K), R2.2
- new net: D67.1 (K), R3.2
- new net CTL_CLK_BUF: D66.2 (A), U9.6
- new net DATA_CLK_BUF: D65.2 (A), U9.3
- new net RESET_BUF: D67.2 (A), U9.8
- no-connect marks 0 -> 1
Other:
- note added: "Clock and reset display"
