File: kicad/projects/cpu_status/cpu_status.sch (KiCad schematic (older format))
At the start: 122 parts, among them J1 Control_signal_backplane, J2 Aux_connection, J3 Bus_connection, J4 MAR_content_in, J5 Conn_01x03_Male, J6 Conn_01x02_Female, J7 ECNZ, Q1 2N3904, U1 74HC245, U11 74HC245, U2 74HC245, U3 74HC245, U4 74HC245, U5 74HC245, U6 74HC245, U7 74HC245, U8 74HC245, U9 74HC126

Commit message: Gerbers generated and zipped. Changed ICs to sockets.
Parts:
- U1, U11, U2, U3, U4, U5, U6, U7, U8: footprint Package_DIP:DIP-20_W7.62mm -> Package_DIP:DIP-20_W7.62mm_Socket
- U9: footprint Package_DIP:DIP-14_W7.62mm -> Package_DIP:DIP-14_W7.62mm_Socket
Changed lines of the file:
@@
 F 0 "U3" H 3600 7550 50  0000 C CNN
 F 1 "74HC245" H 4050 7550 50  0000 C CNN
-F 2 "Package_DIP:DIP-20_W7.62mm" H 3450 6850 50  0001 C CNN
+F 2 "Package_DIP:DIP-20_W7.62mm_Socket" H 3450 6850 50  0001 C CNN
 F 3 "" H 3450 6850 50  0001 C CNN
 	1    3800 6850
@@
 F 0 "U1" H 1800 2900 50  0000 C CNN
 F 1 "74HC245" H 2250 2900 50  0000 C CNN
-F 2 "Package_DIP:DIP-20_W7.62mm" H 1650 2200 50  0001 C CNN
+F 2 "Package_DIP:DIP-20_W7.62mm_Socket" H 1650 2200 50  0001 C CNN
 F 3 "" H 1650 2200 50  0001 C CNN
 	1    2000 2200
@@
 F 0 "U5" H 6650 2850 50  0000 C CNN
 F 1 "74HC245" H 7100 2850 50  0000 C CNN
-F 2 "Package_DIP:DIP-20_W7.62mm" H 6500 2150 50  0001 C CNN
+F 2 "Package_DIP:DIP-20_W7.62mm_Socket" H 6500 2150 50  0001 C CNN
 F 3 "" H 6500 2150 50  0001 C CNN
 	1    6850 2150
@@
 F 0 "U2" H 1850 5000 50  0000 C CNN
 F 1 "74HC245" H 2300 5000 50  0000 C CNN
-F 2 "Package_DIP:DIP-20_W7.62mm" H 1700 4300 50  0001 C CNN
+F 2 "Package_DIP:DIP-20_W7.62mm_Socket" H 1700 4300 50  0001 C CNN
 F 3 "" H 1700 4300 50  0001 C CNN
 	1    2050 4300
@@
 F 0 "U4" H 3600 9600 50  0000 C CNN
 F 1 "74HC245" H 4050 9600 50  0000 C CNN
-F 2 "Package_DIP:DIP-20_W7.62mm" H 3450 8900 50  0001 C CNN
+F 2 "Package_DIP:DIP-20_W7.62mm_Socket" H 3450 8900 50  0001 C CNN
 F 3 "" H 3450 8900 50  0001 C CNN
 	1    3800 8900
@@
 F 0 "U6" H 6650 4800 50  0000 C CNN
 F 1 "74HC245" H 7100 4800 50  0000 C CNN
-F 2 "Package_DIP:DIP-20_W7.62mm" H 6500 4100 50  0001 C CNN
+F 2 "Package_DIP:DIP-20_W7.62mm_Socket" H 6500 4100 50  0001 C CNN
 F 3 "" H 6500 4100 50  0001 C CNN
 	1    6850 4100
@@
 F 0 "U7" H 6650 6750 50  0000 C CNN
 F 1 "74HC245" H 7100 6750 50  0000 C CNN
-F 2 "Package_DIP:DIP-20_W7.62mm" H 6500 6050 50  0001 C CNN
+F 2 "Package_DIP:DIP-20_W7.62mm_Socket" H 6500 6050 50  0001 C CNN
 F 3 "" H 6500 6050 50  0001 C CNN
 	1    6850 6050
@@
 F 0 "U8" H 6650 8700 50  0000 C CNN
 F 1 "74HC245" H 7100 8700 50  0000 C CNN
-F 2 "Package_DIP:DIP-20_W7.62mm" H 6500 8000 50  0001 C CNN
+F 2 "Package_DIP:DIP-20_W7.62mm_Socket" H 6500 8000 50  0001 C CNN
 F 3 "" H 6500 8000 50  0001 C CNN
 	1    6850 8000
@@
 F 0 "U11" H 12450 6450 50  0000 C CNN
 F 1 "74HC245" H 12900 6450 50  0000 C CNN
-F 2 "Package_DIP:DIP-20_W7.62mm" H 12300 5750 50  0001 C CNN
+F 2 "Package_DIP:DIP-20_W7.62mm_Socket" H 12300 5750 50  0001 C CNN
 F 3 "" H 12300 5750 50  0001 C CNN
 	1    12650 5750
@@
 F 0 "U9" H 13050 7400 50  0000 C CNN
 F 1 "74HC126" H 13450 7400 50  0000 C CNN
-F 2 "Package_DIP:DIP-14_W7.62mm" H 13300 7200 50  0001 C CNN
+F 2 "Package_DIP:DIP-14_W7.62mm_Socket" H 13300 7200 50  0001 C CNN
 F 3 "http://www.ti.com/lit/gpn/sn74HC126" H 13300 7200 50  0001 C CNN
 	1    13300 7200
@@
 F 0 "U9" H 13050 8050 50  0000 C CNN
 F 1 "74HC126" H 13450 8050 50  0000 C CNN
-F 2 "Package_DIP:DIP-14_W7.62mm" H 13300 7850 50  0001 C CNN
+F 2 "Package_DIP:DIP-14_W7.62mm_Socket" H 13300 7850 50  0001 C CNN
 F 3 "http://www.ti.com/lit/gpn/sn74HC126" H 13300 7850 50  0001 C CNN
 	2    13300 7850
@@
 F 0 "U9" H 13050 8650 50  0000 C CNN
 F 1 "74HC126" H 13400 8650 50  0000 C CNN
-F 2 "Package_DIP:DIP-14_W7.62mm" H 13300 8450 50  0001 C CNN
+F 2 "Package_DIP:DIP-14_W7.62mm_Socket" H 13300 8450 50  0001 C CNN
 F 3 "http://www.ti.com/lit/gpn/sn74HC126" H 13300 8450 50  0001 C CNN
 	3    13300 8450
@@
 F 0 "U9" H 10500 10067 50  0000 C CNN
 F 1 "74HC126" H 10500 9976 50  0000 C CNN
-F 2 "Package_DIP:DIP-14_W7.62mm" H 10500 9750 50  0001 C CNN
+F 2 "Package_DIP:DIP-14_W7.62mm_Socket" H 10500 9750 50  0001 C CNN
 F 3 "http://www.ti.com/lit/gpn/sn74HC126" H 10500 9750 50  0001 C CNN
 	4    10500 9750
@@
 F 0 "U9" H 11050 10150 50  0000 L CNN
 F 1 "74HC126" H 11400 10150 50  0000 L CNN
-F 2 "Package_DIP:DIP-14_W7.62mm" H 11350 9750 50  0001 C CNN
+F 2 "Package_DIP:DIP-14_W7.62mm_Socket" H 11350 9750 50  0001 C CNN
 F 3 "http://www.ti.com/lit/gpn/sn74HC126" H 11350 9750 50  0001 C CNN
 	5    11350 9750
