File: kicad/projects/alu_res_flags/alu_res_flags.sch (KiCad schematic (older format))
At the start: 57 parts, among them J1 RES_CRRYBRRW_EQ_IN, J2 Aux_connection, J3 Bus_connection, J4 Control_signal_backplane, J5 ECNZ_OUT, U1 74HCT04, U10 74HCT245, U11 74HCT173, U12 74HCT245, U2 74HCT377, U3 74HCT377, U4 74HCT245, U5 74HCT245, U6 74HCT27, U7 74HCT27, U8 74HCT30, U9 74HCT245

Commit message: Added more large caps, shrunk vias a bit
Parts:
- added C14, C15: 33uF, Capacitor_THT:CP_Radial_D6.3mm_P2.50mm, symbol Device:CP
- C13: value 330uF -> 33uF
Connections:
- net GND: now also C14.2, C15.2
- net VCC: now also C14.1, C15.1
Other:
- moved on the sheet: C13
Changed lines of the file:
@@
 L power:VCC #PWR0101
 U 1 1 5FBFC2EF
-P 2950 7150
-F 0 "#PWR0101" H 2950 7000 50  0001 C CNN
-F 1 "VCC" H 3050 7200 50  0000 C CNN
-F 2 "" H 2950 7150 50  0001 C CNN
-F 3 "" H 2950 7150 50  0001 C CNN
-	1    2950 7150
+P 18450 5900
+F 0 "#PWR0101" H 18450 5750 50  0001 C CNN
+F 1 "VCC" H 18550 5950 50  0000 C CNN
+F 2 "" H 18450 5900 50  0001 C CNN
+F 3 "" H 18450 5900 50  0001 C CNN
+	1    18450 5900
 	1    0    0    -1
 $EndComp
@@
 L power:GND #PWR0102
 U 1 1 5FBFCB14
-P 2950 7350
-F 0 "#PWR0102" H 2950 7100 50  0001 C CNN
-F 1 "GND" H 2800 7300 50  0000 C CNN
-F 2 "" H 2950 7350 50  0001 C CNN
-F 3 "" H 2950 7350 50  0001 C CNN
-	1    2950 7350
+P 18450 6100
+F 0 "#PWR0102" H 18450 5850 50  0001 C CNN
+F 1 "GND" H 18300 6050 50  0000 C CNN
+F 2 "" H 18450 6100 50  0001 C CNN
+F 3 "" H 18450 6100 50  0001 C CNN
+	1    18450 6100
 	-1   0    0    1
 $EndComp
@@
 L power:PWR_FLAG #FLG0101
 U 1 1 5FBFEF19
-P 3300 7150
-F 0 "#FLG0101" H 3300 7225 50  0001 C CNN
-F 1 "PWR_FLAG" H 3550 7200 50  0000 C CNN
-F 2 "" H 3300 7150 50  0001 C CNN
-F 3 "~" H 3300 7150 50  0001 C CNN
-	1    3300 7150
+P 18800 5900
+F 0 "#FLG0101" H 18800 5975 50  0001 C CNN
+F 1 "PWR_FLAG" H 19050 5950 50  0000 C CNN
+F 2 "" H 18800 5900 50  0001 C CNN
+F 3 "~" H 18800 5900 50  0001 C CNN
+	1    18800 5900
 	1    0    0    -1
 $EndComp
@@
 L power:PWR_FLAG #FLG0102
 U 1 1 5FBFF8F5
-P 3300 7350
-F 0 "#FLG0102" H 3300 7425 50  0001 C CNN
-F 1 "PWR_FLAG" H 3550 7400 50  0000 C CNN
-F 2 "" H 3300 7350 50  0001 C CNN
-F 3 "~" H 3300 7350 50  0001 C CNN
-	1    3300 7350
-	1    0    0    -1
-$EndComp
-Wire Wire Line
-	2650 7150 2950 7150
-Connection ~ 2650 7150
-Connection ~ 2950 7150
-Wire Wire Line
-	2950 7150 3200 7150
-Wire Wire Line
-	2650 7350 2950 7350
-Connection ~ 2650 7350
-Connection ~ 2950 7350
-Wire Wire Line
-	2950 7350 3300 7350
+P 18800 6100
+F 0 "#FLG0102" H 18800 6175 50  0001 C CNN
+F 1 "PWR_FLAG" H 19050 6150 50  0000 C CNN
+F 2 "" H 18800 6100 50  0001 C CNN
+F 3 "~" H 18800 6100 50  0001 C CNN
+	1    18800 6100
+	1    0    0    -1
+$EndComp
+Wire Wire Line
+	18150 5900 18450 5900
+Connection ~ 18450 5900
+Wire Wire Line
+	18450 5900 18700 5900
+Wire Wire Line
+	18150 6100 18450 6100
+Connection ~ 18450 6100
+Wire Wire Line
+	18450 6100 18800 6100
 Wire Wire Line
 	10800 3650 9550 3650
@@
 L Device:CP C13
 U 1 1 5FCF3BAB
-P 3950 7200
-F 0 "C13" H 4068 7246 50  0000 L CNN
-F 1 "330uF" H 4068 7155 50  0000 L CNN
-F 2 "Capacitor_THT:CP_Radial_D6.3mm_P2.50mm" H 3988 7050 50  0001 C CNN
-F 3 "~" H 3950 7200 50  0001 C CNN
-	1    3950 7200
-	1    0    0    -1
-$EndComp
-Wire Wire Line
-	3300 7350 3950 7350
-Connection ~ 3300 7350
-Wire Wire Line
-	3950 7050 3950 6900
-Wire Wire Line
-	3950 6900 3200 6900
-Wire Wire Line
-	3200 6900 3200 7150
-Connection ~ 3200 7150
-Wire Wire Line
-	3200 7150 3300 7150
+P 19450 5950
+F 0 "C13" H 19568 5996 50  0000 L CNN
+F 1 "33uF" H 19568 5905 50  0000 L CNN
+F 2 "Capacitor_THT:CP_Radial_D6.3mm_P2.50mm" H 19488 5800 50  0001 C CNN
+F 3 "~" H 19450 5950 50  0001 C CNN
+	1    19450 5950
+	1    0    0    -1
+$EndComp
+Wire Wire Line
+	18800 6100 19450 6100
+Connection ~ 18800 6100
+Wire Wire Line
+	19450 5800 19450 5650
+Wire Wire Line
+	19450 5650 18700 5650
+Wire Wire Line
+	18700 5650 18700 5900
+Connection ~ 18700 5900
+Wire Wire Line
+	18700 5900 18800 5900
+Text Label 18150 5900 2    50   ~ 0
+VCC
+Text Label 18150 6100 2    50   ~ 0
+GND
+$Comp
+L Device:CP C14
+U 1 1 5FCEADB2
+P 19950 5950
+F 0 "C14" H 20068 5996 50  0000 L CNN
+F 1 "33uF" H 20068 5905 50  0000 L CNN
+F 2 "Capacitor_THT:CP_Radial_D6.3mm_P2.50mm" H 19988 5800 50  0001 C CNN
+F 3 "~" H 19950 5950 50  0001 C CNN
+	1    19950 5950
+	1    0    0    -1
+$EndComp
+$Comp
+L Device:CP C15
+U 1 1 5FCEB59A
+P 20500 5950
+F 0 "C15" H 20618 5996 50  0000 L CNN
+F 1 "33uF" H 20618 5905 50  0000 L CNN
+F 2 "Capacitor_THT:CP_Radial_D6.3mm_P2.50mm" H 20538 5800 50  0001 C CNN
+F 3 "~" H 20500 5950 50  0001 C CNN
+	1    20500 5950
+	1    0    0    -1
+$EndComp
+Connection ~ 19450 5800
+Wire Wire Line
+	19450 5800 19950 5800
+Connection ~ 19950 5800
+Wire Wire Line
+	19950 5800 20500 5800
+Wire Wire Line
+	20500 6100 19950 6100
+Connection ~ 19450 6100
+Connection ~ 19950 6100
+Wire Wire Line
+	19950 6100 19450 6100
 $EndSCHEMATC

Commit message: Move kikad libs to sixteen bit location and update projects.
Parts:
- D1, D10, D11, D12, D13, D14, D15, D16, D17, D18, D19, D2, D20, D21, D22, D23, D24, D3, D4, D5, D6, D7, D8, D9: footprint eight-bit-computer:LED_D5.0mm_Horizontal_O3.81mm_Z3.0mm -> sixteen-bit-computer:LED_D5.0mm_Horizontal_O3.81mm_Z3.0mm
- J2: footprint eight-bit-computer:aux-connection -> sixteen-bit-computer:aux-connection; symbol eight-bit-computer:Aux_connection -> sixteen-bit-computer:Aux_connection
- J3: footprint eight-bit-computer:bus-connection -> sixteen-bit-computer:bus-connection; symbol eight-bit-computer:Bus_connection -> sixteen-bit-computer:Bus_connection
- J4: footprint eight-bit-computer:backplane-connector-single-row-annotated -> sixteen-bit-computer:backplane-connector-single-row-annotated; symbol eight-bit-computer:Control_signal_backplane -> sixteen-bit-computer:Control_signal_backplane
- U10, U12, U4, U5, U9: symbol eight-bit-computer:74HCT245 -> sixteen-bit-computer:74HCT245
- U11: symbol eight-bit-computer:74HCT173 -> sixteen-bit-computer:74HCT173
- U2, U3: symbol eight-bit-computer:74HCT377 -> sixteen-bit-computer:74HCT377
- U6, U7: symbol eight-bit-computer:74HCT27 -> sixteen-bit-computer:74HCT27
- U8: symbol eight-bit-computer:74HCT30 -> sixteen-bit-computer:74HCT30

Commit message: Switch to HC series chips and fix some labelling in program counter or register PCB.
Parts:
- U1: value 74HCT04 -> 74HC04; symbol 74xx:74HCT04 -> 74xx:74HC04
- U10, U12, U4, U5, U9: value 74HCT245 -> 74HC245; symbol sixteen-bit-computer:74HCT245 -> sixteen-bit-computer:74HC245
- U11: value 74HCT173 -> 74HC173; symbol sixteen-bit-computer:74HCT173 -> sixteen-bit-computer:74HC173
- U2, U3: value 74HCT377 -> 74HC377; symbol sixteen-bit-computer:74HCT377 -> sixteen-bit-computer:74HC377
- U6, U7: value 74HCT27 -> 74HC27; symbol sixteen-bit-computer:74HCT27 -> sixteen-bit-computer:74HC27
- U8: value 74HCT30 -> 74HC30; symbol sixteen-bit-computer:74HCT30 -> sixteen-bit-computer:74HC30
Changed lines of the file:
@@
 $EndDescr
 $Comp
-L sixteen-bit-computer:74HCT27 U6
+L sixteen-bit-computer:74HC27 U6
 U 1 1 5FB0B931
 P 7400 7250
 F 0 "U6" H 7700 7450 50  0000 C CNN
-F 1 "74HCT27" H 7400 7450 50  0000 C CNN
+F 1 "74HC27" H 7400 7450 50  0000 C CNN
 F 2 "Package_DIP:DIP-14_W7.62mm_Socket" H 7400 7250 50  0001 C CNN
 F 3 "https://www.ti.com/lit/ds/symlink/cd74hct27.pdf" H 7400 7250 50  0001 C CNN
@@
 $EndComp
 $Comp
-L sixteen-bit-computer:74HCT27 U6
+L sixteen-bit-computer:74HC27 U6
 U 2 1 5FB0CD47
 P 7400 7700
 F 0 "U6" H 7700 7900 50  0000 C CNN
-F 1 "74HCT27" H 7400 7900 50  0000 C CNN
+F 1 "74HC27" H 7400 7900 50  0000 C CNN
 F 2 "Package_DIP:DIP-14_W7.62mm_Socket" H 7400 7700 50  0001 C CNN
 F 3 "https://www.ti.com/lit/ds/symlink/cd74hct27.pdf" H 7400 7700 50  0001 C CNN
@@
 $EndComp
 $Comp
-L sixteen-bit-computer:74HCT27 U6
+L sixteen-bit-computer:74HC27 U6
 U 3 1 5FB0E763
 P 7400 8150
 F 0 "U6" H 7700 8350 50  0000 C CNN
-F 1 "74HCT27" H 7400 8350 50  0000 C CNN
+F 1 "74HC27" H 7400 8350 50  0000 C CNN
 F 2 "Package_DIP:DIP-14_W7.62mm_Socket" H 7400 8150 50  0001 C CNN
 F 3 "https://www.ti.com/lit/ds/symlink/cd74hct27.pdf" H 7400 8150 50  0001 C CNN
@@
 $EndComp
 $Comp
-L sixteen-bit-computer:74HCT27 U6
+L sixteen-bit-computer:74HC27 U6
 U 4 1 5FB1033F
 P 17550 3750
 F 0 "U6" H 17300 4100 50  0000 L CNN
-F 1 "74HCT27" H 17650 4100 50  0000 L CNN
+F 1 "74HC27" H 17650 4100 50  0000 L CNN
 F 2 "Package_DIP:DIP-14_W7.62mm_Socket" H 17550 3750 50  0001 C CNN
 F 3 "https://www.ti.com/lit/ds/symlink/cd74hct27.pdf" H 17550 3750 50  0001 C CNN
@@
 $EndComp
 $Comp
-L sixteen-bit-computer:74HCT27 U7
+L sixteen-bit-computer:74HC27 U7
 U 1 1 5FB13856
 P 7400 8850
 F 0 "U7" H 7700 9050 50  0000 C CNN
-F 1 "74HCT27" H 7400 9050 50  0000 C CNN
+F 1 "74HC27" H 7400 9050 50  0000 C CNN
 F 2 "Package_DIP:DIP-14_W7.62mm_Socket" H 7400 8850 50  0001 C CNN
 F 3 "https://www.ti.com/lit/ds/symlink/cd74hct27.pdf" H 7400 8850 50  0001 C CNN
@@
 $EndComp
 $Comp
-L sixteen-bit-computer:74HCT27 U7
+L sixteen-bit-computer:74HC27 U7
 U 2 1 5FB14A4F
 P 7400 9300
 F 0 "U7" H 7700 9500 50  0000 C CNN
-F 1 "74HCT27" H 7400 9500 50  0000 C CNN
+F 1 "74HC27" H 7400 9500 50  0000 C CNN
 F 2 "Package_DIP:DIP-14_W7.62mm_Socket" H 7400 9300 50  0001 C CNN
 F 3 "https://www.ti.com/lit/ds/symlink/cd74hct27.pdf" H 7400 9300 50  0001 C CNN
@@
 $EndComp
 $Comp
-L sixteen-bit-computer:74HCT27 U7
+L sixteen-bit-computer:74HC27 U7
 U 3 1 5FB1651F
 P 7400 9750
 F 0 "U7" H 7700 9950 50  0000 C CNN
-F 1 "74HCT27" H 7400 9950 50  0000 C CNN
+F 1 "74HC27" H 7400 9950 50  0000 C CNN
 F 2 "Package_DIP:DIP-14_W7.62mm_Socket" H 7400 9750 50  0001 C CNN
 F 3 "https://www.ti.com/lit/ds/symlink/cd74hct27.pdf" H 7400 9750 50  0001 C CNN
@@
 $EndComp
 $Comp
-L sixteen-bit-computer:74HCT27 U7
+L sixteen-bit-computer:74HC27 U7
 U 4 1 5FB17B44
 P 18700 3750
 F 0 "U7" H 18450 4100 50  0000 L CNN
-F 1 "74HCT27" H 18800 4100 50  0000 L CNN
+F 1 "74HC27" H 18800 4100 50  0000 L CNN
 F 2 "Package_DIP:DIP-14_W7.62mm_Socket" H 18700 3750 50  0001 C CNN
 F 3 "https://www.ti.com/lit/ds/symlink/cd74hct27.pdf" H 18700 3750 50  0001 C CNN
@@
 $EndComp
 $Comp
-L sixteen-bit-computer:74HCT377 U2
+L sixteen-bit-computer:74HC377 U2
 U 1 1 5FB1FEEC
 P 3250 5100
 F 0 "U2" H 3000 5750 50  0000 C CNN
-F 1 "74HCT377" H 3500 5750 50  0000 C CNN
+F 1 "74HC377" H 3500 5750 50  0000 C CNN
 F 2 "Package_DIP:DIP-20_W7.62mm_Socket" H 3250 5100 50  0001 C CNN
 F 3 "http://www.ti.com/lit/gpn/sn74LS377" H 3250 5100 50  0001 C CNN
@@
 $EndComp
 $Comp
-L sixteen-bit-computer:74HCT245 U10
+L sixteen-bit-computer:74HC245 U10
 U 1 1 5FB232A9
 P 10800 4900
 F 0 "U10" H 10600 5600 50  0000 C CNN
-F 1 "74HCT245" H 11050 5600 50  0000 C CNN
+F 1 "74HC245" H 11050 5600 50  0000 C CNN
 F 2 "Package_DIP:DIP-20_W7.62mm_Socket" H 10450 4900 50  0001 C CNN
 F 3 "" H 10450 4900 50  0001 C CNN
@@
 $EndComp
 $Comp
-L sixteen-bit-computer:74HCT245 U4
+L sixteen-bit-computer:74HC245 U4
 U 1 1 5FB23C97
 P 6800 2650
 F 0 "U4" H 6600 3350 50  0000 C CNN
-F 1 "74HCT245" H 7050 3350 50  0000 C CNN
+F 1 "74HC245" H 7050 3350 50  0000 C CNN
 F 2 "Package_DIP:DIP-20_W7.62mm_Socket" H 6450 2650 50  0001 C CNN
 F 3 "" H 6450 2650 50  0001 C CNN
@@
 $EndComp
 $Comp
-L sixteen-bit-computer:74HCT245 U5
+L sixteen-bit-computer:74HC245 U5
 U 1 1 5FB24682
 P 6800 4850
 F 0 "U5" H 6600 5550 50  0000 C CNN
-F 1 "74HCT245" H 7050 5550 50  0000 C CNN
+F 1 "74HC245" H 7050 5550 50  0000 C CNN
 F 2 "Package_DIP:DIP-20_W7.62mm_Socket" H 6450 4850 50  0001 C CNN
 F 3 "" H 6450 4850 50  0001 C CNN
@@
 $EndComp
 $Comp
-L sixteen-bit-computer:74HCT377 U3
+L sixteen-bit-computer:74HC377 U3
 U 1 1 5FB25053
 P 3300 2900
 F 0 "U3" H 3050 3550 50  0000 C CNN
-F 1 "74HCT377" H 3550 3550 50  0000 C CNN
+F 1 "74HC377" H 3550 3550 50  0000 C CNN
 F 2 "Package_DIP:DIP-20_W7.62mm_Socket" H 3300 2900 50  0001 C CNN
 F 3 "http://www.ti.com/lit/gpn/sn74LS377" H 3300 2900 50  0001 C CNN
@@
 $EndComp
 $Comp
-L sixteen-bit-computer:74HCT245 U12
+L sixteen-bit-computer:74HC245 U12
 U 1 1 5FB32788
 P 16500 8050
 F 0 "U12" H 16300 8750 50  0000 C CNN
-F 1 "74HCT245" H 16750 8750 50  0000 C CNN
+F 1 "74HC245" H 16750 8750 50  0000 C CNN
 F 2 "Package_DIP:DIP-20_W7.62mm_Socket" H 16150 8050 50  0001 C CNN
 F 3 "" H 16150 8050 50  0001 C CNN
@@
 $EndComp
 $Comp
-L sixteen-bit-computer:74HCT173 U11
+L sixteen-bit-computer:74HC173 U11
 U 1 1 5FB1DAED
 P 13800 8800
 F 0 "U11" H 13550 9550 50  0000 C CNN
-F 1 "74HCT173" H 14050 9550 50  0000 C CNN
+F 1 "74HC173" H 14050 9550 50  0000 C CNN
 F 2 "Package_DIP:DIP-16_W7.62mm_Socket" H 13800 8800 50  0001 C CNN
 F 3 "http://www.ti.com/lit/ds/symlink/cd74hc173.pdf" H 13800 8800 50  0001 C CNN
@@
 $EndComp
 $Comp
-L 74xx:74HCT04 U1
+L 74xx:74HC04 U1
 U 1 1 5FB8CBBD
 P 1750 3400
 F 0 "U1" H 1750 3717 50  0000 C CNN
-F 1 "74HCT04" H 1750 3626 50  0000 C CNN
+F 1 "74HC04" H 1750 3626 50  0000 C CNN
 F 2 "Package_DIP:DIP-14_W7.62mm_Socket" H 1750 3400 50  0001 C CNN
 F 3 "https://assets.nexperia.com/documents/data-sheet/74HC_HCT04.pdf" H 1750 3400 50  0001 C CNN
@@
 $EndComp
 $Comp
-L 74xx:74HCT04 U1
+L 74xx:74HC04 U1
 U 2 1 5FB8E6DD
 P 12150 9000
 F 0 "U1" H 12150 9317 50  0000 C CNN
-F 1 "74HCT04" H 12150 9226 50  0000 C CNN
+F 1 "74HC04" H 12150 9226 50  0000 C CNN
 F 2 "Package_DIP:DIP-14_W7.62mm_Socket" H 12150 9000 50  0001 C CNN
 F 3 "https://assets.nexperia.com/documents/data-sheet/74HC_HCT04.pdf" H 12150 9000 50  0001 C CNN
@@
 $EndComp
 $Comp
-L 74xx:74HCT04 U1
+L 74xx:74HC04 U1
 U 3 1 5FB8F91F
 P 9850 8450
 F 0 "U1" H 9850 8767 50  0000 C CNN
-F 1 "74HCT04" H 9850 8676 50  0000 C CNN
+F 1 "74HC04" H 9850 8676 50  0000 C CNN
 F 2 "Package_DIP:DIP-14_W7.62mm_Socket" H 9850 8450 50  0001 C CNN
 F 3 "https://assets.nexperia.com/documents/data-sheet/74HC_HCT04.pdf" H 9850 8450 50  0001 C CNN
@@
 $EndComp
 $Comp
-L 74xx:74HCT04 U1
+L 74xx:74HC04 U1
 U 4 1 5FB920C9
 P 5000 2100
 F 0 "U1" H 5000 2417 50  0000 C CNN
-F 1 "74HCT04" H 5000 2326 50  0000 C CNN
+F 1 "74HC04" H 5000 2326 50  0000 C CNN
 F 2 "Package_DIP:DIP-14_W7.62mm_Socket" H 5000 2100 50  0001 C CNN
 F 3 "https://assets.nexperia.com/documents/data-sheet/74HC_HCT04.pdf" H 5000 2100 50  0001 C CNN
@@
 $EndComp
 $Comp
-L 74xx:74HCT04 U1
+L 74xx:74HC04 U1
 U 5 1 5FB93894
 P 17550 4800
 F 0 "U1" H 17550 5117 50  0000 C CNN
-F 1 "74HCT04" H 17550 5026 50  0000 C CNN
+F 1 "74HC04" H 17550 5026 50  0000 C CNN
 F 2 "Package_DIP:DIP-14_W7.62mm_Socket" H 17550 4800 50  0001 C CNN
 F 3 "https://assets.nexperia.com/documents/data-sheet/74HC_HCT04.pdf" H 17550 4800 50  0001 C CNN
@@
 $EndComp
 $Comp
-L 74xx:74HCT04 U1
+L 74xx:74HC04 U1
 U 6 1 5FB95C2E
 P 18750 4800
 F 0 "U1" H 18750 5117 50  0000 C CNN
-F 1 "74HCT04" H 18750 5026 50  0000 C CNN
+F 1 "74HC04" H 18750 5026 50  0000 C CNN
 F 2 "Package_DIP:DIP-14_W7.62mm_Socket" H 18750 4800 50  0001 C CNN
 F 3 "https://assets.nexperia.com/documents/data-sheet/74HC_HCT04.pdf" H 18750 4800 50  0001 C CNN
@@
 $EndComp
 $Comp
-L 74xx:74HCT04 U1
+L 74xx:74HC04 U1
 U 7 1 5FB98A6E
 P 16300 3750
 F 0 "U1" H 16050 4100 50  0000 L CNN
-F 1 "74HCT04" H 16400 4100 50  0000 L CNN
+F 1 "74HC04" H 16400 4100 50  0000 L CNN
 F 2 "Package_DIP:DIP-14_W7.62mm_Socket" H 16300 3750 50  0001 C CNN
 F 3 "https://assets.nexperia.com/documents/data-sheet/74HC_HCT04.pdf" H 16300 3750 50  0001 C CNN
@@
 VCC
 $Comp
-L sixteen-bit-computer:74HCT245 U9
+L sixteen-bit-computer:74HC245 U9
 U 1 1 5FB211D5
 P 10800 2850
 F 0 "U9" H 10600 3550 50  0000 C CNN
-F 1 "74HCT245" H 11050 3550 50  0000 C CNN
+F 1 "74HC245" H 11050 3550 50  0000 C CNN
 F 2 "Package_DIP:DIP-20_W7.62mm_Socket" H 10450 2850 50  0001 C CNN
 F 3 "" H 10450 2850 50  0001 C CNN
@@
 RES_15
 $Comp
-L sixteen-bit-computer:74HCT30 U8
+L sixteen-bit-computer:74HC30 U8
 U 1 1 5FBBC8A7
 P 8800 8450
 F 0 "U8" H 9267 8975 50  0000 C CNN
-F 1 "74HCT30" H 9267 8884 50  0000 C CNN
+F 1 "74HC30" H 9267 8884 50  0000 C CNN
 F 2 "Package_DIP:DIP-14_W7.62mm_Socket" H 8800 8450 50  0001 C CNN
 F 3 "https://www.ti.com/lit/ds/symlink/cd74hct30.pdf" H 8800 8450 50  0001 C CNN
@@
 $EndComp
 $Comp
-L sixteen-bit-computer:74HCT30 U8
+L sixteen-bit-computer:74HC30 U8
 U 2 1 5FBBF1CA
 P 19750 3750
 F 0 "U8" H 19980 3796 50  0000 L CNN
-F 1 "74HCT30" H 19980 3705 50  0000 L CNN
+F 1 "74HC30" H 19980 3705 50  0000 L CNN
 F 2 "Package_DIP:DIP-14_W7.62mm_Socket" H 19750 3750 50  0001 C CNN
 F 3 "https://www.ti.com/lit/ds/symlink/cd74hct30.pdf" H 19750 3750 50  0001 C CNN
