File: kicad/projects/register16/register16.sch (KiCad schematic (older format))
At the start: 45 parts, among them J1 INPUT_ENABLE, J10 LOW, J2 OUTPUT_ENABLE, J3 CONTENTS, J4 Control_signal_backplane, J5 Aux_connection, J6 Bus_connection, J7 HIGH, J8 LOW, J9 HIGH, U1 74HCT04, U2 74HCT377, U3 74HCT377, U4 74HCT245, U5 74HCT245, U6 74HCT245, U7 74HCT245

Commit message: Move kikad libs to sixteen bit location and update projects.
Parts:
- D1, D10, D11, D12, D13, D14, D15, D16, D2, D3, D4, D5, D6, D7, D8, D9: footprint eight-bit-computer:LED_D5.0mm_Horizontal_O3.81mm_Z3.0mm -> sixteen-bit-computer:LED_D5.0mm_Horizontal_O3.81mm_Z3.0mm
- J4: footprint eight-bit-computer:backplane-connector-annotated -> sixteen-bit-computer:backplane-connector-annotated; symbol eight-bit-computer:Control_signal_backplane -> sixteen-bit-computer:Control_signal_backplane
- J5: footprint eight-bit-computer:aux-connection -> sixteen-bit-computer:aux-connection; symbol eight-bit-computer:Aux_connection -> sixteen-bit-computer:Aux_connection
- J6: footprint eight-bit-computer:bus-connection -> sixteen-bit-computer:bus-connection; symbol eight-bit-computer:Bus_connection -> sixteen-bit-computer:Bus_connection
- U2, U3: symbol eight-bit-computer:74HCT377 -> sixteen-bit-computer:74HCT377
- U4, U5, U6, U7: symbol eight-bit-computer:74HCT245 -> sixteen-bit-computer:74HCT245
Changed lines of the file:
@@
 $EndDescr
 $Comp
-L eight-bit-computer:Aux_connection J5
+L sixteen-bit-computer:Aux_connection J5
 U 1 1 5F84FDFB
 P 9900 4100
 F 0 "J5" H 9812 4725 50  0000 C CNN
 F 1 "Aux_connection" H 9812 4634 50  0000 C CNN
-F 2 "eight-bit-computer:aux-connection" H 9900 4100 50  0001 C CNN
+F 2 "sixteen-bit-computer:aux-connection" H 9900 4100 50  0001 C CNN
 F 3 "~" H 9900 4100 50  0001 C CNN
 	1    9900 4100
@@
 $EndComp
 $Comp
-L eight-bit-computer:Bus_connection J6
+L sixteen-bit-computer:Bus_connection J6
 U 1 1 5F851371
 P 9900 5700
 F 0 "J6" H 9762 6625 50  0000 C CNN
 F 1 "Bus_connection" H 9762 6534 50  0000 C CNN
-F 2 "eight-bit-computer:bus-connection" H 9800 6100 50  0001 C CNN
+F 2 "sixteen-bit-computer:bus-connection" H 9800 6100 50  0001 C CNN
 F 3 "~" H 9800 6100 50  0001 C CNN
 	1    9900 5700
@@
 $EndComp
 $Comp
-L eight-bit-computer:Control_signal_backplane J4
+L sixteen-bit-computer:Control_signal_backplane J4
 U 1 1 5F853275
 P 8850 4950
 F 0 "J4" H 8737 6675 50  0000 C CNN
 F 1 "Control_signal_backplane" H 8737 6584 50  0000 C CNN
-F 2 "eight-bit-computer:backplane-connector-annotated" H 8850 4950 50  0001 C CNN
+F 2 "sixteen-bit-computer:backplane-connector-annotated" H 8850 4950 50  0001 C CNN
 F 3 "~" H 8850 4950 50  0001 C CNN
 	1    8850 4950
@@
 $EndComp
 $Comp
-L eight-bit-computer:74HCT377 U3
+L sixteen-bit-computer:74HCT377 U3
 U 1 1 5F855C32
 P 1950 5950
@@
 $EndComp
 $Comp
-L eight-bit-computer:74HCT377 U2
+L sixteen-bit-computer:74HCT377 U2
 U 1 1 5F857635
 P 1950 4150
@@
 $EndComp
 $Comp
-L eight-bit-computer:74HCT245 U5
+L sixteen-bit-computer:74HCT245 U5
 U 1 1 5F858330
 P 4500 6250
@@
 $EndComp
 $Comp
-L eight-bit-computer:74HCT245 U6
+L sixteen-bit-computer:74HCT245 U6
 U 1 1 5F8AC977
 P 6850 1650
@@
 $EndComp
 $Comp
-L eight-bit-computer:74HCT245 U7
+L sixteen-bit-computer:74HCT245 U7
 U 1 1 5F8ADF71
 P 6850 3750
@@
 F 0 "D15" H 8500 2850 50  0000 C CNN
 F 1 "LED" H 8300 2850 50  0000 C CNN
-F 2 "eight-bit-computer:LED_D5.0mm_Horizontal_O3.81mm_Z3.0mm" H 8750 2900 50  0001 C CNN
+F 2 "sixteen-bit-computer:LED_D5.0mm_Horizontal_O3.81mm_Z3.0mm" H 8750 2900 50  0001 C CNN
 F 3 "~" H 8750 2900 50  0001 C CNN
 	1    8750 2900
@@
 F 0 "D16" H 8500 3000 50  0000 C CNN
 F 1 "LED" H 8300 3000 50  0000 C CNN
-F 2 "eight-bit-computer:LED_D5.0mm_Horizontal_O3.81mm_Z3.0mm" H 8750 3050 50  0001 C CNN
+F 2 "sixteen-bit-computer:LED_D5.0mm_Horizontal_O3.81mm_Z3.0mm" H 8750 3050 50  0001 C CNN
 F 3 "~" H 8750 3050 50  0001 C CNN
 	1    8750 3050
@@
 F 0 "D13" H 8500 2550 50  0000 C CNN
 F 1 "LED" H 8300 2550 50  0000 C CNN
-F 2 "eight-bit-computer:LED_D5.0mm_Horizontal_O3.81mm_Z3.0mm" H 8750 2600 50  0001 C CNN
+F 2 "sixteen-bit-computer:LED_D5.0mm_Horizontal_O3.81mm_Z3.0mm" H 8750 2600 50  0001 C CNN
 F 3 "~" H 8750 2600 50  0001 C CNN
 	1    8750 2600
@@
 F 0 "D14" H 8500 2700 50  0000 C CNN
 F 1 "LED" H 8300 2700 50  0000 C CNN
-F 2 "eight-bit-computer:LED_D5.0mm_Horizontal_O3.81mm_Z3.0mm" H 8750 2750 50  0001 C CNN
+F 2 "sixteen-bit-computer:LED_D5.0mm_Horizontal_O3.81mm_Z3.0mm" H 8750 2750 50  0001 C CNN
 F 3 "~" H 8750 2750 50  0001 C CNN
 	1    8750 2750
@@
 F 0 "D11" H 8500 2250 50  0000 C CNN
 F 1 "LED" H 8300 2250 50  0000 C CNN
-F 2 "eight-bit-computer:LED_D5.0mm_Horizontal_O3.81mm_Z3.0mm" H 8750 2300 50  0001 C CNN
+F 2 "sixteen-bit-computer:LED_D5.0mm_Horizontal_O3.81mm_Z3.0mm" H 8750 2300 50  0001 C CNN
 F 3 "~" H 8750 2300 50  0001 C CNN
 	1    8750 2300
@@
 F 0 "D12" H 8500 2400 50  0000 C CNN
 F 1 "LED" H 8300 2400 50  0000 C CNN
-F 2 "eight-bit-computer:LED_D5.0mm_Horizontal_O3.81mm_Z3.0mm" H 8750 2450 50  0001 C CNN
+F 2 "sixteen-bit-computer:LED_D5.0mm_Horizontal_O3.81mm_Z3.0mm" H 8750 2450 50  0001 C CNN
 F 3 "~" H 8750 2450 50  0001 C CNN
 	1    8750 2450
@@
 F 0 "D9" H 8500 1950 50  0000 C CNN
 F 1 "LED" H 8300 1950 50  0000 C CNN
-F 2 "eight-bit-computer:LED_D5.0mm_Horizontal_O3.81mm_Z3.0mm" H 8750 2000 50  0001 C CNN
+F 2 "sixteen-bit-computer:LED_D5.0mm_Horizontal_O3.81mm_Z3.0mm" H 8750 2000 50  0001 C CNN
 F 3 "~" H 8750 2000 50  0001 C CNN
 	1    8750 2000
@@
 F 0 "D10" H 8500 2100 50  0000 C CNN
 F 1 "LED" H 8300 2100 50  0000 C CNN
-F 2 "eight-bit-computer:LED_D5.0mm_Horizontal_O3.81mm_Z3.0mm" H 8750 2150 50  0001 C CNN
+F 2 "sixteen-bit-computer:LED_D5.0mm_Horizontal_O3.81mm_Z3.0mm" H 8750 2150 50  0001 C CNN
 F 3 "~" H 8750 2150 50  0001 C CNN
 	1    8750 2150
@@
 F 0 "D7" H 8500 1650 50  0000 C CNN
 F 1 "LED" H 8300 1650 50  0000 C CNN
-F 2 "eight-bit-computer:LED_D5.0mm_Horizontal_O3.81mm_Z3.0mm" H 8750 1700 50  0001 C CNN
+F 2 "sixteen-bit-computer:LED_D5.0mm_Horizontal_O3.81mm_Z3.0mm" H 8750 1700 50  0001 C CNN
 F 3 "~" H 8750 1700 50  0001 C CNN
 	1    8750 1700
@@
 F 0 "D8" H 8500 1800 50  0000 C CNN
 F 1 "LED" H 8300 1800 50  0000 C CNN
-F 2 "eight-bit-computer:LED_D5.0mm_Horizontal_O3.81mm_Z3.0mm" H 8750 1850 50  0001 C CNN
+F 2 "sixteen-bit-computer:LED_D5.0mm_Horizontal_O3.81mm_Z3.0mm" H 8750 1850 50  0001 C CNN
 F 3 "~" H 8750 1850 50  0001 C CNN
 	1    8750 1850
@@
 F 0 "D5" H 8500 1350 50  0000 C CNN
 F 1 "LED" H 8300 1350 50  0000 C CNN
-F 2 "eight-bit-computer:LED_D5.0mm_Horizontal_O3.81mm_Z3.0mm" H 8750 1400 50  0001 C CNN
+F 2 "sixteen-bit-computer:LED_D5.0mm_Horizontal_O3.81mm_Z3.0mm" H 8750 1400 50  0001 C CNN
 F 3 "~" H 8750 1400 50  0001 C CNN
 	1    8750 1400
@@
 F 0 "D6" H 8500 1500 50  0000 C CNN
 F 1 "LED" H 8300 1500 50  0000 C CNN
-F 2 "eight-bit-computer:LED_D5.0mm_Horizontal_O3.81mm_Z3.0mm" H 8750 1550 50  0001 C CNN
+F 2 "sixteen-bit-computer:LED_D5.0mm_Horizontal_O3.81mm_Z3.0mm" H 8750 1550 50  0001 C CNN
 F 3 "~" H 8750 1550 50  0001 C CNN
 	1    8750 1550
@@
 F 0 "D3" H 8500 1050 50  0000 C CNN
 F 1 "LED" H 8300 1050 50  0000 C CNN
-F 2 "eight-bit-computer:LED_D5.0mm_Horizontal_O3.81mm_Z3.0mm" H 8750 1100 50  0001 C CNN
+F 2 "sixteen-bit-computer:LED_D5.0mm_Horizontal_O3.81mm_Z3.0mm" H 8750 1100 50  0001 C CNN
 F 3 "~" H 8750 1100 50  0001 C CNN
 	1    8750 1100
@@
 F 0 "D4" H 8500 1200 50  0000 C CNN
 F 1 "LED" H 8300 1200 50  0000 C CNN
-F 2 "eight-bit-computer:LED_D5.0mm_Horizontal_O3.81mm_Z3.0mm" H 8750 1250 50  0001 C CNN
+F 2 "sixteen-bit-computer:LED_D5.0mm_Horizontal_O3.81mm_Z3.0mm" H 8750 1250 50  0001 C CNN
 F 3 "~" H 8750 1250 50  0001 C CNN
 	1    8750 1250
@@
 F 0 "D1" H 8500 750 50  0000 C CNN
 F 1 "LED" H 8300 750 50  0000 C CNN
-F 2 "eight-bit-computer:LED_D5.0mm_Horizontal_O3.81mm_Z3.0mm" H 8750 800 50  0001 C CNN
+F 2 "sixteen-bit-computer:LED_D5.0mm_Horizontal_O3.81mm_Z3.0mm" H 8750 800 50  0001 C CNN
 F 3 "~" H 8750 800 50  0001 C CNN
 	1    8750 800
@@
 F 0 "D2" H 8500 900 50  0000 C CNN
 F 1 "LED" H 8300 900 50  0000 C CNN
-F 2 "eight-bit-computer:LED_D5.0mm_Horizontal_O3.81mm_Z3.0mm" H 8750 950 50  0001 C CNN
+F 2 "sixteen-bit-computer:LED_D5.0mm_Horizontal_O3.81mm_Z3.0mm" H 8750 950 50  0001 C CNN
 F 3 "~" H 8750 950 50  0001 C CNN
 	1    8750 950
@@
 $EndComp
 $Comp
-L eight-bit-computer:74HCT245 U4
+L sixteen-bit-computer:74HCT245 U4
 U 1 1 5F854F6D
 P 4500 4150

Commit message: Switch to HC series chips and fix some labelling in program counter or register PCB.
Parts:
- U1: value 74HCT04 -> 74HC04; symbol 74xx:74HCT04 -> 74xx:74HC04
- U2, U3: value 74HCT377 -> 74HC377; symbol sixteen-bit-computer:74HCT377 -> sixteen-bit-computer:74HC377
- U4, U5, U6, U7: value 74HCT245 -> 74HC245; symbol sixteen-bit-computer:74HCT245 -> sixteen-bit-computer:74HC245
Changed lines of the file:
@@
 $EndComp
 $Comp
-L sixteen-bit-computer:74HCT377 U3
+L sixteen-bit-computer:74HC377 U3
 U 1 1 5F855C32
 P 1950 5950
 F 0 "U3" H 2350 5550 50  0000 C CNN
-F 1 "74HCT377" H 2500 5450 50  0000 C CNN
+F 1 "74HC377" H 2500 5450 50  0000 C CNN
 F 2 "Package_DIP:DIP-20_W7.62mm_Socket" H 1950 5950 50  0001 C CNN
 F 3 "http://www.ti.com/lit/gpn/sn74LS377" H 1950 5950 50  0001 C CNN
@@
 $EndComp
 $Comp
-L sixteen-bit-computer:74HCT377 U2
+L sixteen-bit-computer:74HC377 U2
 U 1 1 5F857635
 P 1950 4150
 F 0 "U2" H 2350 3750 50  0000 C CNN
-F 1 "74HCT377" H 2500 3650 50  0000 C CNN
+F 1 "74HC377" H 2500 3650 50  0000 C CNN
 F 2 "Package_DIP:DIP-20_W7.62mm_Socket" H 1950 4150 50  0001 C CNN
 F 3 "http://www.ti.com/lit/gpn/sn74LS377" H 1950 4150 50  0001 C CNN
@@
 $EndComp
 $Comp
-L sixteen-bit-computer:74HCT245 U5
+L sixteen-bit-computer:74HC245 U5
 U 1 1 5F858330
 P 4500 6250
 F 0 "U5" H 4850 6800 50  0000 C CNN
-F 1 "74HCT245" H 5000 6700 50  0000 C CNN
+F 1 "74HC245" H 5000 6700 50  0000 C CNN
 F 2 "Package_DIP:DIP-20_W7.62mm_Socket" H 4150 6250 50  0001 C CNN
 F 3 "" H 4150 6250 50  0001 C CNN
@@
 $EndComp
 $Comp
-L 74xx:74HCT04 U1
+L 74xx:74HC04 U1
 U 1 1 5F89775D
 P 900 4350
 F 0 "U1" H 900 4050 50  0000 C CNN
-F 1 "74HCT04" H 900 4150 50  0000 C CNN
+F 1 "74HC04" H 900 4150 50  0000 C CNN
 F 2 "Package_DIP:DIP-14_W7.62mm_Socket" H 900 4350 50  0001 C CNN
 F 3 "https://assets.nexperia.com/documents/data-sheet/74HC_HCT04.pdf" H 900 4350 50  0001 C CNN
@@
 $EndComp
 $Comp
-L 74xx:74HCT04 U1
+L 74xx:74HC04 U1
 U 2 1 5F898EF8
 P 3600 3300
 F 0 "U1" H 3600 3000 50  0000 C CNN
-F 1 "74HCT04" H 3600 3100 50  0000 C CNN
+F 1 "74HC04" H 3600 3100 50  0000 C CNN
 F 2 "Package_DIP:DIP-14_W7.62mm_Socket" H 3600 3300 50  0001 C CNN
 F 3 "https://assets.nexperia.com/documents/data-sheet/74HC_HCT04.pdf" H 3600 3300 50  0001 C CNN
@@
 $EndComp
 $Comp
-L 74xx:74HCT04 U1
+L 74xx:74HC04 U1
 U 3 1 5F899C5B
 P 2150 950
 F 0 "U1" H 2150 1267 50  0000 C CNN
-F 1 "74HCT04" H 2150 1176 50  0000 C CNN
+F 1 "74HC04" H 2150 1176 50  0000 C CNN
 F 2 "Package_DIP:DIP-14_W7.62mm_Socket" H 2150 950 50  0001 C CNN
 F 3 "https://assets.nexperia.com/documents/data-sheet/74HC_HCT04.pdf" H 2150 950 50  0001 C CNN
@@
 $EndComp
 $Comp
-L 74xx:74HCT04 U1
+L 74xx:74HC04 U1
 U 4 1 5F89C4C9
 P 2150 1450
 F 0 "U1" H 2150 1767 50  0000 C CNN
-F 1 "74HCT04" H 2150 1676 50  0000 C CNN
+F 1 "74HC04" H 2150 1676 50  0000 C CNN
 F 2 "Package_DIP:DIP-14_W7.62mm_Socket" H 2150 1450 50  0001 C CNN
 F 3 "https://assets.nexperia.com/documents/data-sheet/74HC_HCT04.pdf" H 2150 1450 50  0001 C CNN
@@
 $EndComp
 $Comp
-L 74xx:74HCT04 U1
+L 74xx:74HC04 U1
 U 5 1 5F89DBF3
 P 3000 950
 F 0 "U1" H 3000 1267 50  0000 C CNN
-F 1 "74HCT04" H 3000 1176 50  0000 C CNN
+F 1 "74HC04" H 3000 1176 50  0000 C CNN
 F 2 "Package_DIP:DIP-14_W7.62mm_Socket" H 3000 950 50  0001 C CNN
 F 3 "https://assets.nexperia.com/documents/data-sheet/74HC_HCT04.pdf" H 3000 950 50  0001 C CNN
@@
 $EndComp
 $Comp
-L 74xx:74HCT04 U1
+L 74xx:74HC04 U1
 U 6 1 5F89F049
 P 3000 1450
 F 0 "U1" H 3000 1767 50  0000 C CNN
-F 1 "74HCT04" H 3000 1676 50  0000 C CNN
+F 1 "74HC04" H 3000 1676 50  0000 C CNN
 F 2 "Package_DIP:DIP-14_W7.62mm_Socket" H 3000 1450 50  0001 C CNN
 F 3 "https://assets.nexperia.com/documents/data-sheet/74HC_HCT04.pdf" H 3000 1450 50  0001 C CNN
@@
 $EndComp
 $Comp
-L 74xx:74HCT04 U1
+L 74xx:74HC04 U1
 U 7 1 5F8A0462
 P 1100 1150
 F 0 "U1" H 1330 1196 50  0000 L CNN
-F 1 "74HCT04" H 1330 1105 50  0000 L CNN
+F 1 "74HC04" H 1330 1105 50  0000 L CNN
 F 2 "Package_DIP:DIP-14_W7.62mm_Socket" H 1100 1150 50  0001 C CNN
 F 3 "https://assets.nexperia.com/documents/data-sheet/74HC_HCT04.pdf" H 1100 1150 50  0001 C CNN
@@
 $EndComp
 $Comp
-L sixteen-bit-computer:74HCT245 U6
+L sixteen-bit-computer:74HC245 U6
 U 1 1 5F8AC977
 P 6850 1650
 F 0 "U6" H 7200 2250 50  0000 C CNN
-F 1 "74HCT245" H 7350 2100 50  0000 C CNN
+F 1 "74HC245" H 7350 2100 50  0000 C CNN
 F 2 "Package_DIP:DIP-20_W7.62mm_Socket" H 6500 1650 50  0001 C CNN
 F 3 "" H 6500 1650 50  0001 C CNN
@@
 $EndComp
 $Comp
-L sixteen-bit-computer:74HCT245 U7
+L sixteen-bit-computer:74HC245 U7
 U 1 1 5F8ADF71
 P 6850 3750
 F 0 "U7" H 7200 4350 50  0000 C CNN
-F 1 "74HCT245" H 7350 4200 50  0000 C CNN
+F 1 "74HC245" H 7350 4200 50  0000 C CNN
 F 2 "Package_DIP:DIP-20_W7.62mm_Socket" H 6500 3750 50  0001 C CNN
 F 3 "" H 6500 3750 50  0001 C CNN
@@
 $EndComp
 $Comp
-L sixteen-bit-computer:74HCT245 U4
+L sixteen-bit-computer:74HC245 U4
 U 1 1 5F854F6D
 P 4500 4150
 F 0 "U4" H 4850 4700 50  0000 C CNN
-F 1 "74HCT245" H 5000 4600 50  0000 C CNN
+F 1 "74HC245" H 5000 4600 50  0000 C CNN
 F 2 "Package_DIP:DIP-20_W7.62mm_Socket" H 4150 4150 50  0001 C CNN
 F 3 "" H 4150 4150 50  0001 C CNN
