File: kicad/projects/control_unit_16/control_unit_16.sch (KiCad schematic (older format))
At the start: 54 parts, among them J1 Conn_01x04_Female, J2 Control_signal_backplane, J3 Bus_connection, J4 Aux_connection, J5 Conn_01x16_Female, U1 74HCT04, U10 28C256, U11 28C256, U2 28C256, U3 74HCT173, U4 74HCT377, U5 74HCT161, U6 28C256, U7 74HCT245, U8 74HCT245, U9 74HCT138

Commit message: About half way through control unit PCB layout.
Changed lines of the file:
@@
 $EndDescr
-$Comp
-L eight-bit-computer:74HCT377 U4
-U 1 1 5FD843AB
-P 2600 4000
-F 0 "U4" H 2350 4650 50  0000 C CNN
-F 1 "74HCT377" H 2850 4650 50  0000 C CNN
-F 2 "Package_DIP:DIP-20_W7.62mm" H 2600 4000 50  0001 C CNN
-F 3 "http://www.ti.com/lit/gpn/sn74LS377" H 2600 4000 50  0001 C CNN
-	1    2600 4000
-	1    0    0    -1
-$EndComp
 $Comp
 L eight-bit-computer:74HCT161 U5
@@
 NoConn ~ 11350 3050
 NoConn ~ 11250 3050
-Text Label 2100 3500 2    50   ~ 0
-INST_00
-Text Label 2100 3600 2    50   ~ 0
-INST_01
-Text Label 2100 3700 2    50   ~ 0
-INST_02
-Text Label 2100 3800 2    50   ~ 0
-INST_03
-Text Label 2100 3900 2    50   ~ 0
-INST_04
-Text Label 2100 4000 2    50   ~ 0
-INST_05
-Text Label 2100 4100 2    50   ~ 0
-INST_06
-Text Label 2100 4200 2    50   ~ 0
-INST_07
-Text Label 3100 3500 0    50   ~ 0
-MIR_INST_0
-Text Label 3100 3600 0    50   ~ 0
-MIR_INST_1
-Text Label 3100 3700 0    50   ~ 0
-MIR_INST_2
-Text Label 3100 3800 0    50   ~ 0
-MIR_INST_3
-Text Label 3100 3900 0    50   ~ 0
-MIR_INST_4
-Text Label 3100 4000 0    50   ~ 0
-MIR_INST_5
-Text Label 3100 4100 0    50   ~ 0
-MIR_INST_6
-Text Label 3100 4200 0    50   ~ 0
-MIR_INST_7
 Text Label 2850 650  0    50   ~ 0
 VCC
@@
 Text Label 5750 1800 0    50   ~ 0
 LIN_STEP_7
-Text Label 1500 4400 2    50   ~ 0
-CONTROL_CLOCK
-$Comp
-L Device:C C2
-U 1 1 5FECB829
-P 1650 3350
-F 0 "C2" H 1450 3400 50  0000 L CNN
-F 1 "0.1uF" H 1350 3300 50  0000 L CNN
-F 2 "Capacitor_THT:C_Disc_D4.7mm_W2.5mm_P5.00mm" H 1688 3200 50  0001 C CNN
-F 3 "~" H 1650 3350 50  0001 C CNN
-	1    1650 3350
-	1    0    0    -1
-$EndComp
-Wire Wire Line
-	1650 3200 2600 3200
-Wire Wire Line
-	1650 3500 1650 4500
-Wire Wire Line
-	1650 4800 2600 4800
-Wire Wire Line
-	2100 4500 1650 4500
-Connection ~ 1650 4500
-Wire Wire Line
-	1650 4500 1650 4800
-Wire Wire Line
-	1500 4400 2100 4400
 $Comp
 L eight-bit-computer:74HCT245 U8
@@
 Text Label 6900 3500 0    50   ~ 0
 GND
-Wire Wire Line
-	3100 3500 4050 3500
-Wire Wire Line
-	4050 3600 3100 3600
-Wire Wire Line
-	3100 3700 4050 3700
-Wire Wire Line
-	4050 3800 3100 3800
-Wire Wire Line
-	3100 3900 4050 3900
-Wire Wire Line
-	4050 4000 3100 4000
-Wire Wire Line
-	3100 4100 4050 4100
-Wire Wire Line
-	4050 4200 3100 4200
 $Comp
 L Device:LED D1
@@
 Wire Wire Line
 	1800 6750 1800 7050
-Text Label 2300 3200 0    50   ~ 0
-VCC
-Text Label 2350 4800 0    50   ~ 0
-GND
 Text Label 4350 2800 0    50   ~ 0
 VCC
@@
 Text Label 6450 6700 0    50   ~ 0
 GND
+Text Label 2350 4800 0    50   ~ 0
+GND
+Text Label 2300 3200 0    50   ~ 0
+VCC
+Wire Wire Line
+	4050 3500 3100 3500
+Wire Wire Line
+	3100 3600 4050 3600
+Wire Wire Line
+	4050 3700 3100 3700
+Wire Wire Line
+	3100 3800 4050 3800
+Wire Wire Line
+	4050 3900 3100 3900
+Wire Wire Line
+	3100 4000 4050 4000
+Wire Wire Line
+	4050 4100 3100 4100
+Wire Wire Line
+	3100 4200 4050 4200
+Wire Wire Line
+	1500 4400 2100 4400
+Wire Wire Line
+	1650 4500 1650 4800
+Connection ~ 1650 4500
+Wire Wire Line
+	2100 4500 1650 4500
+Wire Wire Line
+	1650 4800 2600 4800
+Wire Wire Line
+	1650 3500 1650 4500
+Wire Wire Line
+	1650 3200 2600 3200
+$Comp
+L Device:C C2
+U 1 1 5FECB829
+P 1650 3350
+F 0 "C2" H 1450 3400 50  0000 L CNN
+F 1 "0.1uF" H 1350 3300 50  0000 L CNN
+F 2 "Capacitor_THT:C_Disc_D4.7mm_W2.5mm_P5.00mm" H 1688 3200 50  0001 C CNN
+F 3 "~" H 1650 3350 50  0001 C CNN
+	1    1650 3350
+	1    0    0    -1
+$EndComp
+Text Label 1500 4400 2    50   ~ 0
+CONTROL_CLOCK
+Text Label 3100 3500 0    50   ~ 0
+MIR_INST_7
+Text Label 3100 3600 0    50   ~ 0
+MIR_INST_6
+Text Label 3100 3700 0    50   ~ 0
+MIR_INST_5
+Text Label 3100 3800 0    50   ~ 0
+MIR_INST_4
+Text Label 3100 3900 0    50   ~ 0
+MIR_INST_3
+Text Label 3100 4000 0    50   ~ 0
+MIR_INST_2
+Text Label 3100 4100 0    50   ~ 0
+MIR_INST_1
+Text Label 3100 4200 0    50   ~ 0
+MIR_INST_0
+Text Label 2100 3500 2    50   ~ 0
+INST_07
+Text Label 2100 3600 2    50   ~ 0
+INST_06
+Text Label 2100 3700 2    50   ~ 0
+INST_05
+Text Label 2100 3800 2    50   ~ 0
+INST_04
+Text Label 2100 3900 2    50   ~ 0
+INST_03
+Text Label 2100 4000 2    50   ~ 0
+INST_02
+Text Label 2100 4100 2    50   ~ 0
+INST_01
+Text Label 2100 4200 2    50   ~ 0
+INST_00
+$Comp
+L eight-bit-computer:74HCT377 U4
+U 1 1 5FD843AB
+P 2600 4000
+F 0 "U4" H 2350 4650 50  0000 C CNN
+F 1 "74HCT377" H 2850 4650 50  0000 C CNN
+F 2 "Package_DIP:DIP-20_W7.62mm" H 2600 4000 50  0001 C CNN
+F 3 "http://www.ti.com/lit/gpn/sn74LS377" H 2600 4000 50  0001 C CNN
+	1    2600 4000
+	1    0    0    -1
+$EndComp
 $EndSCHEMATC

Commit message: Move kikad libs to sixteen bit location and update projects.
Parts:
- D1, D10, D11, D12, D13, D14, D15, D16, D17, D18, D19, D2, D20, D3, D4, D5, D6, D7, D8, D9: footprint eight-bit-computer:LED_D5.0mm_Horizontal_O3.81mm_Z3.0mm -> sixteen-bit-computer:LED_D5.0mm_Horizontal_O3.81mm_Z3.0mm
- J2: footprint eight-bit-computer:backplane-connector-single-row -> sixteen-bit-computer:backplane-connector-single-row; symbol eight-bit-computer:Control_signal_backplane -> sixteen-bit-computer:Control_signal_backplane
- J3: footprint eight-bit-computer:bus-connection -> sixteen-bit-computer:bus-connection; symbol eight-bit-computer:Bus_connection -> sixteen-bit-computer:Bus_connection
- J4: footprint eight-bit-computer:aux-connection -> sixteen-bit-computer:aux-connection; symbol eight-bit-computer:Aux_connection -> sixteen-bit-computer:Aux_connection
- U3: symbol eight-bit-computer:74HCT173 -> sixteen-bit-computer:74HCT173
- U4: symbol eight-bit-computer:74HCT377 -> sixteen-bit-computer:74HCT377
- U5: symbol eight-bit-computer:74HCT161 -> sixteen-bit-computer:74HCT161
- U7, U8: symbol eight-bit-computer:74HCT245 -> sixteen-bit-computer:74HCT245
- U9: symbol eight-bit-computer:74HCT138 -> sixteen-bit-computer:74HCT138
Changed lines of the file:
@@
 $EndDescr
 $Comp
-L eight-bit-computer:74HCT161 U5
+L sixteen-bit-computer:74HCT161 U5
 U 1 1 5FD857CC
 P 3250 1600
@@
 $EndComp
 $Comp
-L eight-bit-computer:74HCT138 U9
+L sixteen-bit-computer:74HCT138 U9
 U 1 1 5FD88A13
 P 5250 1400
@@
 $EndComp
 $Comp
-L eight-bit-computer:74HCT173 U3
+L sixteen-bit-computer:74HCT173 U3
 U 1 1 5FD8D05D
 P 2400 6450
@@
 $EndComp
 $Comp
-L eight-bit-computer:Aux_connection J4
+L sixteen-bit-computer:Aux_connection J4
 U 1 1 5FD8D921
 P 11150 1500
 F 0 "J4" H 11062 2125 50  0000 C CNN
 F 1 "Aux_connection" H 11062 2034 50  0000 C CNN
-F 2 "eight-bit-computer:aux-connection" H 11150 1500 50  0001 C CNN
+F 2 "sixteen-bit-computer:aux-connection" H 11150 1500 50  0001 C CNN
 F 3 "~" H 11150 1500 50  0001 C CNN
 	1    11150 1500
@@
 $EndComp
 $Comp
-L eight-bit-computer:Bus_connection J3
+L sixteen-bit-computer:Bus_connection J3
 U 1 1 5FD8FB3B
 P 9700 1800
 F 0 "J3" H 9562 2725 50  0000 C CNN
 F 1 "Bus_connection" H 9562 2634 50  0000 C CNN
-F 2 "eight-bit-computer:bus-connection" H 9600 2200 50  0001 C CNN
+F 2 "sixteen-bit-computer:bus-connection" H 9600 2200 50  0001 C CNN
 F 3 "~" H 9600 2200 50  0001 C CNN
 	1    9700 1800
@@
 $EndComp
 $Comp
-L eight-bit-computer:Control_signal_backplane J2
+L sixteen-bit-computer:Control_signal_backplane J2
 U 1 1 5FD91862
 P 9400 5450
 F 0 "J2" H 9287 7175 50  0000 C CNN
 F 1 "Control_signal_backplane" H 9287 7084 50  0000 C CNN
-F 2 "eight-bit-computer:backplane-connector-single-row" H 9400 5450 50  0001 C CNN
+F 2 "sixteen-bit-computer:backplane-connector-single-row" H 9400 5450 50  0001 C CNN
 F 3 "~" H 9400 5450 50  0001 C CNN
 	1    9400 5450
@@
 F 0 "D20" H 6450 2100 50  0000 C CNN
 F 1 "LED" H 6300 2100 50  0000 C CNN
-F 2 "eight-bit-computer:LED_D5.0mm_Horizontal_O3.81mm_Z3.0mm" H 6700 2150 50  0001 C CNN
+F 2 "sixteen-bit-computer:LED_D5.0mm_Horizontal_O3.81mm_Z3.0mm" H 6700 2150 50  0001 C CNN
 F 3 "~" H 6700 2150 50  0001 C CNN
 	1    6700 2150
@@
 F 0 "D19" H 6450 1950 50  0000 C CNN
 F 1 "LED" H 6300 1950 50  0000 C CNN
-F 2 "eight-bit-computer:LED_D5.0mm_Horizontal_O3.81mm_Z3.0mm" H 6700 2000 50  0001 C CNN
+F 2 "sixteen-bit-computer:LED_D5.0mm_Horizontal_O3.81mm_Z3.0mm" H 6700 2000 50  0001 C CNN
 F 3 "~" H 6700 2000 50  0001 C CNN
 	1    6700 2000
@@
 F 0 "D18" H 6450 1800 50  0000 C CNN
 F 1 "LED" H 6300 1800 50  0000 C CNN
-F 2 "eight-bit-computer:LED_D5.0mm_Horizontal_O3.81mm_Z3.0mm" H 6700 1850 50  0001 C CNN
+F 2 "sixteen-bit-computer:LED_D5.0mm_Horizontal_O3.81mm_Z3.0mm" H 6700 1850 50  0001 C CNN
 F 3 "~" H 6700 1850 50  0001 C CNN
 	1    6700 1850
@@
 F 0 "D17" H 6450 1650 50  0000 C CNN
 F 1 "LED" H 6300 1650 50  0000 C CNN
-F 2 "eight-bit-computer:LED_D5.0mm_Horizontal_O3.81mm_Z3.0mm" H 6700 1700 50  0001 C CNN
+F 2 "sixteen-bit-computer:LED_D5.0mm_Horizontal_O3.81mm_Z3.0mm" H 6700 1700 50  0001 C CNN
 F 3 "~" H 6700 1700 50  0001 C CNN
 	1    6700 1700
@@
 F 0 "D16" H 6450 1500 50  0000 C CNN
 F 1 "LED" H 6300 1500 50  0000 C CNN
-F 2 "eight-bit-computer:LED_D5.0mm_Horizontal_O3.81mm_Z3.0mm" H 6700 1550 50  0001 C CNN
+F 2 "sixteen-bit-computer:LED_D5.0mm_Horizontal_O3.81mm_Z3.0mm" H 6700 1550 50  0001 C CNN
 F 3 "~" H 6700 1550 50  0001 C CNN
 	1    6700 1550
@@
 F 0 "D15" H 6450 1350 50  0000 C CNN
 F 1 "LED" H 6300 1350 50  0000 C CNN
-F 2 "eight-bit-computer:LED_D5.0mm_Horizontal_O3.81mm_Z3.0mm" H 6700 1400 50  0001 C CNN
+F 2 "sixteen-bit-computer:LED_D5.0mm_Horizontal_O3.81mm_Z3.0mm" H 6700 1400 50  0001 C CNN
 F 3 "~" H 6700 1400 50  0001 C CNN
 	1    6700 1400
@@
 F 0 "D14" H 6450 1200 50  0000 C CNN
 F 1 "LED" H 6300 1200 50  0000 C CNN
-F 2 "eight-bit-computer:LED_D5.0mm_Horizontal_O3.81mm_Z3.0mm" H 6700 1250 50  0001 C CNN
+F 2 "sixteen-bit-computer:LED_D5.0mm_Horizontal_O3.81mm_Z3.0mm" H 6700 1250 50  0001 C CNN
 F 3 "~" H 6700 1250 50  0001 C CNN
 	1    6700 1250
@@
 F 0 "D13" H 6450 1050 50  0000 C CNN
 F 1 "LED" H 6300 1050 50  0000 C CNN
-F 2 "eight-bit-computer:LED_D5.0mm_Horizontal_O3.81mm_Z3.0mm" H 6700 1100 50  0001 C CNN
+F 2 "sixteen-bit-computer:LED_D5.0mm_Horizontal_O3.81mm_Z3.0mm" H 6700 1100 50  0001 C CNN
 F 3 "~" H 6700 1100 50  0001 C CNN
 	1    6700 1100
@@
 F 0 "D5" H 5400 3450 50  0000 C CNN
 F 1 "LED" H 5250 3450 50  0000 C CNN
-F 2 "eight-bit-computer:LED_D5.0mm_Horizontal_O3.81mm_Z3.0mm" H 5650 3500 50  0001 C CNN
+F 2 "sixteen-bit-computer:LED_D5.0mm_Horizontal_O3.81mm_Z3.0mm" H 5650 3500 50  0001 C CNN
 F 3 "~" H 5650 3500 50  0001 C CNN
 	1    5650 3500
@@
 F 0 "D6" H 5400 3600 50  0000 C CNN
 F 1 "LED" H 5250 3600 50  0000 C CNN
-F 2 "eight-bit-computer:LED_D5.0mm_Horizontal_O3.81mm_Z3.0mm" H 5650 3650 50  0001 C CNN
+F 2 "sixteen-bit-computer:LED_D5.0mm_Horizontal_O3.81mm_Z3.0mm" H 5650 3650 50  0001 C CNN
 F 3 "~" H 5650 3650 50  0001 C CNN
 	1    5650 3650
@@
 F 0 "D7" H 5400 3750 50  0000 C CNN
 F 1 "LED" H 5250 3750 50  0000 C CNN
-F 2 "eight-bit-computer:LED_D5.0mm_Horizontal_O3.81mm_Z3.0mm" H 5650 3800 50  0001 C CNN
+F 2 "sixteen-bit-computer:LED_D5.0mm_Horizontal_O3.81mm_Z3.0mm" H 5650 3800 50  0001 C CNN
 F 3 "~" H 5650 3800 50  0001 C CNN
 	1    5650 3800
@@
 F 0 "D8" H 5400 3900 50  0000 C CNN
 F 1 "LED" H 5250 3900 50  0000 C CNN
-F 2 "eight-bit-computer:LED_D5.0mm_Horizontal_O3.81mm_Z3.0mm" H 5650 3950 50  0001 C CNN
+F 2 "sixteen-bit-computer:LED_D5.0mm_Horizontal_O3.81mm_Z3.0mm" H 5650 3950 50  0001 C CNN
 F 3 "~" H 5650 3950 50  0001 C CNN
 	1    5650 3950
@@
 F 0 "D9" H 5400 4050 50  0000 C CNN
 F 1 "LED" H 5250 4050 50  0000 C CNN
-F 2 "eight-bit-computer:LED_D5.0mm_Horizontal_O3.81mm_Z3.0mm" H 5650 4100 50  0001 C CNN
+F 2 "sixteen-bit-computer:LED_D5.0mm_Horizontal_O3.81mm_Z3.0mm" H 5650 4100 50  0001 C CNN
 F 3 "~" H 5650 4100 50  0001 C CNN
 	1    5650 4100
@@
 F 0 "D10" H 5400 4200 50  0000 C CNN
 F 1 "LED" H 5250 4200 50  0000 C CNN
-F 2 "eight-bit-computer:LED_D5.0mm_Horizontal_O3.81mm_Z3.0mm" H 5650 4250 50  0001 C CNN
+F 2 "sixteen-bit-computer:LED_D5.0mm_Horizontal_O3.81mm_Z3.0mm" H 5650 4250 50  0001 C CNN
 F 3 "~" H 5650 4250 50  0001 C CNN
 	1    5650 4250
@@
 F 0 "D11" H 5400 4350 50  0000 C CNN
 F 1 "LED" H 5250 4350 50  0000 C CNN
-F 2 "eight-bit-computer:LED_D5.0mm_Horizontal_O3.81mm_Z3.0mm" H 5650 4400 50  0001 C CNN
+F 2 "sixteen-bit-computer:LED_D5.0mm_Horizontal_O3.81mm_Z3.0mm" H 5650 4400 50  0001 C CNN
 F 3 "~" H 5650 4400 50  0001 C CNN
 	1    5650 4400
@@
 F 0 "D12" H 5400 4500 50  0000 C CNN
 F 1 "LED" H 5250 4500 50  0000 C CNN
-F 2 "eight-bit-computer:LED_D5.0mm_Horizontal_O3.81mm_Z3.0mm" H 5650 4550 50  0001 C CNN
+F 2 "sixteen-bit-computer:LED_D5.0mm_Horizontal_O3.81mm_Z3.0mm" H 5650 4550 50  0001 C CNN
 F 3 "~" H 5650 4550 50  0001 C CNN
 	1    5650 4550
@@
 LIN_STEP_7
 $Comp
-L eight-bit-computer:74HCT245 U8
+L sixteen-bit-computer:74HCT245 U8
 U 1 1 5FED6485
 P 4600 3750
@@
 F 0 "D1" H 5850 5800 50  0000 C CNN
 F 1 "LED" H 5700 5800 50  0000 C CNN
-F 2 "eight-bit-computer:LED_D5.0mm_Horizontal_O3.81mm_Z3.0mm" H 6100 5850 50  0001 C CNN
+F 2 "sixteen-bit-computer:LED_D5.0mm_Horizontal_O3.81mm_Z3.0mm" H 6100 5850 50  0001 C CNN
 F 3 "~" H 6100 5850 50  0001 C CNN
 	1    6100 5850
@@
 F 0 "D2" H 5850 5950 50  0000 C CNN
 F 1 "LED" H 5700 5950 50  0000 C CNN
-F 2 "eight-bit-computer:LED_D5.0mm_Horizontal_O3.81mm_Z3.0mm" H 6100 6000 50  0001 C CNN
+F 2 "sixteen-bit-computer:LED_D5.0mm_Horizontal_O3.81mm_Z3.0mm" H 6100 6000 50  0001 C CNN
 F 3 "~" H 6100 6000 50  0001 C CNN
 	1    6100 6000
@@
 F 0 "D3" H 5850 6100 50  0000 C CNN
 F 1 "LED" H 5700 6100 50  0000 C CNN
-F 2 "eight-bit-computer:LED_D5.0mm_Horizontal_O3.81mm_Z3.0mm" H 6100 6150 50  0001 C CNN
+F 2 "sixteen-bit-computer:LED_D5.0mm_Horizontal_O3.81mm_Z3.0mm" H 6100 6150 50  0001 C CNN
 F 3 "~" H 6100 6150 50  0001 C CNN
 	1    6100 6150
@@
 F 0 "D4" H 5850 6250 50  0000 C CNN
 F 1 "LED" H 5700 6250 50  0000 C CNN
-F 2 "eight-bit-computer:LED_D5.0mm_Horizontal_O3.81mm_Z3.0mm" H 6100 6300 50  0001 C CNN
+F 2 "sixteen-bit-computer:LED_D5.0mm_Horizontal_O3.81mm_Z3.0mm" H 6100 6300 50  0001 C CNN
 F 3 "~" H 6100 6300 50  0001 C CNN
 	1    6100 6300
@@
 $EndComp
 $Comp
-L eight-bit-computer:74HCT245 U7
+L sixteen-bit-computer:74HCT245 U7
 U 1 1 5FFC3890
 P 4750 6100
@@
 INST_00
 $Comp
-L eight-bit-computer:74HCT377 U4
+L sixteen-bit-computer:74HCT377 U4
 U 1 1 5FD843AB
 P 2600 4000

Commit message: Switch to HC series chips and fix some labelling in program counter or register PCB.
Parts:
- U1: value 74HCT04 -> 74HC04; symbol 74xx:74HCT04 -> 74xx:74HC04
- U3: value 74HCT173 -> 74HC173; symbol sixteen-bit-computer:74HCT173 -> sixteen-bit-computer:74HC173
- U4: value 74HCT377 -> 74HC377; symbol sixteen-bit-computer:74HCT377 -> sixteen-bit-computer:74HC377
- U5: value 74HCT161 -> 74HC161; symbol sixteen-bit-computer:74HCT161 -> sixteen-bit-computer:74HC161
- U7, U8: value 74HCT245 -> 74HC245; symbol sixteen-bit-computer:74HCT245 -> sixteen-bit-computer:74HC245
- U9: value 74HCT138 -> 74HC138; symbol sixteen-bit-computer:74HCT138 -> sixteen-bit-computer:74HC138
Changed lines of the file:
@@
 $EndDescr
 $Comp
-L sixteen-bit-computer:74HCT161 U5
+L sixteen-bit-computer:74HC161 U5
 U 1 1 5FD857CC
 P 3250 1600
 F 0 "U5" H 3000 2250 50  0000 C CNN
-F 1 "74HCT161" H 3550 2250 50  0000 C CNN
+F 1 "74HC161" H 3550 2250 50  0000 C CNN
 F 2 "Package_DIP:DIP-16_W7.62mm" H 3250 1600 50  0001 C CNN
 F 3 "https://www.ti.com/lit/ds/symlink/cd54hc163.pdf" H 3250 1600 50  0001 C CNN
@@
 $EndComp
 $Comp
-L sixteen-bit-computer:74HCT138 U9
+L sixteen-bit-computer:74HC138 U9
 U 1 1 5FD88A13
 P 5250 1400
 F 0 "U9" H 5000 1850 50  0000 C CNN
-F 1 "74HCT138" H 5500 1850 50  0000 C CNN
+F 1 "74HC138" H 5500 1850 50  0000 C CNN
 F 2 "Package_DIP:DIP-16_W7.62mm" H 5250 1400 50  0001 C CNN
 F 3 "https://www.ti.com/lit/ds/symlink/sn74hct138.pdf" H 5250 1400 50  0001 C CNN
@@
 $EndComp
 $Comp
-L sixteen-bit-computer:74HCT173 U3
+L sixteen-bit-computer:74HC173 U3
 U 1 1 5FD8D05D
 P 2400 6450
 F 0 "U3" H 2150 7200 50  0000 C CNN
-F 1 "74HCT173" H 2650 7200 50  0000 C CNN
+F 1 "74HC173" H 2650 7200 50  0000 C CNN
 F 2 "Package_DIP:DIP-16_W7.62mm" H 2400 6450 50  0001 C CNN
 F 3 "http://www.ti.com/lit/ds/symlink/cd74hc173.pdf" H 2400 6450 50  0001 C CNN
@@
 $EndComp
 $Comp
-L 74xx:74HCT04 U1
+L 74xx:74HC04 U1
 U 1 1 5FDAA11A
 P 1350 1600
 F 0 "U1" H 1350 1917 50  0000 C CNN
-F 1 "74HCT04" H 1350 1826 50  0000 C CNN
+F 1 "74HC04" H 1350 1826 50  0000 C CNN
 F 2 "Package_DIP:DIP-14_W7.62mm" H 1350 1600 50  0001 C CNN
 F 3 "https://assets.nexperia.com/documents/data-sheet/74HC_HCT04.pdf" H 1350 1600 50  0001 C CNN
@@
 $EndComp
 $Comp
-L 74xx:74HCT04 U1
+L 74xx:74HC04 U1
 U 2 1 5FDAB5DB
 P 1350 2100
 F 0 "U1" H 1350 2417 50  0000 C CNN
-F 1 "74HCT04" H 1350 2326 50  0000 C CNN
+F 1 "74HC04" H 1350 2326 50  0000 C CNN
 F 2 "Package_DIP:DIP-14_W7.62mm" H 1350 2100 50  0001 C CNN
 F 3 "https://assets.nexperia.com/documents/data-sheet/74HC_HCT04.pdf" H 1350 2100 50  0001 C CNN
@@
 $EndComp
 $Comp
-L 74xx:74HCT04 U1
+L 74xx:74HC04 U1
 U 3 1 5FDACA10
 P 12400 5200
 F 0 "U1" H 12400 5517 50  0000 C CNN
-F 1 "74HCT04" H 12400 5426 50  0000 C CNN
+F 1 "74HC04" H 12400 5426 50  0000 C CNN
 F 2 "Package_DIP:DIP-14_W7.62mm" H 12400 5200 50  0001 C CNN
 F 3 "https://assets.nexperia.com/documents/data-sheet/74HC_HCT04.pdf" H 12400 5200 50  0001 C CNN
@@
 $EndComp
 $Comp
-L 74xx:74HCT04 U1
+L 74xx:74HC04 U1
 U 4 1 5FDAE4A7
 P 13000 5200
 F 0 "U1" H 13000 5517 50  0000 C CNN
-F 1 "74HCT04" H 13000 5426 50  0000 C CNN
+F 1 "74HC04" H 13000 5426 50  0000 C CNN
 F 2 "Package_DIP:DIP-14_W7.62mm" H 13000 5200 50  0001 C CNN
 F 3 "https://assets.nexperia.com/documents/data-sheet/74HC_HCT04.pdf" H 13000 5200 50  0001 C CNN
@@
 $EndComp
 $Comp
-L 74xx:74HCT04 U1
+L 74xx:74HC04 U1
 U 5 1 5FDAF775
 P 13550 5200
 F 0 "U1" H 13550 5517 50  0000 C CNN
-F 1 "74HCT04" H 13550 5426 50  0000 C CNN
+F 1 "74HC04" H 13550 5426 50  0000 C CNN
 F 2 "Package_DIP:DIP-14_W7.62mm" H 13550 5200 50  0001 C CNN
 F 3 "https://assets.nexperia.com/documents/data-sheet/74HC_HCT04.pdf" H 13550 5200 50  0001 C CNN
@@
 $EndComp
 $Comp
-L 74xx:74HCT04 U1
+L 74xx:74HC04 U1
 U 6 1 5FDB0B8C
 P 14100 5200
 F 0 "U1" H 14100 5517 50  0000 C CNN
-F 1 "74HCT04" H 14100 5426 50  0000 C CNN
+F 1 "74HC04" H 14100 5426 50  0000 C CNN
 F 2 "Package_DIP:DIP-14_W7.62mm" H 14100 5200 50  0001 C CNN
 F 3 "https://assets.nexperia.com/documents/data-sheet/74HC_HCT04.pdf" H 14100 5200 50  0001 C CNN
@@
 $EndComp
 $Comp
-L 74xx:74HCT04 U1
+L 74xx:74HC04 U1
 U 7 1 5FDB292F
 P 11350 5000
 F 0 "U1" H 11580 5046 50  0000 L CNN
-F 1 "74HCT04" H 11580 4955 50  0000 L CNN
+F 1 "74HC04" H 11580 4955 50  0000 L CNN
 F 2 "Package_DIP:DIP-14_W7.62mm" H 11350 5000 50  0001 C CNN
 F 3 "https://assets.nexperia.com/documents/data-sheet/74HC_HCT04.pdf" H 11350 5000 50  0001 C CNN
@@
 LIN_STEP_7
 $Comp
-L sixteen-bit-computer:74HCT245 U8
+L sixteen-bit-computer:74HC245 U8
 U 1 1 5FED6485
 P 4600 3750
 F 0 "U8" H 4400 4450 50  0000 C CNN
-F 1 "74HCT245" H 4850 4450 50  0000 C CNN
+F 1 "74HC245" H 4850 4450 50  0000 C CNN
 F 2 "Package_DIP:DIP-20_W7.62mm" H 4250 3750 50  0001 C CNN
 F 3 "" H 4250 3750 50  0001 C CNN
@@
 $EndComp
 $Comp
-L sixteen-bit-computer:74HCT245 U7
+L sixteen-bit-computer:74HC245 U7
 U 1 1 5FFC3890
 P 4750 6100
 F 0 "U7" H 4550 6800 50  0000 C CNN
-F 1 "74HCT245" H 5000 6800 50  0000 C CNN
+F 1 "74HC245" H 5000 6800 50  0000 C CNN
 F 2 "Package_DIP:DIP-20_W7.62mm" H 4400 6100 50  0001 C CNN
 F 3 "" H 4400 6100 50  0001 C CNN
@@
 INST_00
 $Comp
-L sixteen-bit-computer:74HCT377 U4
+L sixteen-bit-computer:74HC377 U4
 U 1 1 5FD843AB
 P 2600 4000
 F 0 "U4" H 2350 4650 50  0000 C CNN
-F 1 "74HCT377" H 2850 4650 50  0000 C CNN
+F 1 "74HC377" H 2850 4650 50  0000 C CNN
 F 2 "Package_DIP:DIP-20_W7.62mm" H 2600 4000 50  0001 C CNN
 F 3 "http://www.ti.com/lit/gpn/sn74LS377" H 2600 4000 50  0001 C CNN
