File: kicad/projects/rom_counter/rom_counter.kicad_sch (KiCad schematic)
At the start: 27 parts, among them J1 peripheral_addr_bus_connector, J2 peripheral_aux_connector, J3 peripheral_membank_connector, J4 Conn_02x16_Odd_Even, J5 Conn_01x16_Socket, J6 Conn_01x02_Socket, U1 28C256, U10 74HC161, U11 74HC245, U12 74HC245, U2 28C256, U3 74HC30, U4 74HC30, U5 74HC32, U6 74HC00, U7 74HC161, U8 74HC161, U9 74HC161

Commit message: Connect up counter chips in rom counter schematic.
Parts:
- added J7: Conn_01x02_Pin, symbol Connector:Conn_01x02_Pin
- added R3: 10K, Resistor_THT:R_Axial_DIN0207_L6.3mm_D2.5mm_P10.16mm_Horizontal, symbol Device:R_US
- D1, D2: footprint (none) -> sixteen-bit-computer:LED_D5.0mm_Horizontal_O3.81mm_Z3.0mm
- J4: footprint (none) -> Connector_PinHeader_2.54mm:PinHeader_2x16_P2.54mm_Vertical
- J5: footprint (none) -> Connector_PinSocket_2.54mm:PinSocket_1x16_P2.54mm_Horizontal
- J6: footprint (none) -> Connector_PinSocket_2.54mm:PinSocket_1x02_P2.54mm_Horizontal
- R1, R2: footprint (none) -> Resistor_THT:R_Axial_DIN0207_L6.3mm_D2.5mm_P10.16mm_Horizontal
- U1, U2: footprint (none) -> Package_DIP:DIP-28_W15.24mm_Socket
- U10, U7, U8, U9: footprint (none) -> Package_DIP:DIP-16_W7.62mm_Socket
- U11, U12: footprint (none) -> Package_DIP:DIP-20_W7.62mm_Socket
- U3, U4, U5, U6: footprint (none) -> Package_DIP:DIP-14_W7.62mm_Socket
Connections:
- net GND: now also U10.3 (P0), U10.4 (P1), U10.5 (P2), U10.6 (P3), U7.3 (P0), U7.4 (P1), U7.5 (P2), U7.6 (P3), U8.3 (P0), U8.4 (P1), U8.5 (P2), U8.6 (P3), U9.3 (P0), U9.4 (P1), U9.5 (P2), U9.6 (P3)
- net VCC: now also R3.2
- net at U8.1 (~{MR}): now also U10.1 (~{MR}), U7.1 (~{MR}), U9.1 (~{MR})
- net at U8.10 (TE): now also U7.15 (TC)
- net COUNT_07: now reaches U8.11 (Q3)
- net COUNT_06: now reaches U8.12 (Q2)
- net COUNT_05: now reaches U8.13 (Q1)
- net COUNT_04: now reaches U8.14 (Q0)
- net at U8.15 (TC): now also U9.10 (TE)
- net at U8.2 (CP): now also U10.2 (CP), U7.2 (CP), U9.2 (CP)
- net at U8.7 (PE): now also U10.7 (PE), U7.10 (TE), U9.7 (PE)
- net at U8.9 (~{SPE}): now also U10.9 (~{SPE}), U7.7 (PE), U9.9 (~{SPE})
- net at U10.10 (TE): now also U9.15 (TC)
- net COUNT_15: now reaches U10.11 (Q3)
- net COUNT_14: now reaches U10.12 (Q2)
- net COUNT_13: now reaches U10.13 (Q1)
- net COUNT_12: now reaches U10.14 (Q0)
- net COUNT_11: now reaches U9.11 (Q3)
- net COUNT_10: now reaches U9.12 (Q2)
- net COUNT_09: now reaches U9.13 (Q1)
- net COUNT_08: now reaches U9.14 (Q0)
- net COUNT_03: now reaches U7.11 (Q3)
- net COUNT_02: now reaches U7.12 (Q2)
- net COUNT_01: now reaches U7.13 (Q1)
- net COUNT_00: now reaches U7.14 (Q0)
Other:
- moved on the sheet: D1, J6, R1, U10, U5C, U6B, U7, U8, U9

Commit message: most of schematic done for rom counter
Parts:
- added C1, C10, C11, C12, C2, C3, C4, C5, C6, C7, C8, C9: C, symbol Device:C
- added R4: 10K, Resistor_THT:R_Axial_DIN0207_L6.3mm_D2.5mm_P10.16mm_Horizontal, symbol Device:R_US
- R1, R2: value R_US -> 1K
Connections:
- net ADDR_BUS_00: now also U1.10 (A0), U2.10 (A0)
- net ADDR_BUS_01: now also U1.9 (A1), U2.9 (A1)
- net ADDR_BUS_02: now also U1.8 (A2), U2.8 (A2)
- net ADDR_BUS_03: now also U1.7 (A3), U2.7 (A3)
- net ADDR_BUS_04: now also U1.6 (A4), U2.6 (A4)
- net ADDR_BUS_05: now also U1.5 (A5), U2.5 (A5)
- net ADDR_BUS_06: now also U1.4 (A6), U2.4 (A6)
- net ADDR_BUS_07: now also U1.3 (A7), U2.3 (A7)
- net ADDR_BUS_08: now also U1.25 (A8), U2.25 (A8)
- net ADDR_BUS_09: now also U1.24 (A9), U2.24 (A9)
- net ADDR_BUS_10: now also U1.21 (A10), U2.21 (A10)
- net ADDR_BUS_11: now also U1.23 (A11), U2.23 (A11)
- net ADDR_BUS_12: now also U1.2 (A12), U2.2 (A12)
- net ADDR_BUS_13: now also U1.26 (A13), U2.26 (A13)
- net ADDR_BUS_14: now also U1.1 (A14), U2.1 (A14)
- net BANK_BUS_00: now also J4.1 (Pin_1)
- net BANK_BUS_01: now also J4.3 (Pin_3)
- net BANK_BUS_02: now also J4.5 (Pin_5)
- net BANK_BUS_03: now also J4.7 (Pin_7)
- net BANK_BUS_04: now also J4.9 (Pin_9)
- net BANK_BUS_05: now also J4.11 (Pin_11)
- net BANK_BUS_06: now also J4.13 (Pin_13)
- net BANK_BUS_07: now also J4.15 (Pin_15)
- net BANK_BUS_08: now also J4.17 (Pin_17)
- net BANK_BUS_09: now also J4.19 (Pin_19)
- net BANK_BUS_10: now also J4.21 (Pin_21)
- net BANK_BUS_11: now also J4.23 (Pin_23)
- net BANK_BUS_12: now also J4.25 (Pin_25)
- net BANK_BUS_13: now also J4.27 (Pin_27)
- net BANK_BUS_14: now also J4.29 (Pin_29)
- net BANK_BUS_15: now also J4.31 (Pin_31)
- net COUNT_00: now also J5.1 (Pin_1), U11.2 (A1)
- net COUNT_01: now also J5.2 (Pin_2), U11.3 (A2)
- net COUNT_02: now also J5.3 (Pin_3), U11.4 (A3)
- net COUNT_03: now also J5.4 (Pin_4), U11.5 (A3)
- net COUNT_04: now also J5.5 (Pin_5), U11.6 (A5)
- net COUNT_05: now also J5.6 (Pin_6), U11.7 (A6)
- net COUNT_06: now also J5.7 (Pin_7), U11.8 (A7)
- net COUNT_07: now also J5.8 (Pin_8), U11.9 (A8)
- net COUNT_08: now also J5.9 (Pin_9), U12.2 (A1)
- net COUNT_09: now also J5.10 (Pin_10), U12.3 (A2)
- net COUNT_10: now also J5.11 (Pin_11), U12.4 (A3)
- net COUNT_11: now also J5.12 (Pin_12), U12.5 (A3)
- net COUNT_12: now also J5.13 (Pin_13), U12.6 (A5)
- net COUNT_13: now also J5.14 (Pin_14), U12.7 (A6)
- net COUNT_14: now also J5.15 (Pin_15), U12.8 (A7)
- net COUNT_15: now also J5.16 (Pin_16), U12.9 (A8)
- net CTL_CLK: now also U10.2 (CP), U7.2 (CP), U8.2 (CP), U9.2 (CP)
- net DATA_BUS_00: now also U1.11 (D0), U11.18 (B1)
- net DATA_BUS_01: now also U1.12 (D1), U11.17 (B2)
- net DATA_BUS_02: now also U1.13 (D2), U11.16 (B3)
- net DATA_BUS_03: now also U1.15 (D3), U11.15 (B4)
- net DATA_BUS_04: now also U1.16 (D4), U11.14 (B5)
- net DATA_BUS_05: now also U1.17 (D5), U11.13 (B6)
- net DATA_BUS_06: now also U1.18 (D6), U11.12 (B7)
- net DATA_BUS_07: now also U1.19 (D7), U11.11 (B8)
- net DATA_BUS_08: now also U12.18 (B1), U2.11 (D0)
- net DATA_BUS_09: now also U12.17 (B2), U2.12 (D1)
- net DATA_BUS_10: now also U12.16 (B3), U2.13 (D2)
- net DATA_BUS_11: now also U12.15 (B4), U2.15 (D3)
- net DATA_BUS_12: now also U12.14 (B5), U2.16 (D4)
- net DATA_BUS_13: now also U12.13 (B6), U2.17 (D5)
- net DATA_BUS_14: now also U12.12 (B7), U2.18 (D6)
- net DATA_BUS_15: now also U12.11 (B8), U2.19 (D7)
- net GND: now also R1.2, U1.14 (GND), U1.20 (~{CS}), U10.8 (GND), U11.10 (GND), U12.10 (GND), U2.14 (GND), U2.20 (~{CS}), U3.7 (GND), U4.7 (GND), U5.12, U5.13, U5.7 (GND), U6.7 (GND), U7.8 (GND), U8.8 (GND), U9.8 (GND), C1.1, C10.1, C11.2, C12.2, C2.1, C3.1, C4.1, C5.1, C6.1, C7.1, C8.1, C9.1
- net RESET: now also U6.4, U6.5
- net RFM: now also U6.12, U6.2
- net VCC: now also U1.27 (~{WE}), U1.28 (VCC), U10.16 (VCC), U10.7 (PE), U10.9 (~{SPE}), U11.1 (DIR), U11.20 (VCC), U12.1 (DIR), U12.20 (VCC), U2.27 (~{WE}), U2.28 (VCC), U3.14 (VCC), U4.14 (VCC), U5.14 (VCC), U6.14 (VCC), U7.10 (TE), U7.16 (VCC), U7.7 (PE), U7.9 (~{SPE}), U8.16 (VCC), U8.7 (PE), U8.9 (~{SPE}), U9.16 (VCC), U9.7 (PE), U9.9 (~{SPE}), C1.2, C10.2, C11.1, C12.1, C2.2, C3.2, C4.2, C5.2, C6.2, C7.2, C8.2, C9.2, R4.2
- net ~{ROM OE}: now reaches U1.22 (~{OE})
- net ~{ROM OE}: now also U2.22 (~{OE}), U6.3
- net ~{COUNTER ADDRESSED}: now reaches U6.10
- net ~{COUNTER ADDRESSED}: now also J6.1 (Pin_1), J6.2 (Pin_2), U6.9, R4.1
- net COUNTER ADDRESSED: now reaches U6.8
- net COUNTER ADDRESSED: now also U5.10, U5.9, U6.13
- net at R2.1: now also D2.1 (K)
- net at U10.1 (~{MR}), U7.1 (~{MR}), U8.1 (~{MR})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: now also J7.1 (Pin_1), R3.1
- net at U6.6: now also J7.2 (Pin_2)
- net at RN2.2 (R1): now also J4.32 (Pin_32), U4.12 (H)
- net at RN2.3 (R2): now also J4.30 (Pin_30), U4.11 (G)
- net at RN2.4 (R3): now also J4.28 (Pin_28), U4.6 (F)
- net at RN2.5 (R4): now also J4.26 (Pin_26), U4.5 (E)
- net at RN2.6 (R5): now also J4.24 (Pin_24), U4.4 (D)
- net at RN2.7 (R6): now also J4.22 (Pin_22), U4.3 (C)
- net at RN2.8 (R7): now also J4.20 (Pin_20), U4.2 (B)
- net at RN2.9 (R8): now also J4.18 (Pin_18), U4.1 (A)
- net at D1.1 (K): now also R1.1
- net at D1.2 (A): now also U5.8
- net ROM ADDRESSED: now reaches U6.1
- net ROM ADDRESSED: now also U5.3, U5.4, U5.5
- net ~{COUNTER OE}: now reaches U11.19 (~{OE})
- net ~{COUNTER OE}: now also U12.19 (~{OE}), U6.11
- net at RN1.2 (R1): now also J4.2 (Pin_2), U3.1 (A)
- net at RN1.3 (R2): now also J4.4 (Pin_4), U3.2 (B)
- net at RN1.4 (R3): now also J4.6 (Pin_6), U3.3 (C)
- net at RN1.5 (R4): now also J4.8 (Pin_8), U3.4 (D)
- net at RN1.6 (R5): now also J4.10 (Pin_10), U3.5 (E)
- net at RN1.7 (R6): now also J4.12 (Pin_12), U3.6 (F)
- net at RN1.8 (R7): now also J4.14 (Pin_14), U3.11 (G)
- net at RN1.9 (R8): now also J4.16 (Pin_16), U3.12 (H)
- net at D2.2 (A): now also U5.6
- net at U3.8 (~{Y}): now also U5.1
- net at U5.2: now also U4.8 (~{Y})
- no-connect marks 0 -> 2
Other:
- moved on the sheet: D1, D2, J4, J5, J6, J7, R1, R2, R3, RN1, RN2, U1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

Commit message: Start PCB layout of ROM counter.
Parts:
- C1, C10, C11, C12, C2, C3, C4, C5, C6, C7, C8, C9: footprint (none) -> Capacitor_THT:C_Disc_D5.0mm_W2.5mm_P5.00mm
- J7: footprint (none) -> Connector_PinHeader_2.54mm:PinHeader_1x02_P2.54mm_Horizontal
Connections:
- net BANK_BUS_00: now also J4.31 (Pin_31); no longer J4.1 (Pin_1)
- net BANK_BUS_01: now also J4.29 (Pin_29); no longer J4.3 (Pin_3)
- net BANK_BUS_02: now also J4.27 (Pin_27); no longer J4.5 (Pin_5)
- net BANK_BUS_03: now also J4.25 (Pin_25); no longer J4.7 (Pin_7)
- net BANK_BUS_04: now also J4.23 (Pin_23); no longer J4.9 (Pin_9)
- net BANK_BUS_05: now also J4.21 (Pin_21); no longer J4.11 (Pin_11)
- net BANK_BUS_06: now also J4.19 (Pin_19); no longer J4.13 (Pin_13)
- net BANK_BUS_07: now also J4.17 (Pin_17); no longer J4.15 (Pin_15)
- net BANK_BUS_08: now also J4.15 (Pin_15); no longer J4.17 (Pin_17)
- net BANK_BUS_09: now also J4.13 (Pin_13); no longer J4.19 (Pin_19)
- net BANK_BUS_10: now also J4.11 (Pin_11); no longer J4.21 (Pin_21)
- net BANK_BUS_11: now also J4.9 (Pin_9); no longer J4.23 (Pin_23)
- net BANK_BUS_12: now also J4.7 (Pin_7); no longer J4.25 (Pin_25)
- net BANK_BUS_13: now also J4.5 (Pin_5); no longer J4.27 (Pin_27)
- net BANK_BUS_14: now also J4.3 (Pin_3); no longer J4.29 (Pin_29)
- net BANK_BUS_15: now also J4.1 (Pin_1); no longer J4.31 (Pin_31)
- net ~{COUNTER ADDRESSED}: no longer J6.1 (Pin_1), J6.2 (Pin_2), R4.1, U6.10, U6.9
- new net: J6.1 (Pin_1), J6.2 (Pin_2), R4.1, U6.10, U6.9
Other:
- note added: "Counter and reset control"
- note added: "Counter content and bus output control"
- note added: "ROM bank selection and output enable"
- moved on the sheet: C1, C10, C11, C12, C2, C3, C4, C5, C6, C7, C8, C9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

Commit message: More PCB work on ROM counter.
Connections:
- net GND: now also R2.2
- net VCC: now also RN1.1 (common), RN2.1 (common)
Changed lines of the file:
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@@
 (kicad_sch (version 20230121) (generator eeschema)
   (paper "B")
+  (bus_alias "ADDR_BUS" (members "ADDR_BUS_00" "ADDR_BUS_01" "ADDR_BUS_02" "ADDR_BUS_03" "ADDR_BUS_04" "ADDR_BUS_05" "ADDR_BUS_06" "ADDR_BUS_07" "ADDR_BUS_08" "ADDR_BUS_09" "ADDR_BUS_10" "ADDR_BUS_11" "ADDR_BUS_12" "ADDR_BUS_13" "ADDR_BUS_14" "ADDR_BUS_15"))
   (bus_alias "DATA_BUS" (members "DATA_BUS_00" "DATA_BUS_01" "DATA_BUS_02" "DATA_BUS_03" "DATA_BUS_04" "DATA_BUS_05" "DATA_BUS_06" "DATA_BUS_07" "DATA_BUS_08" "DATA_BUS_09" "DATA_BUS_10" "DATA_BUS_11" "DATA_BUS_12" "DATA_BUS_13" "DATA_BUS_14" "DATA_BUS_15"))
   (bus_alias "BANK_BUS" (members "BANK_BUS_00" "BANK_BUS_01" "BANK_BUS_02" "BANK_BUS_03" "BANK_BUS_04" "BANK_BUS_05" "BANK_BUS_06" "BANK_BUS_07" "BANK_BUS_08" "BANK_BUS_09" "BANK_BUS_10" "BANK_BUS_11" "BANK_BUS_12" "BANK_BUS_13" "BANK_BUS_14" "BANK_BUS_15"))
-  (bus_alias "ADDR_BUS" (members "ADDR_BUS_00" "ADDR_BUS_01" "ADDR_BUS_02" "ADDR_BUS_03" "ADDR_BUS_04" "ADDR_BUS_05" "ADDR_BUS_06" "ADDR_BUS_07" "ADDR_BUS_08" "ADDR_BUS_09" "ADDR_BUS_10" "ADDR_BUS_11" "ADDR_BUS_12" "ADDR_BUS_13" "ADDR_BUS_14" "ADDR_BUS_15"))
   (junction (at 214.63 130.175) (diameter 0) (color 0 0 0 0)
   )
@@
     (stroke (width 0) (type default))
   )
+  (wire (pts (xy 204.47 174.625) (xy 204.47 172.085))
+    (stroke (width 0) (type default))
+  )
   (wire (pts (xy 224.79 74.93) (xy 240.03 74.93))
     (stroke (width 0) (type default))
@@
     (effects (font (size 1.27 1.27)) (justify left bottom))
   )
+  (label "VCC" (at 204.47 106.045 0) (fields_autoplaced)
+    (effects (font (size 1.27 1.27)) (justify left bottom))
+  )
   (label "BANK_BUS_00" (at 78.74 146.685 0) (fields_autoplaced)
     (effects (font (size 1.27 1.27)) (justify left bottom))
@@
     (effects (font (size 1.27 1.27)) (justify right bottom))
   )
+  (label "GND" (at 304.8 123.19 0) (fields_autoplaced)
+    (effects (font (size 1.27 1.27)) (justify left bottom))
+  )
   (label "COUNT_13" (at 47.625 97.79 270) (fields_autoplaced)
     (effects (font (size 1.27 1.27)) (justify right bottom))
@@
     (effects (font (size 1.27 1.27)) (justify left bottom))
   )
+  (label "VCC" (at 204.47 174.625 0) (fields_autoplaced)
+    (effects (font (size 1.27 1.27)) (justify left bottom))
+  )

Commit message: Labelling on Counter Rom board, tiny bit more to go.
Parts:
- RN1, RN2: value R_Network08_US -> 10K
Connections:
- net COUNTER ADDRESSED LED: now reaches D1.2 (A), U5.8
- net ROM ADDRESSED LED: now reaches D2.2 (A), U5.6
Changed lines of the file:
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@@
 (kicad_sch (version 20230121) (generator eeschema)
   (paper "B")
+  (bus_alias "BANK_BUS" (members "BANK_BUS_00" "BANK_BUS_01" "BANK_BUS_02" "BANK_BUS_03" "BANK_BUS_04" "BANK_BUS_05" "BANK_BUS_06" "BANK_BUS_07" "BANK_BUS_08" "BANK_BUS_09" "BANK_BUS_10" "BANK_BUS_11" "BANK_BUS_12" "BANK_BUS_13" "BANK_BUS_14" "BANK_BUS_15"))
+  (bus_alias "DATA_BUS" (members "DATA_BUS_00" "DATA_BUS_01" "DATA_BUS_02" "DATA_BUS_03" "DATA_BUS_04" "DATA_BUS_05" "DATA_BUS_06" "DATA_BUS_07" "DATA_BUS_08" "DATA_BUS_09" "DATA_BUS_10" "DATA_BUS_11" "DATA_BUS_12" "DATA_BUS_13" "DATA_BUS_14" "DATA_BUS_15"))
   (bus_alias "ADDR_BUS" (members "ADDR_BUS_00" "ADDR_BUS_01" "ADDR_BUS_02" "ADDR_BUS_03" "ADDR_BUS_04" "ADDR_BUS_05" "ADDR_BUS_06" "ADDR_BUS_07" "ADDR_BUS_08" "ADDR_BUS_09" "ADDR_BUS_10" "ADDR_BUS_11" "ADDR_BUS_12" "ADDR_BUS_13" "ADDR_BUS_14" "ADDR_BUS_15"))
-  (bus_alias "DATA_BUS" (members "DATA_BUS_00" "DATA_BUS_01" "DATA_BUS_02" "DATA_BUS_03" "DATA_BUS_04" "DATA_BUS_05" "DATA_BUS_06" "DATA_BUS_07" "DATA_BUS_08" "DATA_BUS_09" "DATA_BUS_10" "DATA_BUS_11" "DATA_BUS_12" "DATA_BUS_13" "DATA_BUS_14" "DATA_BUS_15"))
-  (bus_alias "BANK_BUS" (members "BANK_BUS_00" "BANK_BUS_01" "BANK_BUS_02" "BANK_BUS_03" "BANK_BUS_04" "BANK_BUS_05" "BANK_BUS_06" "BANK_BUS_07" "BANK_BUS_08" "BANK_BUS_09" "BANK_BUS_10" "BANK_BUS_11" "BANK_BUS_12" "BANK_BUS_13" "BANK_BUS_14" "BANK_BUS_15"))
   (junction (at 214.63 130.175) (diameter 0) (color 0 0 0 0)
   )
@@
   (junction (at 274.32 123.19) (diameter 0) (color 0 0 0 0)
   )
+  (junction (at 289.56 123.19) (diameter 0) (color 0 0 0 0)
+  )
   (junction (at 219.71 135.255) (diameter 0) (color 0 0 0 0)
   )
@@
   )
   (junction (at 234.315 213.36) (diameter 0) (color 0 0 0 0)
+  )
+  (junction (at 59.055 66.675) (diameter 0) (color 0 0 0 0)
   )
   (junction (at 59.055 40.005) (diameter 0) (color 0 0 0 0)
@@
     (stroke (width 0) (type default))
   )
+  (wire (pts (xy 59.055 66.675) (xy 59.055 74.295))
+    (stroke (width 0) (type default))
+  )
   (wire (pts (xy 217.17 145.415) (xy 229.87 145.415))
     (stroke (width 0) (type default))
@@
     (stroke (width 0) (type default))
   )
-  (wire (pts (xy 56.515 66.675) (xy 64.135 66.675))
+  (wire (pts (xy 56.515 66.675) (xy 59.055 66.675))
     (stroke (width 0) (type default))
   )
@@
     (stroke (width 0) (type default))
   )
+  (wire (pts (xy 289.56 112.395) (xy 289.56 123.19))
+    (stroke (width 0) (type default))
+  )
   (wire (pts (xy 93.98 33.655) (xy 97.155 33.655))
     (stroke (width 0) (type default))
@@
   )
   (bus (pts (xy 94.615 156.845) (xy 94.615 159.385))
+    (stroke (width 0) (type default))
+  )
+  (wire (pts (xy 59.055 66.675) (xy 64.135 66.675))
     (stroke (width 0) (type default))
   )
@@
     (effects (font (size 1.27 1.27)) (justify left bottom))
   )
+  (label "ROM ADDRESSED LED" (at 289.56 112.395 180) (fields_autoplaced)
+    (effects (font (size 1.27 1.27)) (justify right bottom))
+  )
   (label "BANK_BUS_04" (at 78.74 156.845 0) (fields_autoplaced)
     (effects (font (size 1.27 1.27)) (justify left bottom))
@@
   (label "COUNT_13" (at 109.22 110.49 180) (fields_autoplaced)
     (effects (font (size 1.27 1.27)) (justify right bottom))
+  )
+  (label "COUNTER ADDRESSED LED" (at 59.055 74.295 0) (fields_autoplaced)
+    (effects (font (size 1.27 1.27)) (justify left bottom))
   )
   (label "ADDR_BUS_13" (at 39.37 216.535 0) (fields_autoplaced)
@@
       (effects (font (size 1.27 1.27)) (justify left))
     )
-    (property "Value" "R_Network08_US" (at 225.425 164.846 0)
+    (property "Value" "10K" (at 225.425 164.846 0)
       (effects (font (size 1.27 1.27)) (justify left))
     )
@@
       (effects (font (size 1.27 1.27)) (justify left))
     )
-    (property "Value" "R_Network08_US" (at 224.79 113.284 0)
+    (property "Value" "10K" (at 224.79 113.284 0)
       (effects (font (size 1.27 1.27)) (justify left))
     )
