File: kicad/templates/cpu_board/cpu_board.kicad_sch (KiCad schematic)
At the start: 6 parts, among them J1 Aux_connection, J2 Bus_connection, J3 Control_signal_backplane

Commit message: Start gamepad.
Parts:
- added C1: C, Capacitor_THT:C_Disc_D5.0mm_W2.5mm_P5.00mm, symbol Device:C
- added D1, D2: LED, sixteen-bit-computer:LED_D5.0mm_Horizontal_O3.81mm_Z3.0mm, symbol Device:LED
- added J4: Conn_01x03_Pin, Connector_PinHeader_2.54mm:PinHeader_1x03_P2.54mm_Horizontal, symbol Connector:Conn_01x03_Pin
- added J5: Conn_01x16_Socket, Connector_PinSocket_2.54mm:PinSocket_1x16_P2.54mm_Horizontal, symbol Connector:Conn_01x16_Socket
- added J6: Conn_01x02_Socket, Connector_PinSocket_2.54mm:PinSocket_1x02_P2.54mm_Horizontal, symbol Connector:Conn_01x02_Socket
- added R1: R_US, Resistor_THT:R_Axial_DIN0207_L6.3mm_D2.5mm_P10.16mm_Horizontal, symbol Device:R_US
- added TP1: TestPoint, Connector_Pin:Pin_D1.0mm_L10.0mm, symbol Connector:TestPoint
- C97, C98, C99: footprint (none) -> Capacitor_THT:CP_Radial_D6.3mm_P2.50mm
- J1: footprint (none) -> sixteen-bit-computer:aux-connection
- J2: footprint (none) -> sixteen-bit-computer:bus-connection
- J3: footprint (none) -> sixteen-bit-computer:backplane-connector-single-row-annotated
Connections:
- net GND: now also J1.3 (GND), J1.4 (GND), C1.2, J6.2 (Pin_2), R1.2, TP1.1
- net VCC: now also J1.1 (VCC), J1.2 (VCC), C1.1, J6.1 (Pin_1), R1.1
