File: kicad/projects/video_cursor/video_cursor.kicad_pcb (KiCad board)
At the start: 2 copper layers, 203.2 x 97.8 mm, 27 parts, among them J1 peripheral_addr_bus_connector, J2 peripheral_aux_connector, J3 peripheral_membank_connector, J4 Conn_01x16_Socket, J5 Conn_01x16_Socket, J6 Conn_01x16_Socket, U1 74HC245, U10 74HC245, U11 74HC245, U12 74HC02, U13 74HC08, U14 74HC123, U15 74HC04, U2 74HC245, U3 74HC245, U4 74HC245, U5 74HC245, U6 74HC245, U7 74HC138, U8 74HC377, U9 74HC377

Commit message: Roughing out the video baords - time to switch to 157s for bank sel as well.
Parts:
- removed U15: 74HC04, Package_DIP:DIP-14_W7.62mm_Socket
- U12: value 74HC02 -> 74HC08
- U13: value 74HC08 -> 74HC00
- U14: value 74HC123 -> 74HC32; footprint Package_DIP:DIP-16_W7.62mm_Socket -> Package_DIP:DIP-14_W7.62mm_Socket
- moved U7 146.1 mm to (185.4, 63.5)
- moved U13 127.4 mm to (78.7, 83.8)
- moved U10 121.9 mm to (66.0, 129.5)
- moved U11 121.9 mm to (104.1, 129.5)
- moved U8 121.9 mm to (66.0, 114.3)
- moved U9 121.9 mm to (104.1, 114.3)
- moved U14 99.2 mm to (104.1, 83.8)
- moved U1 96.5 mm to (152.4, 83.8)
- moved U4 96.5 mm to (152.4, 114.3)
- moved U2 91.4 mm to (185.4, 83.8)
- moved U5 91.4 mm to (185.4, 114.3)
- moved U3 86.4 mm to (218.4, 83.8)
- moved U6 86.4 mm to (218.4, 114.3)
- moved U12 21.6 mm to (160.0, 63.5)
Routing:
- net (no net): track 1422.4 -> 1524.0 mm
