File: kicad/projects/gamepad/gamepad.kicad_sch (KiCad schematic)
At the start: 77 parts, among them J1 peripheral_addr_bus_connector, J10 Pad 2 SNES, J11 Conn_01x03_Pin, J2 peripheral_aux_connector, J3 peripheral_membank_connector, J4 PAD 1 ACTIVE, J5 PAD 2 ACTIVE, J6 Conn_02x05_Odd_Even, J7 Pad 1 header, J8 Pad 1 SNES, J9 Pad 2 header, U1 74HC161, U10 74HC245, U11 74HC245, U12 74HC245, U13 74HC245, U14 74HC00, U15 74HC00, U2 74HC161, U3 74HC595, U4 74HC595, U5 74HC595, U6 74HC595, U7 74HC14, U8 74HC00, U9 74HC161

Commit message: Part way through simplifying gamepad PCB.
Parts:
- removed C14: C, Capacitor_THT:C_Disc_D5.0mm_W2.5mm_P5.00mm, symbol Device:C
- removed TP2: Shift out reg CLK, Connector_Pin:Pin_D1.0mm_L10.0mm, symbol Connector:TestPoint
- removed TP3: Shift Serial CLK, Connector_Pin:Pin_D1.0mm_L10.0mm, symbol Connector:TestPoint
- removed TP7: RCO, Connector_Pin:Pin_D1.0mm_L10.0mm, symbol Connector:TestPoint
- removed TP8: Raw Gamepad Latch, Connector_Pin:Pin_D1.0mm_L10.0mm, symbol Connector:TestPoint
- removed TP9: Raw Shift out reg CLK, Connector_Pin:Pin_D1.0mm_L10.0mm, symbol Connector:TestPoint
- removed U14: 74HC00, Package_DIP:DIP-14_W7.62mm_Socket, symbol 74xx:74HC00
- removed U2: 74HC161, Package_DIP:DIP-16_W7.62mm_Socket, symbol sixteen-bit-computer:74HC161
- added R10, R7, R8: 10K, Resistor_THT:R_Axial_DIN0207_L6.3mm_D2.5mm_P10.16mm_Horizontal, symbol Device:R_US
- added R9: 4K7, Resistor_THT:R_Axial_DIN0207_L6.3mm_D2.5mm_P10.16mm_Horizontal, symbol Device:R_US
- added U2: 74HC123, Package_DIP:DIP-16_W7.62mm_Socket, symbol 74xx:74HC123
- C10, C11: value C -> 30pF
- TP4: value Gamepad CLK -> TC
Connections:
- net BASE CLK: now also J10.6 (Pin_6), J7.4 (Pin_4), J8.6 (Pin_6), J9.4 (Pin_4)
- net GAMEPAD LATCH: now also U2.13 (Q); no longer U7.12
- net GND: now also U7.11, U7.13, U7.9, U2.1 (A), U2.10 (B), U2.6 (Cext), U2.8 (GND), U2.9 (A); no longer C10.2
- net PAD 1 DATA: now also R7.2
- net PAD 2 DATA: now also R8.2
- net VCC: now also R10.2, R7.1, R8.1, R9.2, U2.11 (Clr), U2.16 (VCC), U2.3 (Clr)
- net ~{BASE CLK}: now also U3.11 (SRCLK), U4.11 (SRCLK), U5.11 (SRCLK), U6.11 (SRCLK)
- net at C10.1: now also R9.1, U2.15 (RCext); no longer U7.13
- net at C11.1: now also R10.1, U2.7 (RCext); no longer U7.11
- net TC: now reaches U9.15 (TC)
- net TC: now also TP4.1, U3.12 (RCLK), U4.12 (RCLK), U5.12 (RCLK), U6.12 (RCLK), U2.2 (B)
- removed net GAMEPAD CLK: J10.6 (Pin_6), J7.4 (Pin_4), J8.6 (Pin_6), J9.4 (Pin_4), TP4.1, U7.8
- removed net SHIFT OUT REG CLK: U3.12 (RCLK), U4.12 (RCLK), U5.12 (RCLK), U6.12 (RCLK), U7.10
- removed net SHIFT SERIAL CLK: U3.11 (SRCLK), U4.11 (SRCLK), U5.11 (SRCLK), U6.11 (SRCLK), U7.9, U9.14 (Q0)
- new net: C10.2, U2.14 (Cext)
- no-connect marks 53 -> 54
Other:
- note added: "Pulse Generation"
- moved on the sheet: C17, TP1, TP4, U15E, U7D, U7E, U7F

Commit message: Finishing touches on gamepad.
Parts:
- removed C17: C, Capacitor_THT:C_Disc_D5.0mm_W2.5mm_P5.00mm, symbol Device:C
- removed U15: 74HC00, Package_DIP:DIP-14_W7.62mm_Socket, symbol 74xx:74HC00
- removed U7: 74HC14, Package_DIP:DIP-14_W7.62mm_Socket, symbol 74xx:74HC14
- added U14: 74HC04, Package_DIP:DIP-14_W7.62mm_Socket, symbol 74xx:74HC04
Connections:
- net BASE CLK: now also U14.13
- net GND: now also C10.2, U2.14 (Cext), U14.5, U14.7 (GND); no longer U8.12, U8.13
- net MEMACTIVE_RFM: now also U14.4
- net MEM_ACTIVE: now also U8.13
- net PAD 1 DATA: now also U14.11
- net PAD 2 DATA: now also U14.9
- net RFM_WTM: now also U14.1
- net VCC: now also U14.14 (VCC)
- net ~{BASE CLK}: now also U14.12
- net at U5.14 (SER): now also U14.8
- net at U8.11: now also U14.3
- net at U3.14 (SER): now also U14.10
- net PAD 1 ADDR LED renamed ~{PAD 1 ADDR LED}
- net PAD 2 ADDR LED renamed ~{PAD 2 ADDR LED}
- new net: U14.2, U8.12
- no-connect marks 54 -> 50
Other:
- note removed: "Clock div by 2"
- moved on the sheet: C10, U8D
