File: kicad/projects/ram/ram.kicad_sch (KiCad schematic)
At the start: 40 parts, among them J1 peripheral_addr_bus_connector, J2 peripheral_aux_connector, J3 peripheral_membank_connector, J5 Conn_02x16_Odd_Even, U1 74HC02, U10 74HC30, U11 74HC32, U12 74HC08, U2 74HC08, U3 74HC123, U4 74HC04, U5 74HC245, U6 74HC245, U7 628128_DIP32_SSOP32, U8 628128_DIP32_SSOP32, U9 74HC30

Commit message: First pass of RAM PCB complete
Parts:
- added C14: C, Capacitor_THT:C_Disc_D5.0mm_W2.5mm_P5.00mm, symbol Device:C
- added D1: LED, sixteen-bit-computer:LED_D5.0mm_Horizontal_O3.81mm_Z3.0mm, symbol Device:LED
- added R3: 1K, Resistor_THT:R_Axial_DIN0207_L6.3mm_D2.5mm_P10.16mm_Horizontal, symbol Device:R_US
- added TP5: GND, Connector_Pin:Pin_D1.0mm_L10.0mm, symbol Connector:TestPoint
- added TP6: Data Clk, Connector_Pin:Pin_D1.0mm_L10.0mm, symbol Connector:TestPoint
- RN1, RN2: value R_Network08_US -> 10K
- TP1: value TestPoint -> Long Pulse / RAM ~{WE}; footprint Connector_PinHeader_2.54mm:PinHeader_1x01_P2.54mm_Vertical -> Connector_Pin:Pin_D1.0mm_L10.0mm
- TP2: value TestPoint -> Data Buf Dir; footprint Connector_PinHeader_2.54mm:PinHeader_1x01_P2.54mm_Vertical -> Connector_Pin:Pin_D1.0mm_L10.0mm
- TP3: value TestPoint -> Data Buf ~{OE}; footprint Connector_PinHeader_2.54mm:PinHeader_1x01_P2.54mm_Vertical -> Connector_Pin:Pin_D1.0mm_L10.0mm
- TP4: value TestPoint -> Short Pulse; footprint Connector_PinHeader_2.54mm:PinHeader_1x01_P2.54mm_Vertical -> Connector_Pin:Pin_D1.0mm_L10.0mm
Connections:
- net DATA_CLK: now also TP6.1
- net GND: now also C14.1, D1.1 (K), TP5.1; no longer U11.4, U11.5
- net VCC: now also C14.2
- net at U11.3, U12.2, U12.4: now also U11.4, U11.5
- net at U11.6: now also R3.2
- net RW_BUF_DIR renamed DATA_BUF_DIR
- net RW_BUF_~{OE} renamed DATA_BUF_~{OE}
- new net: D1.2 (A), R3.1
- no-connect marks 13 -> 12
Other:
- moved on the sheet: U11B, U12A, U12B

Commit message: RAM converted to single line rfm wtm.
Connections:
- net ADDRESSED_RFM: now also U12.11; no longer U12.3
- net GND: no longer U12.12, U12.13, U4.1
- net at U11.4, U11.5, U12.4: now also U12.13, U12.3; no longer U11.3, U12.2
- net at U4.2: now also U12.12
- net RFM renamed MEM_ACT
- net WTM renamed RFM_WTM
- net RFM_WTM: now also U4.1
- new net BANK_ADDRESSED: U11.3, U12.2
- no-connect marks 12 -> 10
Other:
- moved on the sheet: C1, C2, D1, J5, R1, R2, R3, RN1, RN2, TP1, TP2, TP3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

Commit message: RAM tech checks complete.
Parts:
- added R4: 10K, Resistor_THT:R_Axial_DIN0207_L6.3mm_D2.5mm_P10.16mm_Horizontal, symbol Device:R_US
- C97, C98, C99: value C_Polarized -> 33uF
Connections:
- net ADDRESSED_RFM: now also U11.10; no longer U4.11
- net DATA_BUF_DIR: now also U11.9; no longer U4.13
- net DATA_BUF_~{OE}: now also U4.10, R4.2; no longer U2.8
- net GND: now also C1.1, C2.1, U2.10, U2.9, U3.14 (Cext), U3.6 (Cext), U4.13; no longer U11.10, U11.9
- net VCC: now also R4.1
- net at U4.12: no longer U2.9
- net at U11.8: now also U4.11
- no-connect marks 10 -> 11
Other:
- moved on the sheet: U11C, U12C, U2C, U4B, U4E, U4F
