File: kicad/projects/video_bank_sel_cursor/video_bank_sel_cursor.kicad_sch (KiCad schematic)
At the start: 28 parts, among them J1 peripheral_addr_bus_connector, J2 peripheral_aux_connector, J3 peripheral_membank_connector, J4 Conn_01x16_Socket, J5 Conn_01x16_Socket, J6 Conn_01x16_Socket, J7 Conn_01x16_Socket, U1 74HC245, U10 74HC10, U11 74HC377, U12 74HC377, U13 74HC04, U14 74HC245, U15 74HC245, U2 74HC245, U3 74HC245, U4 74HC245, U5 74HC245, U6 74HC245, U7 74HC245, U8 74HC245, U9 74HC10

Commit message: Add music planning and some extra work planning video card layouts.
Parts:
- removed J6: Conn_01x16_Socket, Connector_PinSocket_2.54mm:PinSocket_1x16_P2.54mm_Horizontal, symbol Connector:Conn_01x16_Socket
Changed lines of the file:
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@@
 (kicad_sch (version 20230121) (generator eeschema)
   (paper "B")
+  (bus_alias "DATA_BUS" (members "DATA_BUS_00" "DATA_BUS_01" "DATA_BUS_02" "DATA_BUS_03" "DATA_BUS_04" "DATA_BUS_05" "DATA_BUS_06" "DATA_BUS_07" "DATA_BUS_08" "DATA_BUS_09" "DATA_BUS_10" "DATA_BUS_11" "DATA_BUS_12" "DATA_BUS_13" "DATA_BUS_14" "DATA_BUS_15"))
   (bus_alias "ADDR_BUS" (members "ADDR_BUS_00" "ADDR_BUS_01" "ADDR_BUS_02" "ADDR_BUS_03" "ADDR_BUS_04" "ADDR_BUS_05" "ADDR_BUS_06" "ADDR_BUS_07" "ADDR_BUS_08" "ADDR_BUS_09" "ADDR_BUS_10" "ADDR_BUS_11" "ADDR_BUS_12" "ADDR_BUS_13" "ADDR_BUS_14" "ADDR_BUS_15"))
-  (bus_alias "DATA_BUS" (members "DATA_BUS_00" "DATA_BUS_01" "DATA_BUS_02" "DATA_BUS_03" "DATA_BUS_04" "DATA_BUS_05" "DATA_BUS_06" "DATA_BUS_07" "DATA_BUS_08" "DATA_BUS_09" "DATA_BUS_10" "DATA_BUS_11" "DATA_BUS_12" "DATA_BUS_13" "DATA_BUS_14" "DATA_BUS_15"))
   (bus_alias "BANK_BUS" (members "BANK_BUS_00" "BANK_BUS_01" "BANK_BUS_02" "BANK_BUS_03" "BANK_BUS_04" "BANK_BUS_05" "BANK_BUS_06" "BANK_BUS_07" "BANK_BUS_08" "BANK_BUS_09" "BANK_BUS_10" "BANK_BUS_11" "BANK_BUS_12" "BANK_BUS_13" "BANK_BUS_14" "BANK_BUS_15"))
   (junction (at 377.19 33.655) (diameter 0) (color 0 0 0 0)
@@
         )
       )
-    )
-  )
-  (symbol (lib_id "Connector:Conn_01x16_Socket") (at 200.66 207.645 90) (unit 1)
-    (in_bom yes) (on_board yes) (dnp no) (fields_autoplaced)
-    (property "Reference" "J6" (at 201.93 203.2 90)
-      (effects (font (size 1.27 1.27)))
-    )
-    (property "Value" "Conn_01x16_Socket" (at 201.93 205.74 90)
-      (effects (font (size 1.27 1.27)))
-    )
-    (property "Footprint" "Connector_PinSocket_2.54mm:PinSocket_1x16_P2.54mm_Horizontal" (at 200.66 207.645 0)
-      (effects (font (size 1.27 1.27)) hide)
-    )
-    (property "Datasheet" "~" (at 200.66 207.645 0)
-      (effects (font (size 1.27 1.27)) hide)
-    )
-    (pin "1")
-    (pin "10")
-    (pin "11")
-    (pin "12")
-    (pin "13")
-    (pin "14")
-    (pin "15")
-    (pin "16")
-    (pin "2")
-    (pin "3")
-    (pin "4")
-    (pin "5")
-    (pin "6")
-    (pin "7")
-    (pin "8")
-    (pin "9")
-    (instances
-      (project "video_bank_sel_cursor"
-        (path "/0c25b387-1696-4e3f-ab8e-df646088b074"
-          (reference "J6") (unit 1)
-        )
-      )

Commit message: Bit more tweaking and fleshing out of video circuits.
Parts:
- removed U13: 74HC04, Package_DIP:DIP-14_W7.62mm_Socket, symbol 74xx:74HC04
- added C10, C11, C12, C13, C14, C15, C2, C3, C4, C5, C6, C7, C8, C9: C, Capacitor_THT:C_Disc_D5.0mm_W2.5mm_P5.00mm, symbol Device:C
Connections:
- net DATA_BUS_00 is gone; now on net DATA_BUS_0: J1.1 (D_00)
- net DATA_BUS_01 is gone; now on net DATA_BUS_1: J1.2 (D_01)
- net DATA_BUS_02 is gone; now on net DATA_BUS_2: J1.3 (D_02)
- net DATA_BUS_03 is gone; now on net DATA_BUS_3: J1.4 (D_03)
- net DATA_BUS_04 is gone; now on net DATA_BUS_4: J1.5 (D_04)
- net DATA_BUS_05 is gone; now on net DATA_BUS_5: J1.6 (D_05)
- net DATA_BUS_06 is gone; now on net DATA_BUS_6: J1.7 (D_06)
- net DATA_BUS_07 is gone; now on net DATA_BUS_7: J1.8 (D_07)
- net RFM is gone; now on net MEM_ACT: J2.10 (MEM_ACT)
- net WTM is gone; now on net ~{RFM}/WTM: J2.12 (RFM_WTM)
- net DATA_CLK: now also U11.11 (CP), U12.11 (CP)
- net GND: now also U1.10 (GND), U10.7 (GND), U11.10 (GND), U12.10 (GND), U14.10 (GND), U15.10 (GND), U2.10 (GND), U3.10 (GND), U4.10 (GND), U5.10 (GND), U6.10 (GND), U7.10 (GND), U8.10 (GND), U9.7 (GND), C10.1, C11.1, C12.1, C13.1, C14.2, C15.2, C2.1, C3.1, C4.1, C5.1, C6.1, C7.1, C8.1, C9.1
- net VCC: now also U1.20 (VCC), U10.10, U10.11, U10.14 (VCC), U11.20 (VCC), U12.20 (VCC), U14.20 (VCC), U15.20 (VCC), U2.20 (VCC), U3.20 (VCC), U4.20 (VCC), U5.20 (VCC), U6.20 (VCC), U7.20 (VCC), U8.20 (VCC), U9.13, U9.14 (VCC), U9.2, C10.2, C11.2, C12.2, C13.2, C14.1, C15.1, C2.2, C3.2, C4.2, C5.2, C6.2, C7.2, C8.2, C9.2
- net DATA_BUS_7: now reaches U14.11 (B8)
- net DATA_BUS_7: now also U11.18 (D7), U12.18 (D7), U15.11 (B8)
- net DATA_BUS_6: now reaches U14.12 (B7)
- net DATA_BUS_6: now also U11.17 (D6), U12.17 (D6), U15.12 (B7)
- net DATA_BUS_5: now reaches U14.13 (B6)
- net DATA_BUS_5: now also U11.14 (D5), U12.14 (D5), U15.13 (B6)
- net DATA_BUS_4: now reaches U14.14 (B5)
- net DATA_BUS_4: now also U11.13 (D4), U12.13 (D4), U15.14 (B5)
- net DATA_BUS_3: now reaches U14.15 (B4)
- net DATA_BUS_3: now also U11.8 (D3), U12.8 (D3), U15.15 (B4)
- net DATA_BUS_2: now reaches U14.16 (B3)
- net DATA_BUS_2: now also U11.7 (D2), U12.7 (D2), U15.16 (B3)
- net DATA_BUS_1: now reaches U14.17 (B2)
- net DATA_BUS_1: now also U11.4 (D1), U12.4 (D1), U15.17 (B2)
- net DATA_BUS_0: now reaches U14.18 (B1)
- net DATA_BUS_0: now also U11.3 (D0), U12.3 (D0), U15.18 (B1)
- net ~{CURSOR_ROW_RFM}: now reaches U14.19 (~{OE})
- net ~{CURSOR_ROW_RFM}: now also U9.8
- net CURS_ROW_0: now reaches U14.2 (A1)
- net CURS_ROW_0: now also U11.2 (Q0), U2.2 (A1), U6.2 (A1)
- net CURS_ROW_1: now reaches U14.3 (A2)
- net CURS_ROW_1: now also U11.5 (Q1), U2.3 (A2), U6.3 (A2)
- net CURS_ROW_2: now reaches U14.4 (A3)
- net CURS_ROW_2: now also U11.6 (Q2), U2.4 (A3), U6.4 (A3)
- net CURS_ROW_3: now reaches U14.5 (A3)
- net CURS_ROW_3: now also U11.9 (Q3), U2.5 (A3), U6.5 (A3)
- net CURS_ROW_4: now reaches U14.6 (A5)
- net CURS_ROW_4: now also U11.12 (Q4), U2.6 (A5), U6.6 (A5)
- net CURS_ROW_5: now reaches U14.7 (A6)
- net CURS_ROW_5: now also U11.15 (Q5), U2.7 (A6), U6.7 (A6)
- net CURS_ROW_6: now reaches U14.8 (A7)
- net CURS_ROW_6: now also U11.16 (Q6), U2.8 (A7), U6.8 (A7)
- net CURS_ROW_7: now reaches U14.9 (A8)
- net CURS_ROW_7: now also U11.19 (Q7), U2.9 (A8), U6.9 (A8)
- net ~{CURSOR_COL_RFM}: now reaches U15.19 (~{OE})
- net ~{CURSOR_COL_RFM}: now also U10.6
- net CURS_COL_0: now reaches U15.2 (A1)
- net CURS_COL_0: now also U12.2 (Q0), U4.2 (A1), U8.2 (A1)
- net CURS_COL_1: now reaches U15.3 (A2)
- net CURS_COL_1: now also U12.5 (Q1), U4.3 (A2), U8.3 (A2)
- net CURS_COL_2: now reaches U15.4 (A3)
- net CURS_COL_2: now also U12.6 (Q2), U4.4 (A3), U8.4 (A3)
- net CURS_COL_3: now reaches U15.5 (A3)
- net CURS_COL_3: now also U12.9 (Q3), U4.5 (A3), U8.5 (A3)
- net CURS_COL_4: now reaches U15.6 (A5)
- net CURS_COL_4: now also U12.12 (Q4), U4.6 (A5), U8.6 (A5)
- net CURS_COL_5: now reaches U15.7 (A6)
- net CURS_COL_5: now also U12.15 (Q5), U4.7 (A6), U8.7 (A6)
- net CURS_COL_6: now reaches U15.8 (A7)
- net CURS_COL_6: now also U12.16 (Q6), U4.8 (A7), U8.8 (A7)
- net CURS_COL_7: now reaches U15.9 (A8)
- net CURS_COL_7: now also U12.19 (Q7), U4.9 (A8), U8.9 (A8)
- net OUT_B_ROW_7: now reaches U6.11 (B8)
- net OUT_B_ROW_7: now also J7.16 (Pin_16), U5.11 (B8)
- net OUT_B_ROW_6: now reaches U6.12 (B7)
- net OUT_B_ROW_6: now also J7.15 (Pin_15), U5.12 (B7)
- net OUT_B_ROW_5: now reaches U6.13 (B6)
- net OUT_B_ROW_5: now also J7.14 (Pin_14), U5.13 (B6)
- net OUT_B_ROW_4: now reaches U6.14 (B5)
- net OUT_B_ROW_4: now also J7.13 (Pin_13), U5.14 (B5)
- net OUT_B_ROW_3: now reaches U6.15 (B4)
- net OUT_B_ROW_3: now also J7.12 (Pin_12), U5.15 (B4)
- net OUT_B_ROW_2: now reaches U6.16 (B3)
- net OUT_B_ROW_2: now also J7.11 (Pin_11), U5.16 (B3)
- net OUT_B_ROW_1: now reaches U6.17 (B2)
- net OUT_B_ROW_1: now also J7.10 (Pin_10), U5.17 (B2)
- net OUT_B_ROW_0: now reaches U6.18 (B1)
- net OUT_B_ROW_0: now also J7.9 (Pin_9), U5.18 (B1)
- net ~{BANK_SEL}: now reaches U6.19 (~{OE})
- net ~{BANK_SEL}: now also U1.19 (~{OE}), U10.8, U3.19 (~{OE}), U8.19 (~{OE})
- net BANK_SEL: now reaches U5.19 (~{OE})
- net BANK_SEL: now also U10.9, U2.19 (~{OE}), U4.19 (~{OE}), U7.19 (~{OE})
- net EXT_ROW_0: now reaches U5.2 (A1)
- net EXT_ROW_0: now also J4.9 (Pin_9), U1.2 (A1)
- net EXT_ROW_1: now reaches U5.3 (A2)
- net EXT_ROW_1: now also J4.10 (Pin_10), U1.3 (A2)
- net EXT_ROW_2: now reaches U5.4 (A3)
- net EXT_ROW_2: now also J4.11 (Pin_11), U1.4 (A3)
- net EXT_ROW_3: now reaches U5.5 (A3)
- net EXT_ROW_3: now also J4.12 (Pin_12), U1.5 (A3)
- net EXT_ROW_4: now reaches U5.6 (A5)
- net EXT_ROW_4: now also J4.13 (Pin_13), U1.6 (A5)
- net EXT_ROW_5: now reaches U5.7 (A6)
- net EXT_ROW_5: now also J4.14 (Pin_14), U1.7 (A6)
- net EXT_ROW_6: now reaches U5.8 (A7)
- net EXT_ROW_6: now also J4.15 (Pin_15), U1.8 (A7)
- net EXT_ROW_7: now reaches U5.9 (A8)
- net EXT_ROW_7: now also J4.16 (Pin_16), U1.9 (A8)
- net OUT_A_COL_7: now reaches U4.11 (B8)
- net OUT_A_COL_7: now also J5.8 (Pin_8), U3.11 (B8)
- net OUT_A_COL_6: now reaches U4.12 (B7)
- net OUT_A_COL_6: now also J5.7 (Pin_7), U3.12 (B7)
- net OUT_A_COL_5: now reaches U4.13 (B6)
- net OUT_A_COL_5: now also J5.6 (Pin_6), U3.13 (B6)
- net OUT_A_COL_4: now reaches U4.14 (B5)
- net OUT_A_COL_4: now also J5.5 (Pin_5), U3.14 (B5)
- net OUT_A_COL_3: now reaches U4.15 (B4)
- net OUT_A_COL_3: now also J5.4 (Pin_4), U3.15 (B4)
- net OUT_A_COL_2: now reaches U4.16 (B3)
- net OUT_A_COL_2: now also J5.3 (Pin_3), U3.16 (B3)
- net OUT_A_COL_1: now reaches U4.17 (B2)
- net OUT_A_COL_1: now also J5.2 (Pin_2), U3.17 (B2)
- net OUT_A_COL_0: now reaches U4.18 (B1)
- net OUT_A_COL_0: now also J5.1 (Pin_1), U3.18 (B1)
- net CURSOR_COL_ADDRESSED: now reaches U10.3
- net CURSOR_COL_ADDRESSED: now also U9.3
- net MEM_ACT: now reaches U10.4
- net MEM_ACT: now also U10.2, U9.10, U9.4
- net RFM/~{WTM}: now reaches U10.5
- net RFM/~{WTM}: now also U9.11, U9.12
- net CURSOR_ROW_ADDRESSED: now reaches U9.9
- net CURSOR_ROW_ADDRESSED: now also U10.1
- net OUT_A_ROW_7: now reaches U1.11 (B8)
- net OUT_A_ROW_7: now also J5.16 (Pin_16), U2.11 (B8)
- net OUT_A_ROW_6: now reaches U1.12 (B7)
- net OUT_A_ROW_6: now also J5.15 (Pin_15), U2.12 (B7)
- net OUT_A_ROW_5: now reaches U1.13 (B6)
- net OUT_A_ROW_5: now also J5.14 (Pin_14), U2.13 (B6)
- net OUT_A_ROW_4: now reaches U1.14 (B5)
- net OUT_A_ROW_4: now also J5.13 (Pin_13), U2.14 (B5)
- net OUT_A_ROW_3: now reaches U1.15 (B4)
- net OUT_A_ROW_3: now also J5.12 (Pin_12), U2.15 (B4)
- net OUT_A_ROW_2: now reaches U1.16 (B3)
- net OUT_A_ROW_2: now also J5.11 (Pin_11), U2.16 (B3)
- net OUT_A_ROW_1: now reaches U1.17 (B2)
- net OUT_A_ROW_1: now also J5.10 (Pin_10), U2.17 (B2)
- net OUT_A_ROW_0: now reaches U1.18 (B1)
- net OUT_A_ROW_0: now also J5.9 (Pin_9), U2.18 (B1)
- net EXT_COL_0: now reaches U3.2 (A1)
- net EXT_COL_0: now also J4.1 (Pin_1), U7.2 (A1)
- net EXT_COL_1: now reaches U3.3 (A2)
- net EXT_COL_1: now also J4.2 (Pin_2), U7.3 (A2)
- net EXT_COL_2: now reaches U3.4 (A3)
- net EXT_COL_2: now also J4.3 (Pin_3), U7.4 (A3)
- net EXT_COL_3: now reaches U3.5 (A3)
- net EXT_COL_3: now also J4.4 (Pin_4), U7.5 (A3)
- net EXT_COL_4: now reaches U3.6 (A5)
- net EXT_COL_4: now also J4.5 (Pin_5), U7.6 (A5)
- net EXT_COL_5: now reaches U3.7 (A6)
- net EXT_COL_5: now also J4.6 (Pin_6), U7.7 (A6)
- net EXT_COL_6: now reaches U3.8 (A7)
- net EXT_COL_6: now also J4.7 (Pin_7), U7.8 (A7)
- net EXT_COL_7: now reaches U3.9 (A8)
- net EXT_COL_7: now also J4.8 (Pin_8), U7.9 (A8)
- net OUT_B_COL_0: now reaches J7.1 (Pin_1)
- net OUT_B_COL_0: now also U7.18 (B1), U8.18 (B1)
- net OUT_B_COL_1: now reaches J7.2 (Pin_2)
- net OUT_B_COL_1: now also U7.17 (B2), U8.17 (B2)
- net OUT_B_COL_2: now reaches J7.3 (Pin_3)
- net OUT_B_COL_2: now also U7.16 (B3), U8.16 (B3)
- net OUT_B_COL_3: now reaches J7.4 (Pin_4)
- net OUT_B_COL_3: now also U7.15 (B4), U8.15 (B4)
- net OUT_B_COL_4: now reaches J7.5 (Pin_5)
- net OUT_B_COL_4: now also U7.14 (B5), U8.14 (B5)
- net OUT_B_COL_5: now reaches J7.6 (Pin_6)
- net OUT_B_COL_5: now also U7.13 (B6), U8.13 (B6)
- net OUT_B_COL_6: now reaches J7.7 (Pin_7)
- net OUT_B_COL_6: now also U7.12 (B7), U8.12 (B7)
- net OUT_B_COL_7: now reaches J7.8 (Pin_8)
- net OUT_B_COL_7: now also U7.11 (B8), U8.11 (B8)
- net ~{RFM}/WTM: now reaches U9.1
- net ~{RFM}/WTM: now also U10.13, U9.5
- net ~{CURSOR_COL_WTM}: now reaches U9.6
- net ~{CURSOR_COL_WTM}: now also U12.1 (~{E})
- net ~{CURSOR_ROW_WTM}: now reaches U10.12
- net ~{CURSOR_ROW_WTM}: now also U11.1 (~{E})
- net ADDR_BUS_00: no longer names the net of J1.17 (A_00)
- net ADDR_BUS_01: no longer names the net of J1.18 (A_01)
- net ADDR_BUS_02: no longer names the net of J1.19 (A_02)
- net ADDR_BUS_03: no longer names the net of J1.20 (A_03)
- net ADDR_BUS_04: no longer names the net of J1.21 (A_04)
- net ADDR_BUS_05: no longer names the net of J1.22 (A_05)
- net ADDR_BUS_06: no longer names the net of J1.23 (A_06)
- net ADDR_BUS_07: no longer names the net of J1.24 (A_07)
- net ADDR_BUS_08: no longer names the net of J1.25 (A_08)
- net ADDR_BUS_09: no longer names the net of J1.26 (A_09)
- net ADDR_BUS_10: no longer names the net of J1.27 (A_10)
- net ADDR_BUS_11: no longer names the net of J1.28 (A_11)
- net ADDR_BUS_12: no longer names the net of J1.29 (A_12)
- net ADDR_BUS_13: no longer names the net of J1.30 (A_13)
- net ADDR_BUS_14: no longer names the net of J1.31 (A_14)
- net ADDR_BUS_15: no longer names the net of J1.32 (A_15)
- net BANK_BUS_00: no longer names the net of J3.1 (B_00)
- net BANK_BUS_01: no longer names the net of J3.2 (B_01)
- net BANK_BUS_02: no longer names the net of J3.3 (B_02)
- net BANK_BUS_03: no longer names the net of J3.4 (B_03)
- net BANK_BUS_04: no longer names the net of J3.5 (B_04)
- net BANK_BUS_05: no longer names the net of J3.6 (B_05)
- net BANK_BUS_06: no longer names the net of J3.7 (B_06)
- net BANK_BUS_07: no longer names the net of J3.8 (B_07)
- net BANK_BUS_08: no longer names the net of J3.9 (B_08)
- net BANK_BUS_09: no longer names the net of J3.10 (B_09)
- net BANK_BUS_10: no longer names the net of J3.11 (B_10)
- net BANK_BUS_11: no longer names the net of J3.12 (B_11)
- net BANK_BUS_12: no longer names the net of J3.13 (B_12)
- net BANK_BUS_13: no longer names the net of J3.14 (B_13)
- net BANK_BUS_14: no longer names the net of J3.15 (B_14)
- net BANK_BUS_15: no longer names the net of J3.16 (B_15)
- net DATA_BUS_08: no longer names the net of J1.9 (D_08)
- net DATA_BUS_09: no longer names the net of J1.10 (D_09)
- net DATA_BUS_10: no longer names the net of J1.11 (D_10)
- net DATA_BUS_11: no longer names the net of J1.12 (D_11)
- net DATA_BUS_12: no longer names the net of J1.13 (D_12)
- net DATA_BUS_13: no longer names the net of J1.14 (D_13)
- net DATA_BUS_14: no longer names the net of J1.15 (D_14)
- net DATA_BUS_15: no longer names the net of J1.16 (D_15)
- no-connect marks 0 -> 42
Other:
- moved on the sheet: J2, J4, J5, J7, U1, U10A, U10B, U10C, U10D, U11, U12, U14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

Commit message: Adding video aux and some bits and bieces on video boards.
Parts:
- added J6: video_aux, Connector_PinSocket_2.54mm:PinSocket_1x07_P2.54mm_Horizontal, symbol sixteen-bit-computer:video_aux
- added J8: Conn_01x06_Socket, Connector_PinSocket_2.54mm:PinSocket_1x06_P2.54mm_Horizontal, symbol Connector:Conn_01x06_Socket
- added R2, R3: 10K, Resistor_THT:R_Axial_DIN0207_L6.3mm_D2.5mm_P10.16mm_Horizontal, symbol Device:R_US
Connections:
- net BANK_SEL: now also J6.5 (BANK_SEL)
- net CURSOR_COL_ADDRESSED: now also J8.5 (Pin_5), J8.6 (Pin_6), R2.2
- net CURSOR_ROW_ADDRESSED: now also J8.1 (Pin_1), J8.2 (Pin_2), R3.1
- net GND: now also R2.1, R3.2
- no-connect marks 42 -> 50
Other:
- note added: "Cursor column"
- note added: "Cursor row"
- note added: "Out A column"
- note added: "Out A row"
- note added: "Out B column"
- note added: "Out B row"
- note added: "Read and write decode"

Commit message: Start work on video bank sel cursor.
Connections:
- net CURS_COL_0: now also U15.18 (B1); no longer U15.2 (A1)
- net CURS_COL_1: now also U15.16 (B3), U4.4 (A3), U8.4 (A3); no longer U15.3 (A2), U4.3 (A2), U8.3 (A2)
- net CURS_COL_2: now also U15.14 (B5), U4.6 (A5), U8.6 (A5); no longer U15.4 (A3), U4.4 (A3), U8.4 (A3)
- net CURS_COL_3: now also U15.12 (B7), U4.8 (A7), U8.8 (A7); no longer U15.5 (A3), U4.5 (A3), U8.5 (A3)
- net CURS_COL_4: now also U15.11 (B8), U4.9 (A8), U8.9 (A8); no longer U15.6 (A5), U4.6 (A5), U8.6 (A5)
- net CURS_COL_5: now also U15.13 (B6); no longer U15.7 (A6)
- net CURS_COL_6: now also U15.15 (B4), U4.5 (A3), U8.5 (A3); no longer U15.8 (A7), U4.8 (A7), U8.8 (A7)
- net CURS_COL_7: now also U15.17 (B2), U4.3 (A2), U8.3 (A2); no longer U15.9 (A8), U4.9 (A8), U8.9 (A8)
- net CURS_ROW_0: now also U14.18 (B1); no longer U14.2 (A1)
- net CURS_ROW_1: now also U14.16 (B3), U2.4 (A3), U6.4 (A3); no longer U14.3 (A2), U2.3 (A2), U6.3 (A2)
- net CURS_ROW_2: now also U14.14 (B5), U2.6 (A5), U6.6 (A5); no longer U14.4 (A3), U2.4 (A3), U6.4 (A3)
- net CURS_ROW_3: now also U14.12 (B7), U2.8 (A7), U6.8 (A7); no longer U14.5 (A3), U2.5 (A3), U6.5 (A3)
- net CURS_ROW_4: now also U14.11 (B8), U2.9 (A8), U6.9 (A8); no longer U14.6 (A5), U2.6 (A5), U6.6 (A5)
- net CURS_ROW_5: now also U14.13 (B6); no longer U14.7 (A6)
- net CURS_ROW_6: now also U14.15 (B4), U2.5 (A3), U6.5 (A3); no longer U14.8 (A7), U2.8 (A7), U6.8 (A7)
- net CURS_ROW_7: now also U14.17 (B2), U2.3 (A2), U6.3 (A2); no longer U14.9 (A8), U2.9 (A8), U6.9 (A8)
- net DATA_BUS_0: now also U14.2 (A1), U15.2 (A1); no longer U14.18 (B1), U15.18 (B1)
- net DATA_BUS_1: now also U14.4 (A3), U15.4 (A3); no longer U14.17 (B2), U15.17 (B2)
- net DATA_BUS_2: now also U14.6 (A5), U15.6 (A5); no longer U14.16 (B3), U15.16 (B3)
- net DATA_BUS_3: now also U14.8 (A7), U15.8 (A7); no longer U14.15 (B4), U15.15 (B4)
- net DATA_BUS_4: now also U14.9 (A8), U15.9 (A8); no longer U14.14 (B5), U15.14 (B5)
- net DATA_BUS_5: now also U14.7 (A6), U15.7 (A6); no longer U14.13 (B6), U15.13 (B6)
- net DATA_BUS_6: now also U14.5 (A3), U15.5 (A3); no longer U14.12 (B7), U15.12 (B7)
- net DATA_BUS_7: now also U14.3 (A2), U15.3 (A2); no longer U14.11 (B8), U15.11 (B8)
- net OUT_A_COL_1: now also U4.16 (B3); no longer U4.17 (B2)
- net OUT_A_COL_2: now also U4.14 (B5); no longer U4.16 (B3)
- net OUT_A_COL_3: now also U4.12 (B7); no longer U4.15 (B4)
- net OUT_A_COL_4: now also U4.11 (B8); no longer U4.14 (B5)
- net OUT_A_COL_6: now also U4.15 (B4); no longer U4.12 (B7)
- net OUT_A_COL_7: now also U4.17 (B2); no longer U4.11 (B8)
- net OUT_A_ROW_1: now also U2.16 (B3); no longer U2.17 (B2)
- net OUT_A_ROW_2: now also U2.14 (B5); no longer U2.16 (B3)
- net OUT_A_ROW_3: now also U2.12 (B7); no longer U2.15 (B4)
- net OUT_A_ROW_4: now also U2.11 (B8); no longer U2.14 (B5)
- net OUT_A_ROW_6: now also U2.15 (B4); no longer U2.12 (B7)
- net OUT_A_ROW_7: now also U2.17 (B2); no longer U2.11 (B8)
- net OUT_B_COL_1: now also U8.16 (B3); no longer U8.17 (B2)
- net OUT_B_COL_2: now also U8.14 (B5); no longer U8.16 (B3)
- net OUT_B_COL_3: now also U8.12 (B7); no longer U8.15 (B4)
- net OUT_B_COL_4: now also U8.11 (B8); no longer U8.14 (B5)
- net OUT_B_COL_6: now also U8.15 (B4); no longer U8.12 (B7)
- net OUT_B_COL_7: now also U8.17 (B2); no longer U8.11 (B8)
- net OUT_B_ROW_1: now also U6.16 (B3); no longer U6.17 (B2)
- net OUT_B_ROW_2: now also U6.14 (B5); no longer U6.16 (B3)
- net OUT_B_ROW_3: now also U6.12 (B7); no longer U6.15 (B4)
- net OUT_B_ROW_4: now also U6.11 (B8); no longer U6.14 (B5)
- net OUT_B_ROW_6: now also U6.15 (B4); no longer U6.12 (B7)
- net OUT_B_ROW_7: now also U6.17 (B2); no longer U6.11 (B8)
Other:
- moved on the sheet: C10, C11, C12, C13, C2, C3, C4, C5, C6, C7, C8, C9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
