File: kicad/projects/video_shift_status_delay/video_shift_status_delay.kicad_sch (KiCad schematic)
At the start: 54 parts, among them J1 peripheral_addr_bus_connector, J10 ENABLE DELAY, J2 peripheral_aux_connector, J3 peripheral_membank_connector, J4 Conn_01x16_Socket, J5 Conn_01x16_Socket, J6 video_aux, J7 Conn_01x03_Pin, J8 Conn_01x04_Socket, J9 Conn_02x06_Odd_Even, U1 74HC245, U10 74HC377, U11 74HC138, U12 74HC04, U13 74HC10, U14 74HC04, U15 74HC08, U2 74HC245, U3 74HC245, U4 74HC245, U5 74HC245, U6 74HC245, U7 74HC245, U8 74HC245, U9 74HC245

Commit message: I think all the latest set of boards is done...
Parts:
- removed RN1: 10K, Resistor_THT:R_Array_SIP9, symbol Device:R_Network08_US
- added C16: 0.1uF, Capacitor_THT:C_Disc_D5.0mm_W2.5mm_P5.00mm, symbol Device:C
- added U16: 74HC161, Package_DIP:DIP-16_W7.62mm_Socket, symbol sixteen-bit-computer:74HC161
Connections:
- net BANK_SEL: now also U10.15 (Q5); no longer U10.2 (Q0)
- net DATA_BUS_00: now also U9.2 (A1); no longer U10.7 (D2), U9.9 (A8)
- net DATA_BUS_01: now also U9.3 (A2); no longer U10.4 (D1), U9.8 (A7)
- net DATA_BUS_02: now also U9.4 (A3); no longer U10.3 (D0), U9.7 (A6)
- net DATA_BUS_03: now also U10.8 (D3), U9.5 (A4); no longer U9.6 (A5)
- net DATA_BUS_04: now also U10.13 (D4), U9.6 (A5); no longer U9.5 (A3)
- net GND: now also U10.3 (D0), U10.4 (D1), U10.7 (D2), C16.2, U16.3 (P0), U16.4 (P1), U16.5 (P2), U16.6 (P3), U16.8 (GND); no longer U10.13 (D4), U10.14 (D5), U10.8 (D3), U12.3
- net H_BLANK: now also U9.12 (B7); no longer U9.14 (B5)
- net SHIFT_SEL_0: now also U10.9 (Q3), U9.15 (B4); no longer U10.6 (Q2), U9.11 (B8)
- net SHIFT_SEL_1: now also U10.12 (Q4), U9.14 (B5); no longer U10.5 (Q1), U9.12 (B7)
- net VCC: now also C16.1, U16.1 (~{MR}), U16.10 (TE), U16.16 (VCC), U16.7 (PE), U16.9 (~{SPE})
- net V_BLANK: now also U12.3, U9.11 (B8); no longer U9.15 (B4)
- net FRAME_COUNT_2: now reaches U9.16 (B3)
- net FRAME_COUNT_2: now also U16.12 (Q2)
- net FRAME_COUNT_1: now reaches U9.17 (B2)
- net FRAME_COUNT_1: now also U16.13 (Q1)
- net FRAME_COUNT_0: now reaches U9.18 (B1)
- net FRAME_COUNT_0: now also U16.14 (Q0)
- net at U12.4: now also U16.2 (CP)
- net DATA_BUS_05: now reaches J1.6 (D_05)
- net DATA_BUS_05: now also U10.14 (D5), U9.7 (A6)
- net DATA_BUS_06: now reaches J1.7 (D_06)
- net DATA_BUS_06: now also U9.8 (A7)
- net DATA_BUS_07: now reaches J1.8 (D_07)
- net DATA_BUS_07: now also U9.9 (A8)
- no-connect marks 60 -> 56
Other:
- note added: "Frame count"
- moved on the sheet: C10, C11, C13, J10, J7, J8, J9, R4, R7, R8, RN2, U10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
