File: kicad/projects/shift_rot/shift_rot.kicad_sch (KiCad schematic)
At the start: 47 parts, among them J4 Conn_01x03_Pin, J5 Conn_01x16_Socket, J6 Conn_01x02_Socket, J7 Control_signal_backplane, J8 Bus_connection, J9 Aux_connection, U10 74HC08, U11 74HC574, U12 74HC574, U13 74HC138, U14 74HC157, U16 74HC245, U17 74HC245, U18 74HC02, U19 74HC00, U20 74HC377, U21 74HC377, U3 74HC245, U4 74HC245, U5 74HC245, U6 74HC245, U7 74HC245, U8 74HC245, U9 74HC157

Commit message: Schematic mostly done for shift rot.
Parts:
- added C10, C11, C12, C13, C14, C15, C16, C17, C18, C3, C4, C5, C6, C7, C8, C9: C, Capacitor_THT:C_Disc_D5.0mm_W2.5mm_P5.00mm, symbol Device:C
- added R2: 10K, Resistor_THT:R_Axial_DIN0207_L6.3mm_D2.5mm_P10.16mm_Horizontal, symbol Device:R_US
- added RN1, RN2: R_Network08_US, Resistor_THT:R_Array_SIP9, symbol Device:R_Network08_US
Connections:
- net BUS_11: now also U20.7 (D2); no longer U20.13 (D4)
- net BUS_12: now also U20.17 (D6); no longer U20.8 (D3)
- net BUS_13: now also U20.4 (D1); no longer U20.7 (D2)
- net BUS_14: now also U20.18 (D7); no longer U20.4 (D1)
- net BUS_8: now also U20.13 (D4); no longer U20.18 (D7)
- net BUS_9: now also U20.8 (D3); no longer U20.17 (D6)
- net CNTNT_0: now also J5.1 (Pin_1), U17.9 (A8)
- net CNTNT_1: now also J5.2 (Pin_2), U17.8 (A7)
- net CNTNT_10: now also J5.11 (Pin_11), U16.7 (A6)
- net CNTNT_11: now also J5.12 (Pin_12), U16.6 (A5), U20.6 (Q2); no longer U20.12 (Q4)
- net CNTNT_12: now also J5.13 (Pin_13), U16.5 (A4), U20.16 (Q6); no longer U20.9 (Q3)
- net CNTNT_13: now also J5.14 (Pin_14), U16.4 (A3), U20.5 (Q1); no longer U20.6 (Q2)
- net CNTNT_14: now also J5.15 (Pin_15), U16.3 (A2), U20.19 (Q7); no longer U20.5 (Q1)
- net CNTNT_15: now also J5.16 (Pin_16), U16.2 (A1)
- net CNTNT_2: now also J5.3 (Pin_3), U17.7 (A6)
- net CNTNT_3: now also J5.4 (Pin_4), U17.6 (A5)
- net CNTNT_4: now also J5.5 (Pin_5), U17.5 (A4)
- net CNTNT_5: now also J5.6 (Pin_6), U17.4 (A3)
- net CNTNT_6: now also J5.7 (Pin_7), U17.3 (A2)
- net CNTNT_7: now also J5.8 (Pin_8), U17.2 (A1)
- net CNTNT_8: now also J5.9 (Pin_9), U16.9 (A8), U20.12 (Q4); no longer U20.19 (Q7)
- net CNTNT_9: now also J5.10 (Pin_10), U16.8 (A7), U20.9 (Q3); no longer U20.16 (Q6)
- net DATA_CLK: now also U20.11 (CP), U21.11 (CP)
- net GND: now also J4.3 (Pin_3), U10.7 (GND), U11.10 (GND), U12.10 (GND), U13.4 (~{G2A}), U13.5 (~{G2B}), U13.8 (GND), U14.8 (GND), U16.10 (GND), U17.10 (GND), U18.7 (GND), U19.7 (GND), U3.10 (GND), U4.10 (GND), U5.10 (GND), U6.10 (GND), U7.10 (GND), U8.10 (GND), U9.8 (GND), C10.1, C11.1, C12.1, C13.1, C14.1, C15.1, C16.1, C17.1, C18.1, C3.1, C4.1, C5.1, C6.1, C7.1, C8.1, C9.1, RN1.1 (common), RN2.1 (common)
- net VCC: now also J4.1 (Pin_1), U10.14 (VCC), U11.20 (VCC), U12.20 (VCC), U13.16 (VCC), U13.6 (G1), U14.16 (VCC), U16.1 (DIR), U16.20 (VCC), U17.1 (DIR), U17.20 (VCC), U18.14 (VCC), U19.10, U19.12, U19.13, U19.14 (VCC), U19.4, U19.5, U19.9, U3.20 (VCC), U4.20 (VCC), U5.20 (VCC), U6.20 (VCC), U7.20 (VCC), U8.20 (VCC), U9.16 (VCC), C10.2, C11.2, C12.2, C13.2, C14.2, C15.2, C16.2, C17.2, C18.2, C3.2, C4.2, C5.2, C6.2, C7.2, C8.2, C9.2, R2.1
- net at D12.1 (K): now also RN2.5 (R4)
- net at D12.2 (A): now also U16.14 (B5)
- net SFT_0: now reaches J7.30 (SFT0)
- net SFT_0: now also U13.1 (A)
- net SFT_1: now reaches J7.31 (SFT1)
- net SFT_1: now also U13.2 (B)
- net SFT_2: now reaches J7.32 (SFT2)
- net SFT_2: now also U13.3 (C)
- net at D3.1 (K): now also RN1.4 (R3)
- net at D3.2 (A): now also U17.13 (B6)
- net SAFE_POPPED_CLK: now reaches U11.11 (Cp), U12.11 (Cp), U18.1
- net at U17.11 (B8): now also D1.2 (A)
- net at U17.12 (B7): now also D2.2 (A)
- net at U17.14 (B5): now also D4.2 (A)
- net at U17.15 (B4): now also D5.2 (A)
- net at U17.16 (B3): now also D6.2 (A)
- net at U17.17 (B2): now also D7.2 (A)
- net at U17.18 (B1): now also D8.2 (A)
- net at U17.19 (~{OE}): now also J4.2 (Pin_2), U16.19 (~{OE}), R2.2
- net at D15.1 (K): now also RN2.8 (R7)
- net at D15.2 (A): now also U16.17 (B2)
- net at D8.1 (K): now also RN1.9 (R8)
- net at D2.1 (K): now also RN1.3 (R2)
- net at D6.1 (K): now also RN1.7 (R6)
- net at U16.11 (B8): now also D9.2 (A)
- net at U16.12 (B7): now also D10.2 (A)
- net at U16.13 (B6): now also D11.2 (A)
- net at U16.15 (B4): now also D13.2 (A)
- net at U16.16 (B3): now also D14.2 (A)
- net at U16.18 (B1): now also D16.2 (A)
- net at D10.1 (K): now also RN2.3 (R2)
- net at D9.1 (K): now also RN2.2 (R1)
- net at D16.1 (K): now also RN2.9 (R8)
- net at D4.1 (K): now also RN1.5 (R4)
- net at D5.1 (K): now also RN1.6 (R5)
- net at D14.1 (K): now also RN2.7 (R6)
- net at D13.1 (K): now also RN2.6 (R5)
- net at D1.1 (K): now also RN1.2 (R1)
- net at D7.1 (K): now also RN1.8 (R7)
- net at D11.1 (K): now also RN2.4 (R3)
- no-connect marks 8 -> 40
Other:
- note added: "Control signal decode"
- note added: "LED display"
- note added: "Left shift and rot"
- note added: "Popped bit capture and output"
- note added: "Popped bit selection"
- note added: "Right shift and rot"
- note added: "Rotated/shifted MSB/LSB"
- note added: "Safe clock enable"
- note added: "Straight out"
- note added: "Value to shift"
- moved on the sheet: C1, C2, C97, C98, C99, D1, D10, D11, D12, D13, D14, D15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

Commit message: More PCB work on shift rot
Parts:
- removed TP1: TestPoint, Connector_Pin:Pin_D1.0mm_L10.0mm, symbol Connector:TestPoint
- added R3, R4, R5: 10K, Resistor_THT:R_Axial_DIN0207_L6.3mm_D2.5mm_P10.16mm_Horizontal, symbol Device:R_US
- R1: value R_US -> 10K
Connections:
- net CNTNT_0: now also U14.2 (1A); no longer U14.3 (1B)
- net CNTNT_15: now also U14.3 (1B); no longer U14.2 (1A)
- net GND: now also U14.15 (~{G}); no longer R1.2
- net VCC: now also U3.1 (DIR), U4.1 (DIR), U5.1 (DIR), U6.1 (DIR), U7.1 (DIR), U8.1 (DIR), R3.1, R4.1, R5.1
- net ~{POPPED_BIT_OUT}: now also R5.2
- net ~{STRAIGHT_OUT}: now also R4.2
- net ~{EITHER_LEFT_OR_EITHER_RIGHT} renamed ~{EITHER_LEFT_OR_RIGHT_OUT}
- net ~{EITHER_LEFT} renamed ~{EITHER_RIGHT_OUT}
- net ~{EITHER_RIGHT_OUT}: now also U7.19 (~{OE}), U8.19 (~{OE}), R3.2; no longer U3.19 (~{OE}), U4.19 (~{OE})
- net ~{EITHER_RIGHT} renamed ~{EITHER_LEFT_OUT}
- net ~{EITHER_LEFT_OUT}: now also R1.2, U3.19 (~{OE}), U4.19 (~{OE}); no longer U7.19 (~{OE}), U8.19 (~{OE})
- net ~{EITHER_ROTATE} renamed ~{EITHER_ROTATE_OUT}
Other:
- moved on the sheet: C5, C6, U7, U8

Commit message: Shift rot pretty much done. Final tidy ups on offset preset counter.
Parts:
- C97, C98, C99: value C_Polarized -> 33uF
- RN1, RN2: value R_Network08_US -> 2K
Changed lines of the file:
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@@
       (effects (font (size 1.27 1.27)) (justify left))
     )
-    (property "Value" "C_Polarized" (at 276.225 53.34 0)
+    (property "Value" "33uF" (at 276.225 53.34 0)
       (effects (font (size 1.27 1.27)) (justify left))
     )
@@
       (effects (font (size 1.27 1.27)) (justify left))
     )
-    (property "Value" "C_Polarized" (at 243.84 53.34 0)
+    (property "Value" "33uF" (at 243.84 53.34 0)
       (effects (font (size 1.27 1.27)) (justify left))
     )
@@
       (effects (font (size 1.27 1.27)) (justify left))
     )
-    (property "Value" "C_Polarized" (at 260.35 53.34 0)
+    (property "Value" "33uF" (at 260.35 53.34 0)
       (effects (font (size 1.27 1.27)) (justify left))
     )
@@
       (effects (font (size 1.27 1.27)))
     )
-    (property "Value" "R_Network08_US" (at 373.126 290.83 90)
+    (property "Value" "2K" (at 373.126 290.83 90)
       (effects (font (size 1.27 1.27)))
     )
@@
       (effects (font (size 1.27 1.27)))
     )
-    (property "Value" "R_Network08_US" (at 373.126 346.71 90)
-      (effects (font (size 1.27 1.27)))
-    )
+    (property "Value" "2K" (at 373.126 346.71 90)
+      (effects (font (size 1.27 1.27)))
+    )

Commit message: Shift rot tech checks done
Connections:
- net GND: now also R2.1
- net VCC: no longer R2.1
Changed lines of the file:
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@@
     (fill (type none))
   )
-  (rectangle (start 170.815 394.97) (end 235.585 507.365)
+  (rectangle (start 168.91 394.97) (end 235.585 507.365)
     (stroke (width 0) (type dash))
     (fill (type none))
@@
     (effects (font (size 1.27 1.27)) (justify left bottom))
   )
+  (label "GND" (at 254.635 310.515 0) (fields_autoplaced)
+    (effects (font (size 1.27 1.27)) (justify left bottom))
+  )
   (label "DATA_CLK" (at 197.485 218.44 180) (fields_autoplaced)
     (effects (font (size 1.27 1.27)) (justify right bottom))
@@
     (effects (font (size 1.27 1.27)) (justify right bottom))
   )
-  (label "VCC" (at 254.635 310.515 0) (fields_autoplaced)
-    (effects (font (size 1.27 1.27)) (justify left bottom))
-  )
   (label "BUS_11" (at 226.695 429.26 0) (fields_autoplaced)
