File: kicad/projects/multi_register/multi_register.kicad_pcb (KiCad board)
At the start: 2 copper layers, 203.2 x 97.8 mm, 61 parts, among them J1 Aux_connection, J2 Bus_connection, J3 Control_signal_backplane, J4 Conn_01x03_Pin, U1 74HC574, U10 74HC574, U11 74HC574, U12 74HC574, U13 74HC574, U14 74HC574, U15 74HC238, U16 74HC238, U17 74HC245, U18 74HC245, U19 74HC27, U2 74HC574, U3 74HC574, U4 74HC574, U5 74HC574, U6 74HC574, U7 74HC574, U8 74HC574, U9 74HC574

Commit message: Schematic mostly done for multi reg
Parts:
- added C20: C, Capacitor_THT:C_Disc_D5.0mm_W2.5mm_P5.00mm, F.Cu at (190.5, 104.1)
- added C21: C, Capacitor_THT:C_Disc_D5.0mm_W2.5mm_P5.00mm, F.Cu at (218.4, 116.8)
- added R2: 10K, Resistor_THT:R_Axial_DIN0207_L6.3mm_D2.5mm_P10.16mm_Horizontal, F.Cu at (200.7, 68.6)
- added R3: 10K, Resistor_THT:R_Axial_DIN0207_L6.3mm_D2.5mm_P10.16mm_Horizontal, F.Cu at (210.8, 72.4)
- added R4: 10K, Resistor_THT:R_Axial_DIN0207_L6.3mm_D2.5mm_P10.16mm_Horizontal, F.Cu at (152.4, 68.6)
- added R5: 10K, Resistor_THT:R_Axial_DIN0207_L6.3mm_D2.5mm_P10.16mm_Horizontal, F.Cu at (162.6, 72.4)
- added RN1: R_Network08_US, Resistor_THT:R_Array_SIP9, F.Cu at (190.5, 71.1)
- added RN2: R_Network08_US, Resistor_THT:R_Array_SIP9, F.Cu at (241.3, 71.1)
- added U20: 74HC238, Package_DIP:DIP-16_W7.62mm_Socket, F.Cu at (195.6, 106.7)
- added U21: 74HC00, Package_DIP:DIP-14_W7.62mm_Socket, F.Cu at (223.5, 119.4)
- R1: value R_US -> 10K
- U16: value 74HC238 -> 74HC138
- moved R1 309.9 mm to (248.9, 88.9), turned to -90 degrees
- moved C19 115.1 mm to (190.5, 129.5), turned to 90 degrees
- moved C15 86.2 mm to (190.5, 116.8), turned to 90 degrees
- moved C16 82.8 mm to (218.4, 104.1), turned to 90 degrees
- moved C18 64.9 mm to (205.7, 81.2), turned to 90 degrees
- moved C17 63.6 mm to (165.1, 81.2), turned to 90 degrees
- moved D1 50.8 mm to (200.7, 63.5)
- moved D12 50.8 mm to (226.1, 63.5)
- moved D13 50.8 mm to (219.7, 63.5)
- moved D14 50.8 mm to (213.4, 63.5)
- moved D2 50.8 mm to (194.3, 63.5)
- moved D5 50.8 mm to (175.3, 63.5)
- moved D6 50.8 mm to (168.9, 63.5)
- moved D7 50.8 mm to (162.6, 63.5)
- moved D8 50.8 mm to (251.5, 63.5)
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Connections:
- C15 pad 1: unconnected-(C15-Pad1) -> GND
- C15 pad 2: unconnected-(C15-Pad2) -> VCC
- C16 pad 1: unconnected-(C16-Pad1) -> GND
- C16 pad 2: unconnected-(C16-Pad2) -> VCC
- C17 pad 1: unconnected-(C17-Pad1) -> GND
- C17 pad 2: Net-(U17-VCC) -> VCC
- C18 pad 1: unconnected-(C18-Pad1) -> GND
- C18 pad 2: Net-(U18-VCC) -> VCC
- C19 pad 1: unconnected-(C19-Pad1) -> GND
- C19 pad 2: unconnected-(C19-Pad2) -> VCC
- D1 pad 1: unconnected-(D1-K-Pad1) -> Net-(D1-K)
- D1 pad 2: unconnected-(D1-A-Pad2) -> Net-(D1-A)
- D10 pad 1: unconnected-(D10-K-Pad1) -> Net-(D10-K)
- D10 pad 2: unconnected-(D10-A-Pad2) -> Net-(D10-A)
- D11 pad 1: unconnected-(D11-K-Pad1) -> Net-(D11-K)
- D11 pad 2: unconnected-(D11-A-Pad2) -> Net-(D11-A)
- D12 pad 1: unconnected-(D12-K-Pad1) -> Net-(D12-K)
- D12 pad 2: unconnected-(D12-A-Pad2) -> Net-(D12-A)
- D13 pad 1: unconnected-(D13-K-Pad1) -> Net-(D13-K)
- D13 pad 2: unconnected-(D13-A-Pad2) -> Net-(D13-A)
- D14 pad 1: unconnected-(D14-K-Pad1) -> Net-(D14-K)
- D14 pad 2: unconnected-(D14-A-Pad2) -> Net-(D14-A)
- D2 pad 1: unconnected-(D2-K-Pad1) -> Net-(D2-K)
- D2 pad 2: unconnected-(D2-A-Pad2) -> Net-(D2-A)
- D3 pad 1: unconnected-(D3-K-Pad1) -> Net-(D3-K)
- D3 pad 2: unconnected-(D3-A-Pad2) -> Net-(D3-A)
- D4 pad 1: unconnected-(D4-K-Pad1) -> Net-(D4-K)
- D4 pad 2: unconnected-(D4-A-Pad2) -> Net-(D4-A)
- D5 pad 1: unconnected-(D5-K-Pad1) -> Net-(D5-K)
- D5 pad 2: unconnected-(D5-A-Pad2) -> Net-(D5-A)
- D6 pad 1: unconnected-(D6-K-Pad1) -> Net-(D6-K)
- D6 pad 2: unconnected-(D6-A-Pad2) -> Net-(D6-A)
- D7 pad 1: unconnected-(D7-K-Pad1) -> Net-(D7-K)
- D7 pad 2: unconnected-(D7-A-Pad2) -> Net-(D7-A)
- D8 pad 1: unconnected-(D8-K-Pad1) -> Net-(D8-K)
- D8 pad 2: unconnected-(D8-A-Pad2) -> Net-(D8-A)
- D9 pad 1: unconnected-(D9-K-Pad1) -> Net-(D9-K)
- D9 pad 2: unconnected-(D9-A-Pad2) -> Net-(D9-A)
- J1 pad 6: unconnected-(J1-DATA_CLK-Pad6) -> /DATA_CLK
- J3 pad 3: unconnected-(J3-MR_IN0-Pad3) -> /MR_IN0
- J3 pad 4: unconnected-(J3-MR_IN1-Pad4) -> /MR_IN1
- J3 pad 5: unconnected-(J3-MR_IN2-Pad5) -> /MR_IN2
- J3 pad 6: unconnected-(J3-MR_OUT0-Pad6) -> /MR_OUT0
- J3 pad 7: unconnected-(J3-MR_OUT1-Pad7) -> /MR_OUT1
- J3 pad 8: unconnected-(J3-MR_OUT2-Pad8) -> /MR_OUT2
- J4 pad 1: unconnected-(J4-Pin_1-Pad1) -> VCC
- J4 pad 2: unconnected-(J4-Pin_2-Pad2) -> /LED ~{OE}
- J4 pad 3: unconnected-(J4-Pin_3-Pad3) -> GND
- R1 pad 1: VCC -> /LED ~{OE}
- U1 pad 1: Net-(U1-OE) -> /R0_~{OE}
- U1 pad 11: Net-(U1-Cp) -> /R0_CP
- U10 pad 1: Net-(U10-OE) -> /R4_~{OE}
- U10 pad 11: Net-(U10-Cp) -> /R4_CP
- U11 pad 1: Net-(U11-OE) -> /R5_~{OE}
- U11 pad 11: Net-(U11-Cp) -> /R5_CP
- U12 pad 1: Net-(U11-OE) -> /R5_~{OE}
- U12 pad 11: Net-(U11-Cp) -> /R5_CP
- U13 pad 1: Net-(U13-OE) -> /R6_~{OE}
- U13 pad 11: Net-(U13-Cp) -> /R6_CP
- U14 pad 1: Net-(U13-OE) -> /R6_~{OE}
- U14 pad 11: Net-(U13-Cp) -> /R6_CP
- U15 pad 1: unconnected-(U15-A0-Pad1) -> /MR_IN0
- U15 pad 10: unconnected-(U15-Y5-Pad10) -> /R4_CP
- U15 pad 11: unconnected-(U15-Y4-Pad11) -> /R3_CP
- U15 pad 12: unconnected-(U15-Y3-Pad12) -> /R2_CP
- U15 pad 13: unconnected-(U15-Y2-Pad13) -> /R1_CP
- U15 pad 14: unconnected-(U15-Y1-Pad14) -> /R0_CP
- U15 pad 16: unconnected-(U15-VCC-Pad16) -> VCC
- U15 pad 2: unconnected-(U15-A1-Pad2) -> /MR_IN1
- U15 pad 3: unconnected-(U15-A2-Pad3) -> /MR_IN2
- U15 pad 4: unconnected-(U15-~{E1}-Pad4) -> Net-(U15-~{E1})
- U15 pad 5: unconnected-(U15-~{E2}-Pad5) -> GND
- U15 pad 6: unconnected-(U15-E3-Pad6) -> VCC
- U15 pad 7: unconnected-(U15-Y7-Pad7) -> /R6_CP
- U15 pad 8: unconnected-(U15-GND-Pad8) -> GND
- U15 pad 9: unconnected-(U15-Y6-Pad9) -> /R5_CP
- U16 pad 1: unconnected-(U16-A0-Pad1) -> /MR_OUT0
- U16 pad 10: unconnected-(U16-Y5-Pad10) -> /R4_~{OE}
- U16 pad 11: unconnected-(U16-Y4-Pad11) -> /R3_~{OE}
- U16 pad 12: unconnected-(U16-Y3-Pad12) -> /R2_~{OE}
- U16 pad 13: unconnected-(U16-Y2-Pad13) -> /R1_~{OE}
- U16 pad 14: unconnected-(U16-Y1-Pad14) -> /R0_~{OE}
- U16 pad 16: unconnected-(U16-VCC-Pad16) -> VCC
- U16 pad 2: unconnected-(U16-A1-Pad2) -> /MR_OUT1
- U16 pad 3: unconnected-(U16-A2-Pad3) -> /MR_OUT2
- U16 pad 4: unconnected-(U16-~{E1}-Pad4) -> VCC
- U16 pad 5: unconnected-(U16-~{E2}-Pad5) -> GND
- U16 pad 6: unconnected-(U16-E3-Pad6) -> GND
- U16 pad 7: unconnected-(U16-Y7-Pad7) -> /R6_~{OE}
- U16 pad 8: unconnected-(U16-GND-Pad8) -> GND
- U16 pad 9: unconnected-(U16-Y6-Pad9) -> /R5_~{OE}
- U17 pad 1: unconnected-(U17-DIR-Pad1) -> VCC
- U17 pad 10: unconnected-(U17-GND-Pad10) -> GND
- U17 pad 11: unconnected-(U17-B8-Pad11) -> Net-(D1-A)
- U17 pad 12: unconnected-(U17-B7-Pad12) -> Net-(D2-A)
- U17 pad 13: unconnected-(U17-B6-Pad13) -> Net-(D3-A)
- U17 pad 14: unconnected-(U17-B5-Pad14) -> Net-(D4-A)
- U17 pad 15: unconnected-(U17-B4-Pad15) -> Net-(D5-A)
- U17 pad 16: unconnected-(U17-B3-Pad16) -> Net-(D6-A)
- U17 pad 17: unconnected-(U17-B2-Pad17) -> Net-(D7-A)
- U17 pad 18: unconnected-(U17-B1-Pad18) -> Net-(U17-B1)
- U17 pad 19: unconnected-(U17-~{OE}-Pad19) -> /LED ~{OE}
- U17 pad 2: unconnected-(U17-A1-Pad2) -> Net-(U17-A1)
- U17 pad 20: Net-(U17-VCC) -> VCC
- U17 pad 3: unconnected-(U17-A2-Pad3) -> /R0_IN
- U17 pad 4: unconnected-(U17-A3-Pad4) -> /R1_IN
- U17 pad 5: unconnected-(U17-A4-Pad5) -> /R2_IN
- U17 pad 6: unconnected-(U17-A5-Pad6) -> /R3_IN
- U17 pad 7: unconnected-(U17-A6-Pad7) -> /R4_IN
- U17 pad 8: unconnected-(U17-A7-Pad8) -> /R5_IN
- U17 pad 9: unconnected-(U17-A8-Pad9) -> /R6_IN
- U18 pad 1: unconnected-(U18-DIR-Pad1) -> VCC
- U18 pad 10: unconnected-(U18-GND-Pad10) -> GND
- U18 pad 11: unconnected-(U18-B8-Pad11) -> Net-(D8-K)
- U18 pad 12: unconnected-(U18-B7-Pad12) -> Net-(D9-K)
- U18 pad 13: unconnected-(U18-B6-Pad13) -> Net-(D10-K)
- U18 pad 14: unconnected-(U18-B5-Pad14) -> Net-(D11-K)
- U18 pad 15: unconnected-(U18-B4-Pad15) -> Net-(D12-K)
- U18 pad 16: unconnected-(U18-B3-Pad16) -> Net-(D13-K)
- U18 pad 17: unconnected-(U18-B2-Pad17) -> Net-(D14-K)
- U18 pad 18: unconnected-(U18-B1-Pad18) -> Net-(U18-B1)
- U18 pad 19: unconnected-(U18-~{OE}-Pad19) -> /LED ~{OE}
- U18 pad 2: unconnected-(U18-A1-Pad2) -> Net-(U18-A1)
- U18 pad 20: Net-(U18-VCC) -> VCC
- U18 pad 3: unconnected-(U18-A2-Pad3) -> /R0_~{OE}
- U18 pad 4: unconnected-(U18-A3-Pad4) -> /R1_~{OE}
- U18 pad 5: unconnected-(U18-A4-Pad5) -> /R2_~{OE}
- U18 pad 6: unconnected-(U18-A5-Pad6) -> /R3_~{OE}
- U18 pad 7: unconnected-(U18-A6-Pad7) -> /R4_~{OE}
- U18 pad 8: unconnected-(U18-A7-Pad8) -> /R5_~{OE}
- U18 pad 9: unconnected-(U18-A8-Pad9) -> /R6_~{OE}
- U19 pad 1: unconnected-(U19-Pad1) -> /MR_IN0
- U19 pad 10: unconnected-(U19-Pad10) -> GND
- U19 pad 11: unconnected-(U19-Pad11) -> Net-(U19-Pad11)
- U19 pad 12: unconnected-(U19-Pad12) -> Net-(U19-Pad12)
- U19 pad 13: unconnected-(U19-Pad13) -> /MR_IN2
- U19 pad 14: unconnected-(U19D-VCC-Pad14) -> VCC
- U19 pad 2: unconnected-(U19-Pad2) -> /MR_IN1
- U19 pad 3: unconnected-(U19-Pad3) -> Net-(U19-Pad12)
- U19 pad 4: unconnected-(U19-Pad4) -> GND
- U19 pad 5: unconnected-(U19-Pad5) -> Net-(U19-Pad5)
- U19 pad 6: unconnected-(U19-Pad6) -> Net-(U19-Pad6)
- U19 pad 7: unconnected-(U19D-GND-Pad7) -> GND
- U19 pad 8: unconnected-(U19-Pad8) -> Net-(U19-Pad5)
- U19 pad 9: unconnected-(U19-Pad9) -> Net-(U19-Pad6)
- U2 pad 1: Net-(U1-OE) -> /R0_~{OE}
- U2 pad 11: Net-(U1-Cp) -> /R0_CP
- U3 pad 1: Net-(U3-OE) -> /R1_~{OE}
- U3 pad 11: Net-(U3-Cp) -> /R1_CP
- U4 pad 1: Net-(U3-OE) -> /R1_~{OE}
- U4 pad 11: Net-(U3-Cp) -> /R1_CP
- U5 pad 1: Net-(U5-OE) -> /R2_~{OE}
- U5 pad 11: Net-(U5-Cp) -> /R2_CP
- U6 pad 1: Net-(U5-OE) -> /R2_~{OE}
- U6 pad 11: Net-(U5-Cp) -> /R2_CP
- U7 pad 1: Net-(U7-OE) -> /R3_~{OE}
- U7 pad 11: Net-(U7-Cp) -> /R3_CP
- U8 pad 1: Net-(U7-OE) -> /R3_~{OE}
- U8 pad 11: Net-(U7-Cp) -> /R3_CP
- U9 pad 1: Net-(U10-OE) -> /R4_~{OE}
- U9 pad 11: Net-(U10-Cp) -> /R4_CP

Commit message: Added clock pulse generator
Parts:
- removed TP1: TestPoint, Connector_Pin:Pin_D1.0mm_L10.0mm
- added C22: C, Capacitor_THT:C_Disc_D5.0mm_W2.5mm_P5.00mm, F.Cu at (213.4, 129.5)
- added C23: C, Capacitor_THT:C_Disc_D5.0mm_W2.5mm_P5.00mm, F.Cu at (243.8, 134.7)
- added C24: 0pF, Capacitor_THT:C_Disc_D5.0mm_W2.5mm_P5.00mm, F.Cu at (243.8, 114.3)
- added J5: CLOCK SEL, Connector_PinHeader_2.54mm:PinHeader_1x03_P2.54mm_Horizontal, F.Cu at (241.3, 88.9)
- added J6: CP_DIRECT, Connector_PinHeader_2.54mm:PinHeader_1x02_P2.54mm_Vertical, F.Cu at (-2.11, 109.2)
- added J7: CP_PULSE, Connector_PinHeader_2.54mm:PinHeader_1x02_P2.54mm_Vertical, F.Cu at (233.7, 94.0)
- added R6: 10K, Resistor_THT:R_Axial_DIN0207_L6.3mm_D2.5mm_P10.16mm_Horizontal, F.Cu at (248.9, 114.3)
- added R7: 4.7K, Resistor_THT:R_Axial_DIN0207_L6.3mm_D2.5mm_P10.16mm_Horizontal, F.Cu at (248.9, 129.5)
- added R8: 10K, Resistor_THT:R_Axial_DIN0207_L6.3mm_D2.5mm_P10.16mm_Horizontal, F.Cu at (180.3, 134.6)
- added U22: 74HC123, Package_DIP:DIP-16_W7.62mm_Socket, F.Cu at (218.4, 132.1)
- J4: value Conn_01x03_Pin -> LED EN
- moved R1 10.2 mm to (248.9, 99.1)
- moved C15 5.08 mm to (185.4, 116.8)
- moved C19 5.08 mm to (185.4, 129.5)
- moved C20 5.08 mm to (185.4, 104.1)
- moved U16 5.08 mm to (218.4, 106.7)
- moved U19 5.08 mm to (190.5, 132.1)
- moved U20 5.08 mm to (190.5, 106.7)
- moved U21 5.08 mm to (218.4, 119.4)
- moved C16 5.08 mm to (213.4, 104.1)
- moved C21 5.08 mm to (213.4, 116.8)
- moved U15 5.08 mm to (190.5, 119.4)
Connections:
- U15 pad 4: Net-(U15-~{E1}) -> /CHOSEN_CP
- U21 pad 8: Net-(U15-~{E1}) -> /CP_DIRECT

Commit message: WIP on multi reg PCB
Parts:
- moved J7 26.4 mm to (246.9, 71.1)
- moved C24 25.4 mm to (243.8, 139.7), turned to 90 degrees
- moved C23 20.4 mm to (243.8, 114.3)
Routing:
- net VCC: track 0.00 -> 587.3 mm, vias 0 -> 5
- net (no net): track 149.4 -> 0.00 mm
- net /R6_~{OE}: track 0.00 -> 114.1 mm, vias 0 -> 3
- net /CP_DIRECT: track 0.00 -> 73.0 mm, vias 0 -> 4
- net /MR_OUT0: track 0.00 -> 70.0 mm, vias 0 -> 2
- net /R5_~{OE}: track 0.00 -> 67.7 mm, vias 0 -> 1
- net /MR_OUT1: track 0.00 -> 64.4 mm
- net /R4_~{OE}: track 0.00 -> 64.0 mm, vias 0 -> 1
- net /MR_OUT2: track 0.00 -> 60.4 mm
- net /R3_~{OE}: track 0.00 -> 55.6 mm, vias 0 -> 1
- net /CP_PULSE: track 0.00 -> 52.7 mm, vias 0 -> 2
- net /R2_~{OE}: track 0.00 -> 51.7 mm, vias 0 -> 1
- net /R1_~{OE}: track 0.00 -> 48.6 mm, vias 0 -> 1
- net /R0_~{OE}: track 0.00 -> 45.8 mm, vias 0 -> 1
- net /MR_IN2: track 0.00 -> 43.1 mm, vias 0 -> 1
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
Commit message: Big chunk of PCB layout for multi reg done.
Parts:
- moved J6 249.2 mm to (246.9, 99.1), turned to 90 degrees
- moved C23 25.4 mm to (243.8, 139.7), turned to 90 degrees
- moved R6 25.4 mm to (248.9, 139.7), turned to 90 degrees
- moved C24 25.3 mm to (243.8, 114.4), turned to -90 degrees
- moved R7 15.2 mm to (248.9, 114.3)
- moved R1 8.03 mm to (251.5, 106.7), turned to 180 degrees
- moved RN2 5.24 mm to (236.2, 69.8)
- moved R2 3.81 mm to (200.7, 72.4)
- moved R3 3.81 mm to (210.8, 68.6)
- moved R4 3.81 mm to (152.4, 72.4)
- moved R5 3.81 mm to (162.6, 68.6)
- moved RN1 2.84 mm to (193.0, 69.8)
Routing:
- net /DATA_CLK: track 8.67 -> 195.0 mm, vias 0 -> 3
- net /R4_CP: track 0.00 -> 158.5 mm, vias 0 -> 3
- net /R0_CP: track 0.00 -> 154.9 mm, vias 0 -> 6
- net /R4_~{OE}: track 64.0 -> 217.6 mm, vias 1 -> 5
- net /R0_~{OE}: track 45.8 -> 194.1 mm, vias 1 -> 8
- net /R1_CP: track 0.00 -> 146.2 mm, vias 0 -> 5
- net /R3_~{OE}: track 55.6 -> 198.4 mm, vias 1 -> 6
- net /R3_CP: track 0.00 -> 142.4 mm, vias 0 -> 1
- net /R2_CP: track 0.00 -> 139.9 mm, vias 0 -> 3
- net /R1_~{OE}: track 48.6 -> 186.5 mm, vias 1 -> 8
- net /R2_~{OE}: track 51.7 -> 185.4 mm, vias 1 -> 4
- net VCC: track 587.3 -> 696.2 mm, vias 5 -> 19
- net /BUS_0: track 77.5 -> 184.4 mm, vias 0 -> 3
- net /BUS_1: track 74.9 -> 180.9 mm, vias 0 -> 4
- net /BUS_2: track 72.4 -> 176.5 mm, vias 0 -> 4
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
Commit message: Multi reg complete - still needs tech checks.
Parts:
- removed R2, R3, R4, R5: 10K, Resistor_THT:R_Axial_DIN0207_L6.3mm_D2.5mm_P10.16mm_Horizontal
- added D15: LED, sixteen-bit-computer:LED_D5.0mm_Horizontal_O3.81mm_Z3.0mm, F.Cu at (213.4, 63.5)
- added D16: LED, sixteen-bit-computer:LED_D5.0mm_Horizontal_O3.81mm_Z3.0mm, F.Cu at (207.0, 63.5)
- C23: value C -> 0pF
- moved C98 241.0 mm to (175.3, 127.0), turned to -90 degrees
- moved C99 184.4 mm to (144.8, 81.3), turned to 180 degrees
- moved C97 159.2 mm to (61.0, 134.6), turned to 90 degrees
- moved D8 101.7 mm to (149.8, 63.5)
- moved J7 30.5 mm to (248.9, 101.6)
- moved J6 28.0 mm to (248.9, 71.1)
- moved C17 14.0 mm to (151.1, 81.2)
- moved U17 14.0 mm to (156.2, 83.8)
- moved RN1 10.2 mm to (182.9, 71.1)
- moved C24 7.73 mm to (245.1, 122.0)
- moved R1 6.48 mm to (245.1, 105.4), turned to -90 degrees
- moved D10 6.35 mm to (245.1, 63.5)
- moved D4 6.35 mm to (175.3, 63.5)
- moved D1 6.35 mm to (194.3, 63.5)
- moved D11 6.35 mm to (238.8, 63.5)
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Connections:
- RN1 pad 9: unconnected-(RN1-R8-Pad9) -> Net-(D8-K)
- RN2 pad 2: Net-(D8-A) -> Net-(D9-A)
- RN2 pad 3: Net-(D9-A) -> Net-(D10-A)
- RN2 pad 4: Net-(D10-A) -> Net-(D11-A)
- RN2 pad 5: Net-(D11-A) -> Net-(D12-A)
- RN2 pad 6: Net-(D12-A) -> Net-(D13-A)
- RN2 pad 7: Net-(D13-A) -> Net-(D14-A)
- RN2 pad 8: Net-(D14-A) -> Net-(D15-A)
- RN2 pad 9: unconnected-(RN2-R8-Pad9) -> Net-(D16-A)
- U1 pad 1: /R0_~{OE} -> /R1_~{OE}
- U1 pad 11: /R0_CP -> /R1_CP
- U10 pad 1: /R4_~{OE} -> /R5_~{OE}
- U10 pad 11: /R4_CP -> /R5_CP
- U11 pad 1: /R5_~{OE} -> /R6_~{OE}
- U11 pad 11: /R5_CP -> /R6_CP
- U12 pad 1: /R5_~{OE} -> /R6_~{OE}
- U12 pad 11: /R5_CP -> /R6_CP
- U13 pad 1: /R6_~{OE} -> /R7_~{OE}
- U13 pad 11: /R6_CP -> /R7_CP
- U14 pad 1: /R6_~{OE} -> /R7_~{OE}
- U14 pad 11: /R6_CP -> /R7_CP
- U15 pad 10: /R4_CP -> /R5_CP
- U15 pad 11: /R3_CP -> /R4_CP
- U15 pad 12: /R2_CP -> /R3_CP
- U15 pad 13: /R1_CP -> /R2_CP
- U15 pad 14: /R0_CP -> /R1_CP
- U15 pad 7: /R6_CP -> /R7_CP
- U15 pad 9: /R5_CP -> /R6_CP
- U16 pad 10: /R4_~{OE} -> /R5_~{OE}
- U16 pad 11: /R3_~{OE} -> /R4_~{OE}
- U16 pad 12: /R2_~{OE} -> /R3_~{OE}
- U16 pad 13: /R1_~{OE} -> /R2_~{OE}
- U16 pad 14: /R0_~{OE} -> /R1_~{OE}
- U16 pad 15: unconnected-(U16-Y0-Pad15) -> /R0_~{OE}
- U16 pad 7: /R6_~{OE} -> /R7_~{OE}
- U16 pad 9: /R5_~{OE} -> /R6_~{OE}
- U17 pad 18: Net-(U17-B1) -> Net-(D8-A)
- U17 pad 2: Net-(U17-A1) -> /R0_IN
- U17 pad 3: /R0_IN -> /R1_IN
- U17 pad 4: /R1_IN -> /R2_IN
- U17 pad 5: /R2_IN -> /R3_IN
- U17 pad 6: /R3_IN -> /R4_IN
- U17 pad 7: /R4_IN -> /R5_IN
- U17 pad 8: /R5_IN -> /R6_IN
- U17 pad 9: /R6_IN -> /R7_IN
- U18 pad 11: Net-(D8-K) -> Net-(D9-K)
- U18 pad 12: Net-(D9-K) -> Net-(D10-K)
- U18 pad 13: Net-(D10-K) -> Net-(D11-K)
- U18 pad 14: Net-(D11-K) -> Net-(D12-K)
- U18 pad 15: Net-(D12-K) -> Net-(D13-K)
- U18 pad 16: Net-(D13-K) -> Net-(D14-K)
- U18 pad 17: Net-(D14-K) -> Net-(D15-K)
- U18 pad 2: Net-(U18-A1) -> /R0_~{OE}
- U18 pad 3: /R0_~{OE} -> /R1_~{OE}
- U18 pad 4: /R1_~{OE} -> /R2_~{OE}
- U18 pad 5: /R2_~{OE} -> /R3_~{OE}
- U18 pad 6: /R3_~{OE} -> /R4_~{OE}
- U18 pad 7: /R4_~{OE} -> /R5_~{OE}
- U18 pad 8: /R5_~{OE} -> /R6_~{OE}
- U18 pad 9: /R6_~{OE} -> /R7_~{OE}
- U2 pad 1: /R0_~{OE} -> /R1_~{OE}
- U2 pad 11: /R0_CP -> /R1_CP
- U20 pad 10: /R4_IN -> /R5_IN
- U20 pad 11: /R3_IN -> /R4_IN
- U20 pad 12: /R2_IN -> /R3_IN
- U20 pad 13: /R1_IN -> /R2_IN
- U20 pad 14: /R0_IN -> /R1_IN
- U20 pad 15: unconnected-(U20-Y0-Pad15) -> /R0_IN
- U20 pad 7: /R6_IN -> /R7_IN
- U20 pad 9: /R5_IN -> /R6_IN
- U3 pad 1: /R1_~{OE} -> /R2_~{OE}
- U3 pad 11: /R1_CP -> /R2_CP
- U4 pad 1: /R1_~{OE} -> /R2_~{OE}
- U4 pad 11: /R1_CP -> /R2_CP
- U5 pad 1: /R2_~{OE} -> /R3_~{OE}
- U5 pad 11: /R2_CP -> /R3_CP
- U6 pad 1: /R2_~{OE} -> /R3_~{OE}
- U6 pad 11: /R2_CP -> /R3_CP
- U7 pad 1: /R3_~{OE} -> /R4_~{OE}
- U7 pad 11: /R3_CP -> /R4_CP
- U8 pad 1: /R3_~{OE} -> /R4_~{OE}
- U8 pad 11: /R3_CP -> /R4_CP
- U9 pad 1: /R4_~{OE} -> /R5_~{OE}
- U9 pad 11: /R4_CP -> /R5_CP
Routing:
- net VCC: track 696.2 -> 913.7 mm, vias 19 -> 26
- net /R0_~{OE}: track 194.1 -> 17.3 mm, vias 8 -> 1
- net /R7_~{OE}: track 0.00 -> 159.1 mm, vias 0 -> 4
- net /R0_CP: track 154.9 -> 0.00 mm, vias 6 -> 0
- net /R5_CP: track 29.2 -> 161.8 mm
- net /LED ~{OE}: track 0.00 -> 115.0 mm, vias 0 -> 2
- net /R5_~{OE}: track 122.7 -> 220.1 mm, vias 4 -> 6
- net /R7_CP: track 0.00 -> 81.1 mm, vias 0 -> 3
- net /R7_IN: track 0.00 -> 54.1 mm, vias 0 -> 2
- net /R1_IN: track 27.4 -> 58.2 mm, vias 1 -> 2
- net /R2_IN: track 27.4 -> 57.1 mm, vias 1 -> 2
- net /R3_IN: track 27.4 -> 56.0 mm, vias 1 -> 2
- net /R4_IN: track 27.4 -> 54.9 mm, vias 1 -> 2
- net /R5_IN: track 26.6 -> 53.2 mm, vias 1 -> 2
- net /CP_DIRECT: track 76.9 -> 101.1 mm, vias 4 -> 5
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Other:
- board text added: "0"
- board text added: "1"
- board text added: "2"
- board text added: "3"
- board text added: "4"
- board text added: "5"
- board text added: "6"
- board text added: "7"
- board text added: "CP DIR."
- board text added: "CP PUL."
- board text added: "IN"
- board text added: "JLCJLCJLCJLC"
- board text added: "LED OFF"
- board text added: "LED ON"
- board text added: "MULTI REGISTER"
- board text added: "OUT"
- board text added: "v. 1.0"

Commit message: Multi reg tech checks complete
Parts:
- added RN3: 10K, Resistor_THT:R_Array_SIP9, F.Cu at (213.4, 94.0)
- C97, C98, C99: value C_Polarized -> 33uF
- RN1, RN2: value R_Network08_US -> 1K
- moved J7 7.37 mm to (248.9, 109.0), turned to 0 degrees
- moved J6 3.56 mm to (248.9, 74.7)
Connections:
- U15 pad 4: /CHOSEN_CP -> GND
- U15 pad 6: VCC -> /CHOSEN_CP
- U16 pad 4: VCC -> GND
- U16 pad 6: GND -> VCC
- U21 pad 1: VCC -> Net-(U21-Pad1)
- U21 pad 2: VCC -> Net-(U21-Pad1)
- U21 pad 3: unconnected-(U21-Pad3) -> /CP_DIRECT
- U21 pad 8: /CP_DIRECT -> Net-(U21-Pad1)
- U22 pad 1: /CP_DIRECT -> GND
- U22 pad 13: unconnected-(U22A-Q-Pad13) -> /CP_PULSE
- U22 pad 2: VCC -> /CP_DIRECT
- U22 pad 4: /CP_PULSE -> unconnected-(U22A-~{Q}-Pad4)
Routing:
- net Net-(U21-Pad1): track 0.00 -> 21.7 mm
- net GND: track 28.2 -> 46.0 mm
- net VCC: track 913.7 -> 900.6 mm
- net /CP_DIRECT: track 101.1 -> 108.9 mm
- net /CP_PULSE: track 65.6 -> 61.9 mm, vias 2 -> 3
- net /CHOSEN_CP: track 79.3 -> 81.4 mm, vias 3 -> 4
- net /R6_~{OE}: vias 6 -> 5
- net /R5_~{OE}: vias 6 -> 5
- net /R4_~{OE}: vias 6 -> 5
- net /R3_~{OE}: vias 4 -> 3
- net /R2_~{OE}: vias 8 -> 7
- net /R1_~{OE}: vias 8 -> 7
- net /R0_~{OE}: vias 1 -> 0
Other:
- board text added: "CP DIRECT"
- board text added: "CP PULSE"
- board text added: "GND"
- board text added: "LED ~{OE}"
- board text added: "VCC"
- board text removed: "CP DIR."
- board text removed: "CP PUL."
- board text removed: "LED OFF"
- board text removed: "LED ON"
