File: kicad/projects/multi_register/multi_register.kicad_sch (KiCad schematic)
At the start: 61 parts, among them J1 Aux_connection, J2 Bus_connection, J3 Control_signal_backplane, J4 Conn_01x03_Pin, U1 74HC574, U10 74HC574, U11 74HC574, U12 74HC574, U13 74HC574, U14 74HC574, U15 74HC238, U16 74HC238, U17 74HC245, U18 74HC245, U19 74HC27, U2 74HC574, U3 74HC574, U4 74HC574, U5 74HC574, U6 74HC574, U7 74HC574, U8 74HC574, U9 74HC574

Commit message: Continue work on multi reg PCB
Parts:
- removed U16: 74HC238, Package_DIP:DIP-16_W7.62mm_Socket, symbol 74xx:74HC238
- added C20, C21: C, Capacitor_THT:C_Disc_D5.0mm_W2.5mm_P5.00mm, symbol Device:C
- added R2, R3, R4, R5: 10K, symbol Device:R_US
- added RN1, RN2: R_Network08_US, Resistor_THT:R_Array_SIP9, symbol Device:R_Network08_US
- added U16: 74HC138, symbol sixteen-bit-computer:74HC138
- added U20: 74HC238, Package_DIP:DIP-16_W7.62mm_Socket, symbol 74xx:74HC238
- added U21: 74HC00, symbol 74xx:74HC00
Connections:
- net GND: now also C15.1, C16.1, C18.1, U15.5 (~{E2}), U15.8 (GND), U18.10 (GND), U19.10, U19.4, C20.1, R2.1, R3.2, R4.1, R5.2, RN1.1 (common), U16.5 (~{G2B}), U16.6 (G1), U16.8 (GND), U20.4 (~{E1}), U20.5 (~{E2}), U20.8 (GND)
- net VCC: now also C15.2, C16.2, U15.16 (VCC), U15.6 (E3), C20.2, RN2.1 (common), U16.16 (VCC), U16.4 (~{G2A}), U20.16 (VCC), U20.6 (E3)
- net at D5.1 (K): now also RN1.4 (R3)
- net at D5.2 (A): now also U17.13 (B6)
- net MR_IN0: now reaches J3.3 (MR_IN0)
- net MR_IN0: now also U15.1 (A0), U19.1, U20.1 (A0)
- net MR_IN1: now reaches J3.4 (MR_IN1)
- net MR_IN1: now also U15.2 (A1), U19.2, U20.2 (A1)
- net MR_IN2: now reaches J3.5 (MR_IN2)
- net MR_IN2: now also U15.3 (A2), U19.13, U20.3 (A2)
- net MR_OUT0: now reaches J3.6 (MR_OUT0)
- net MR_OUT0: now also U16.1 (A)
- net MR_OUT1: now reaches J3.7 (MR_OUT1)
- net MR_OUT1: now also U16.2 (B)
- net MR_OUT2: now reaches J3.8 (MR_OUT2)
- net MR_OUT2: now also U16.3 (C)
- net R4_CP: now reaches U15.10 (Y5)
- net R3_CP: now reaches U15.11 (Y4)
- net R2_CP: now reaches U15.12 (Y3)
- net R1_CP: now reaches U15.13 (Y2)
- net R0_CP: now reaches U15.14 (Y1)
- net at U15.4 (~{E1}): now also U21.8
- net R6_CP: now reaches U15.7 (Y7)
- net R5_CP: now reaches U15.9 (Y6)
- net at U19.11: now also U21.11
- net at U19.8: now also U19.5
- net at U19.9: now also U19.6, U21.9
- net at D13.1 (K): now also U18.12 (B7)
- net at D13.2 (A): now also RN2.3 (R2)
- net at U17.11 (B8): now also D7.2 (A)
- net at U17.12 (B7): now also D6.2 (A)
- net at U17.14 (B5): now also D4.2 (A)
- net at U17.15 (B4): now also D3.2 (A)
- net at U17.16 (B3): now also D2.2 (A)
- net at U17.17 (B2): now also D1.2 (A)
- net at U17.18 (B1): now also R5.1
- net at U17.2 (A1): now also R4.2
- net R0_IN: now reaches U17.3 (A2)
- net R0_IN: now also U20.14 (Y1)
- net R1_IN: now reaches U17.4 (A3)
- net R1_IN: now also U20.13 (Y2)
- net R2_IN: now reaches U17.5 (A4)
- net R2_IN: now also U20.12 (Y3)
- net R3_IN: now reaches U17.6 (A5)
- net R3_IN: now also U20.11 (Y4)
- net R4_IN: now reaches U17.7 (A6)
- net R4_IN: now also U20.10 (Y5)
- net R5_IN: now reaches U17.8 (A7)
- net R5_IN: now also U20.9 (Y6)
- net R6_IN: now reaches U17.9 (A8)
- net R6_IN: now also U20.7 (Y7)
- net at U19.3: now also U19.12
- net at D3.1 (K): now also RN1.6 (R5)
- net at D14.1 (K): now also U18.11 (B8)
- net at D14.2 (A): now also RN2.2 (R1)
- net at U18.13 (B6): now also D12.1 (K)
- net at U18.14 (B5): now also D11.1 (K)
- net at U18.15 (B4): now also D10.1 (K)
- net at U18.16 (B3): now also D9.1 (K)
- net at U18.17 (B2): now also D8.1 (K)
- net at U18.18 (B1): now also R3.1
- net at U18.2 (A1): now also R2.2
- net R0_~{OE}: now reaches U18.3 (A2)
- net R0_~{OE}: now also U16.14 (Y1)
- net R1_~{OE}: now reaches U18.4 (A3)
- net R1_~{OE}: now also U16.13 (Y2)
- net R2_~{OE}: now reaches U18.5 (A4)
- net R2_~{OE}: now also U16.12 (Y3)
- net R3_~{OE}: now reaches U18.6 (A5)
- net R3_~{OE}: now also U16.11 (Y4)
- net R4_~{OE}: now reaches U18.7 (A6)
- net R4_~{OE}: now also U16.10 (Y5)
- net R5_~{OE}: now reaches U18.8 (A7)
- net R5_~{OE}: now also U16.9 (Y6)
- net R6_~{OE}: now reaches U18.9 (A8)
- net R6_~{OE}: now also U16.7 (Y7)
- net DATA_CLK: now reaches J1.6 (DATA_CLK)
- net DATA_CLK: now also U21.10, U21.12, U21.13
- net at D12.2 (A): now also RN2.4 (R3)
- net at D4.1 (K): now also RN1.5 (R4)
- net at D6.1 (K): now also RN1.3 (R2)
- net at D2.1 (K): now also RN1.7 (R6)
- net at D9.2 (A): now also RN2.7 (R6)
- net at D7.1 (K): now also RN1.2 (R1)
- net at D1.1 (K): now also RN1.8 (R7)
- net at D10.2 (A): now also RN2.6 (R5)
- net at D8.2 (A): now also RN2.8 (R7)
- net at D11.2 (A): now also RN2.5 (R4)
- no-connect marks 2 -> 7
Other:
- note added: "Safe clock enable"
- moved on the sheet: C15, C16, C17, C18, C19, D1, D10, D11, D12, D13, D14, D2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

Commit message: Schematic mostly done for multi reg
Parts:
- R1: value R_US -> 10K
- R2, R3, R4, R5: footprint (none) -> Resistor_THT:R_Axial_DIN0207_L6.3mm_D2.5mm_P10.16mm_Horizontal
- U16: footprint (none) -> Package_DIP:DIP-16_W7.62mm_Socket
- U21: footprint (none) -> Package_DIP:DIP-14_W7.62mm_Socket
Connections:
- net GND: now also C17.1, C19.1, C21.1, J4.3 (Pin_3), U17.10 (GND), U19.7 (GND), U21.7 (GND)
- net R0_CP: now also U1.11 (Cp), U2.11 (Cp)
- net R0_~{OE}: now also U1.1 (OE), U2.1 (OE)
- net R1_CP: now also U3.11 (Cp), U4.11 (Cp)
- net R1_~{OE}: now also U3.1 (OE), U4.1 (OE)
- net R2_CP: now also U5.11 (Cp), U6.11 (Cp)
- net R2_~{OE}: now also U5.1 (OE), U6.1 (OE)
- net R3_CP: now also U7.11 (Cp), U8.11 (Cp)
- net R3_~{OE}: now also U7.1 (OE), U8.1 (OE)
- net R4_CP: now also U10.11 (Cp), U9.11 (Cp)
- net R4_~{OE}: now also U10.1 (OE), U9.1 (OE)
- net R5_CP: now also U11.11 (Cp), U12.11 (Cp)
- net R5_~{OE}: now also U11.1 (OE), U12.1 (OE)
- net R6_CP: now also U13.11 (Cp), U14.11 (Cp)
- net R6_~{OE}: now also U13.1 (OE), U14.1 (OE)
- net VCC: now also C17.2, C18.2, C19.2, C21.2, J4.1 (Pin_1), U17.1 (DIR), U17.20 (VCC), U18.1 (DIR), U18.20 (VCC), U19.14 (VCC), U21.1, U21.14 (VCC), U21.2, U21.4, U21.5; no longer R1.1
- net at D5.1 (K): now also RN1.6 (R5); no longer RN1.4 (R3)
- net at D5.2 (A): now also U17.15 (B4); no longer U17.13 (B6)
- net at D13.1 (K): now also U18.16 (B3); no longer U18.12 (B7)
- net at D13.2 (A): now also RN2.7 (R6); no longer RN2.3 (R2)
- net at U17.11 (B8): now also D1.2 (A); no longer D7.2 (A)
- net at U17.12 (B7): now also D2.2 (A); no longer D6.2 (A)
- net at D3.2 (A): now also U17.13 (B6); no longer U17.15 (B4)
- net at U17.16 (B3): now also D6.2 (A); no longer D2.2 (A)
- net at U17.17 (B2): now also D7.2 (A); no longer D1.2 (A)
- net LED ~{OE}: now reaches U17.19 (~{OE})
- net LED ~{OE}: now also J4.2 (Pin_2), R1.1, U18.19 (~{OE})
- net at D3.1 (K): now also RN1.4 (R3); no longer RN1.6 (R5)
- net at D14.1 (K): now also U18.17 (B2); no longer U18.11 (B8)
- net at D14.2 (A): now also RN2.8 (R7); no longer RN2.2 (R1)
- net at RN2.4 (R3): now also D10.2 (A); no longer D12.2 (A)
- net at RN2.6 (R5): now also D12.2 (A); no longer D10.2 (A)
- net at D9.2 (A): now also RN2.3 (R2); no longer RN2.7 (R6)
- net at D8.2 (A): now also RN2.2 (R1); no longer RN2.8 (R7)
- net at U18.13 (B6): now also D10.1 (K); no longer D12.1 (K)
- net at U18.15 (B4): now also D12.1 (K); no longer D10.1 (K)
- net at D9.1 (K): now also U18.12 (B7); no longer U18.16 (B3)
- net at D8.1 (K): now also U18.11 (B8); no longer U18.17 (B2)
- net at D6.1 (K): now also RN1.7 (R6); no longer RN1.3 (R2)
- net at D2.1 (K): now also RN1.3 (R2); no longer RN1.7 (R6)
- net at RN1.2 (R1): now also D1.1 (K); no longer D7.1 (K)
- net at RN1.8 (R7): now also D7.1 (K); no longer D1.1 (K)
- no-connect marks 7 -> 35
Other:
- note added: "Input enable decode and display"
- note added: "OE Decode and display"
- moved on the sheet: C17, C19, C21, D1, D10, D11, D12, D13, D14, D2, D3, D4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

Commit message: Added clock pulse generator
Parts:
- removed TP1: TestPoint, Connector_Pin:Pin_D1.0mm_L10.0mm, symbol Connector:TestPoint
- added C22, C23: C, Capacitor_THT:C_Disc_D5.0mm_W2.5mm_P5.00mm, symbol Device:C
- added C24: 0pF, Capacitor_THT:C_Disc_D5.0mm_W2.5mm_P5.00mm, symbol Device:C
- added J5: CLOCK SEL, Connector_PinHeader_2.54mm:PinHeader_1x03_P2.54mm_Horizontal, symbol Connector:Conn_01x03_Pin
- added J6: CP_DIRECT, Connector_PinHeader_2.54mm:PinHeader_1x02_P2.54mm_Vertical, symbol Connector:Conn_01x02_Pin
- added J7: CP_PULSE, Connector_PinHeader_2.54mm:PinHeader_1x02_P2.54mm_Vertical, symbol Connector:Conn_01x02_Pin
- added R6, R8: 10K, Resistor_THT:R_Axial_DIN0207_L6.3mm_D2.5mm_P10.16mm_Horizontal, symbol Device:R_US
- added R7: 4.7K, Resistor_THT:R_Axial_DIN0207_L6.3mm_D2.5mm_P10.16mm_Horizontal, symbol Device:R_US
- added U22: 74HC123, Package_DIP:DIP-16_W7.62mm_Socket, symbol 74xx:74HC123
- J4: value Conn_01x03_Pin -> LED EN
Connections:
- net GND: now also C22.1, C23.1, C24.1, R8.1, U22.10 (B), U22.14 (Cext), U22.6 (Cext), U22.8 (GND), U22.9 (A)
- net VCC: now also C22.2, R6.1, R7.1, U22.11 (Clr), U22.16 (VCC), U22.2 (B), U22.3 (Clr)
- net CHOSEN_CP: now reaches U15.4 (~{E1})
- net CHOSEN_CP: now also J5.2 (Pin_2), R8.2; no longer U21.8
- new net: C24.2, R7.2, U22.15 (RCext)
- new net: C23.2, R6.2, U22.7 (RCext)
- new net CP_DIRECT: J5.1 (Pin_1), J6.1 (Pin_1), J6.2 (Pin_2), U21.8, U22.1 (A)
- new net CP_PULSE: J5.3 (Pin_3), J7.1 (Pin_1), J7.2 (Pin_2), U22.4 (~{Q})
- no-connect marks 35 -> 38
Other:
- note added: "Registers"
- moved on the sheet: C1, C10, C11, C12, C13, C14, C15, C16, C17, C18, C19, C2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

Commit message: Multi reg complete - still needs tech checks.
Parts:
- removed R2, R3, R4, R5: 10K, Resistor_THT:R_Axial_DIN0207_L6.3mm_D2.5mm_P10.16mm_Horizontal, symbol Device:R_US
- added D15, D16: LED, sixteen-bit-computer:LED_D5.0mm_Horizontal_O3.81mm_Z3.0mm, symbol Device:LED
- C23: value C -> 0pF
Connections:
- net R0_CP is gone; now on net R1_CP: U1.11 (Cp), U15.14 (Y1), U2.11 (Cp)
- net R0_IN: now also U17.2 (A1), U20.15 (Y0); no longer U17.3 (A2), U20.14 (Y1)
- net R0_~{OE}: now also U16.15 (Y0), U18.2 (A1); no longer U1.1 (OE), U16.14 (Y1), U18.3 (A2), U2.1 (OE)
- net R1_CP: no longer U15.13 (Y2), U3.11 (Cp), U4.11 (Cp)
- net R1_IN: now also U17.3 (A2), U20.14 (Y1); no longer U17.4 (A3), U20.13 (Y2)
- net R1_~{OE}: now also U1.1 (OE), U16.14 (Y1), U18.3 (A2), U2.1 (OE); no longer U16.13 (Y2), U18.4 (A3), U3.1 (OE), U4.1 (OE)
- net R2_CP: now also U15.13 (Y2), U3.11 (Cp), U4.11 (Cp); no longer U15.12 (Y3), U5.11 (Cp), U6.11 (Cp)
- net R2_IN: now also U17.4 (A3), U20.13 (Y2); no longer U17.5 (A4), U20.12 (Y3)
- net R2_~{OE}: now also U16.13 (Y2), U18.4 (A3), U3.1 (OE), U4.1 (OE); no longer U16.12 (Y3), U18.5 (A4), U5.1 (OE), U6.1 (OE)
- net R3_CP: now also U15.12 (Y3), U5.11 (Cp), U6.11 (Cp); no longer U15.11 (Y4), U7.11 (Cp), U8.11 (Cp)
- net R3_IN: now also U17.5 (A4), U20.12 (Y3); no longer U17.6 (A5), U20.11 (Y4)
- net R3_~{OE}: now also U16.12 (Y3), U18.5 (A4), U5.1 (OE), U6.1 (OE); no longer U16.11 (Y4), U18.6 (A5), U7.1 (OE), U8.1 (OE)
- net R4_CP: now also U15.11 (Y4), U7.11 (Cp), U8.11 (Cp); no longer U10.11 (Cp), U15.10 (Y5), U9.11 (Cp)
- net R4_IN: now also U17.6 (A5), U20.11 (Y4); no longer U17.7 (A6), U20.10 (Y5)
- net R4_~{OE}: now also U16.11 (Y4), U18.6 (A5), U7.1 (OE), U8.1 (OE); no longer U10.1 (OE), U16.10 (Y5), U18.7 (A6), U9.1 (OE)
- net R5_CP: now also U10.11 (Cp), U15.10 (Y5), U9.11 (Cp); no longer U11.11 (Cp), U12.11 (Cp), U15.9 (Y6)
- net R5_IN: now also U17.7 (A6), U20.10 (Y5); no longer U17.8 (A7), U20.9 (Y6)
- net R5_~{OE}: now also U10.1 (OE), U16.10 (Y5), U18.7 (A6), U9.1 (OE); no longer U11.1 (OE), U12.1 (OE), U16.9 (Y6), U18.8 (A7)
- net R6_CP: now also U11.11 (Cp), U12.11 (Cp), U15.9 (Y6); no longer U13.11 (Cp), U14.11 (Cp), U15.7 (Y7)
- net R6_IN: now also U17.8 (A7), U20.9 (Y6); no longer U17.9 (A8), U20.7 (Y7)
- net R6_~{OE}: now also U11.1 (OE), U12.1 (OE), U16.9 (Y6), U18.8 (A7); no longer U13.1 (OE), U14.1 (OE), U16.7 (Y7), U18.9 (A8)
- net at D13.1 (K): now also U18.15 (B4); no longer U18.16 (B3)
- net at D13.2 (A): now also RN2.6 (R5); no longer RN2.7 (R6)
- net at U17.18 (B1): now also D8.2 (A)
- net at D14.1 (K): now also U18.16 (B3); no longer U18.17 (B2)
- net at D14.2 (A): now also RN2.7 (R6); no longer RN2.8 (R7)
- net at RN2.2 (R1): now also D9.2 (A); no longer D8.2 (A)
- net at RN2.3 (R2): now also D10.2 (A); no longer D9.2 (A)
- net at RN2.4 (R3): now also D11.2 (A); no longer D10.2 (A)
- net at RN2.5 (R4): now also D12.2 (A); no longer D11.2 (A)
- net at RN2.9 (R8): now also D16.2 (A)
- net at U18.11 (B8): now also D9.1 (K); no longer D8.1 (K)
- net at U18.12 (B7): now also D10.1 (K); no longer D9.1 (K)
- net at U18.13 (B6): now also D11.1 (K); no longer D10.1 (K)
- net at U18.14 (B5): now also D12.1 (K); no longer D11.1 (K)
- net at U18.18 (B1): now also D16.1 (K)
- net at RN1.9 (R8): now also D8.1 (K)
- new net: D15.2 (A), RN2.8 (R7)
- new net: D15.1 (K), U18.17 (B2)
- new net R7_CP: U13.11 (Cp), U14.11 (Cp), U15.7 (Y7)
- new net R7_IN: U17.9 (A8), U20.7 (Y7)
- new net R7_~{OE}: U13.1 (OE), U14.1 (OE), U16.7 (Y7), U18.9 (A8)
- no-connect marks 38 -> 34
Other:
- moved on the sheet: D10, D11, D12, D13, D14, D8, D9

Commit message: Multi reg tech checks complete
Parts:
- added RN3: 10K, Resistor_THT:R_Array_SIP9, symbol Device:R_Network08_US
- C97, C98, C99: value C_Polarized -> 33uF
- RN1, RN2: value R_Network08_US -> 1K
Connections:
- net CHOSEN_CP: now also U15.6 (E3); no longer U15.4 (~{E1})
- net CP_DIRECT: now also U21.3, U22.2 (B); no longer U21.8, U22.1 (A)
- net CP_PULSE: now also U22.13 (Q); no longer U22.4 (~{Q})
- net GND: now also U15.4 (~{E1}), U16.4 (~{G2A}), U22.1 (A); no longer U16.6 (G1)
- net R0_~{OE}: now also RN3.2 (R1)
- net R1_~{OE}: now also RN3.3 (R2)
- net R2_~{OE}: now also RN3.4 (R3)
- net R3_~{OE}: now also RN3.5 (R4)
- net R4_~{OE}: now also RN3.6 (R5)
- net R5_~{OE}: now also RN3.7 (R6)
- net R6_~{OE}: now also RN3.8 (R7)
- net R7_~{OE}: now also RN3.9 (R8)
- net VCC: now also U16.6 (G1), RN3.1 (common); no longer U15.6 (E3), U16.4 (~{G2A}), U21.1, U21.2, U22.2 (B)
- new net: U21.1, U21.2, U21.8
- no-connect marks 34 -> 33
Other:
- moved on the sheet: C18, D10, D11, D12, D13, D14, D15, D16, D9, J4, J5, J7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
