File: kicad/projects/offest_preset_counter/offset_preset_counter.kicad_sch (KiCad schematic)
At the start: 47 parts, among them J1 Control_signal_backplane, J2 Aux_connection, J3 Conn_01x16_Pin, J4 Conn_01x03_Pin, J5 Conn_01x02_Socket, J6 Conn_01x16_Socket, U1 74HC04, U2 74HC245, U3 74HC161, U4 74HC161, U5 74HC161, U6 74HC161, U7 74HC245, U8 74HC245, U9 74HC245

Commit message: More work on presettable counter with offset PCB.
Parts:
- added C13, C14, C15, C16: 0.1uF, Capacitor_THT:C_Disc_D5.0mm_W2.5mm_P5.00mm, symbol Device:C
- added J10, J12, J14: HIGH, Connector_Wire:SolderWire-0.5sqmm_1x01_D0.9mm_OD2.3mm, symbol Connector:Conn_01x01_Socket
- added J11, J13, J15: LOW, Connector_Wire:SolderWire-0.5sqmm_1x01_D0.9mm_OD2.3mm, symbol Connector:Conn_01x01_Socket
- added J7: CS_0, Connector_Wire:SolderWire-0.5sqmm_1x01_D0.9mm_OD2.3mm, symbol Connector:Conn_01x01_Socket
- added J8: CS_1, Connector_Wire:SolderWire-0.5sqmm_1x01_D0.9mm_OD2.3mm, symbol Connector:Conn_01x01_Socket
- added J9: CS_2, Connector_Wire:SolderWire-0.5sqmm_1x01_D0.9mm_OD2.3mm, symbol Connector:Conn_01x01_Socket
- added U10: 74HC138, Package_DIP:DIP-16_W7.62mm_Socket, symbol sixteen-bit-computer:74HC138
- added U11, U12: 74HC574, Package_DIP:DIP-20_W7.62mm_Socket, symbol sixteen-bit-computer:74HC574
- added U13: 74HC08, Package_DIP:DIP-14_W7.62mm_Socket, symbol sixteen-bit-computer:74HC08
- C10, C11, C12: footprint (none) -> Capacitor_THT:CP_Radial_D6.3mm_P2.50mm
- J1: footprint (none) -> sixteen-bit-computer:backplane-connector-annotated
- J2: footprint (none) -> sixteen-bit-computer:aux-connection
- J3: footprint (none) -> sixteen-bit-computer:bus-connection
- J4: footprint (none) -> Connector_PinHeader_2.54mm:PinHeader_1x03_P2.54mm_Horizontal
- J5: footprint (none) -> Connector_PinSocket_2.54mm:PinSocket_1x02_P2.54mm_Horizontal
- J6: footprint (none) -> Connector_PinSocket_2.54mm:PinSocket_1x16_P2.54mm_Horizontal
- U2, U7, U8, U9: footprint (none) -> Package_DIP:DIP-20_W7.62mm_Socket
- U3, U4, U5, U6: footprint (none) -> Package_DIP:DIP-16_W7.62mm_Socket
Connections:
- net PC_IN is gone; now on net VCC: U1.1
- net CTL_CLK: now also U11.11 (Cp), U12.11 (Cp)
- net CTNT_00: now also U12.2 (D0); no longer J6.16 (Pin_16), U7.9 (A8), U9.11 (B8)
- net CTNT_01: now also U12.3 (D1); no longer J6.15 (Pin_15), U7.8 (A7), U9.12 (B7)
- net CTNT_02: now also U12.4 (D2); no longer J6.14 (Pin_14), U7.7 (A6), U9.13 (B6)
- net CTNT_03: now also U12.5 (D3); no longer J6.13 (Pin_13), U7.6 (A5), U9.14 (B5)
- net CTNT_04: now also U12.6 (D4); no longer J6.12 (Pin_12), U7.5 (A4), U9.15 (B4)
- net CTNT_05: now also U12.7 (D5); no longer J6.11 (Pin_11), U7.4 (A3), U9.16 (B3)
- net CTNT_06: now also U12.8 (D6); no longer J6.10 (Pin_10), U7.3 (A2), U9.17 (B2)
- net CTNT_07: now also U12.9 (D7); no longer J6.9 (Pin_9), U7.2 (A1), U9.18 (B1)
- net CTNT_08: now also U11.2 (D0); no longer J6.8 (Pin_8), U2.11 (B8), U8.9 (A8)
- net CTNT_09: now also U11.3 (D1); no longer J6.7 (Pin_7), U2.12 (B7), U8.8 (A7)
- net CTNT_10: now also U11.4 (D2); no longer J6.6 (Pin_6), U2.13 (B6), U8.7 (A6)
- net CTNT_11: now also U11.5 (D3); no longer J6.5 (Pin_5), U2.14 (B5), U8.6 (A5)
- net CTNT_12: now also U11.6 (D4); no longer J6.4 (Pin_4), U2.15 (B4), U8.5 (A4)
- net CTNT_13: now also U11.7 (D5); no longer J6.3 (Pin_3), U2.16 (B3), U8.4 (A3)
- net CTNT_14: now also U11.8 (D6); no longer J6.2 (Pin_2), U2.17 (B2), U8.3 (A2)
- net CTNT_15: now also U11.9 (D7); no longer J6.1 (Pin_1), U2.18 (B1), U8.2 (A1)
- net GND: now also C13.1, C14.1, C15.1, C16.1, J11.1 (Pin_1), J13.1 (Pin_1), J15.1 (Pin_1), U10.4 (~{G2A}), U10.5 (~{G2B}), U10.8 (GND), U11.1 (OE), U11.10 (GND), U12.1 (OE), U12.10 (GND), U13.7 (GND); no longer U1.11, U1.13, U1.9
- net VCC: now also U1.11, U1.13, U1.9, C13.2, C14.2, C15.2, C16.2, J10.1 (Pin_1), J12.1 (Pin_1), J14.1 (Pin_1), U10.16 (VCC), U10.6 (G1), U11.20 (VCC), U12.20 (VCC), U13.10, U13.14 (VCC), U13.4, U13.5, U13.9
- net PC_COUNT renamed EITHER_COUNT
- net EITHER_COUNT: now also U1.6
- net PC_OUT renamed ~{EITHER_COUNT}
- net ~{EITHER_COUNT}: now also U13.3
- net ~{PC_IN} renamed ~{IN}
- net ~{IN}: now also U10.14 (Y1); no longer U1.2
- net ~{PC_OUT} renamed ~{EITHER_OUT}
- net ~{EITHER_OUT}: now also U13.11; no longer U1.6
- new net CS_0: J7.1 (Pin_1), U10.1 (A)
- new net CS_01: J8.1 (Pin_1), U10.2 (B)
- new net CS_02: J9.1 (Pin_1), U10.3 (C)
- new net CTNT_MOD_00: J6.16 (Pin_16), U12.19 (Q0), U7.9 (A8), U9.11 (B8)
- new net CTNT_MOD_01: J6.15 (Pin_15), U12.18 (Q1), U7.8 (A7), U9.12 (B7)
- new net CTNT_MOD_02: J6.14 (Pin_14), U12.17 (Q2), U7.7 (A6), U9.13 (B6)
- new net CTNT_MOD_03: J6.13 (Pin_13), U12.16 (Q3), U7.6 (A5), U9.14 (B5)
- new net CTNT_MOD_04: J6.12 (Pin_12), U12.15 (Q4), U7.5 (A4), U9.15 (B4)
- new net CTNT_MOD_05: J6.11 (Pin_11), U12.14 (Q5), U7.4 (A3), U9.16 (B3)
- new net CTNT_MOD_06: J6.10 (Pin_10), U12.13 (Q6), U7.3 (A2), U9.17 (B2)
- new net CTNT_MOD_07: J6.9 (Pin_9), U12.12 (Q7), U7.2 (A1), U9.18 (B1)
- new net CTNT_MOD_08: J6.8 (Pin_8), U11.19 (Q0), U2.11 (B8), U8.9 (A8)
- new net CTNT_MOD_09: J6.7 (Pin_7), U11.18 (Q1), U2.12 (B7), U8.8 (A7)
- new net CTNT_MOD_10: J6.6 (Pin_6), U11.17 (Q2), U2.13 (B6), U8.7 (A6)
- new net CTNT_MOD_11: J6.5 (Pin_5), U11.16 (Q3), U2.14 (B5), U8.6 (A5)
- new net CTNT_MOD_12: J6.4 (Pin_4), U11.15 (Q4), U2.15 (B4), U8.5 (A4)
- new net CTNT_MOD_13: J6.3 (Pin_3), U11.14 (Q5), U2.16 (B3), U8.4 (A3)
- new net CTNT_MOD_14: J6.2 (Pin_2), U11.13 (Q6), U2.17 (B2), U8.3 (A2)
- new net CTNT_MOD_15: J6.1 (Pin_1), U11.12 (Q7), U2.18 (B1), U8.2 (A1)
- new net ~{COUNT}: U10.12 (Y3), U13.1
- new net ~{OUT_AND_COUNT}: U10.11 (Y4), U13.13, U13.2
- new net ~{OUT}: U10.13 (Y2), U13.12
- no-connect marks 36 -> 43
Other:
- moved on the sheet: C2, C4, C9, J6, R2, U1A, U1B, U1C, U1D, U1E, U1F, U2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

Commit message: Almost done on counter reg PCB.
Connections:
- net GND: now also J4.3 (Pin_3); no longer J4.1 (Pin_1)
- net VCC: now also J4.1 (Pin_1), U13.12, U13.13; no longer J4.3 (Pin_3), U13.4, U13.5
- net ~{COUNT}: now also U13.4; no longer U13.1
- net ~{EITHER_COUNT}: now also U13.6; no longer U13.3
- net ~{EITHER_OUT}: now also U13.3; no longer U13.11
- net ~{OUT_AND_COUNT}: now also U13.5; no longer U13.13
- net ~{OUT}: now also U13.1; no longer U13.12
Other:
- moved on the sheet: J4, U13A, U13B, U13C, U13D
Changed lines of the file:
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@@
   (junction (at 45.72 210.82) (diameter 0) (color 0 0 0 0)
   )
-  (junction (at 354.33 73.66) (diameter 0) (color 0 0 0 0)
-  )
   (junction (at 222.25 82.55) (diameter 0) (color 0 0 0 0)
   )
   (junction (at 312.42 204.47) (diameter 0) (color 0 0 0 0)
   )
+  (junction (at 354.33 61.595) (diameter 0) (color 0 0 0 0)
+  )
   (junction (at 113.03 90.17) (diameter 0) (color 0 0 0 0)
   )
@@
   (junction (at 196.85 41.91) (diameter 0) (color 0 0 0 0)
   )
+  (junction (at 354.33 73.66) (diameter 0) (color 0 0 0 0)
+  )
   (junction (at 292.1 49.53) (diameter 0) (color 0 0 0 0)
   )
@@
   (junction (at 141.605 154.305) (diameter 0) (color 0 0 0 0)
   )
-  (junction (at 354.33 61.595) (diameter 0) (color 0 0 0 0)
-  )
   (junction (at 344.17 212.09) (diameter 0) (color 0 0 0 0)
   )
@@
     (stroke (width 0) (type default))
   )
-  (wire (pts (xy 128.27 97.79) (xy 175.26 97.79))
+  (wire (pts (xy 354.33 56.515) (xy 354.33 61.595))
     (stroke (width 0) (type default))
   )
-  (wire (pts (xy 163.83 329.565) (xy 166.37 329.565))
+  (wire (pts (xy 128.27 97.79) (xy 175.26 97.79))
     (stroke (width 0) (type default))
   )
-  (wire (pts (xy 354.33 26.035) (xy 354.33 56.515))
+  (wire (pts (xy 163.83 329.565) (xy 166.37 329.565))
     (stroke (width 0) (type default))
   )
@@
     (stroke (width 0) (type default))
   )
-  (wire (pts (xy 354.33 56.515) (xy 354.33 61.595))
+  (wire (pts (xy 354.33 26.035) (xy 354.33 56.515))
     (stroke (width 0) (type default))
   )
@@
     (stroke (width 0) (type default))
   )
+  (wire (pts (xy 354.33 61.595) (xy 354.33 73.66))
+    (stroke (width 0) (type default))
+  )
   (wire (pts (xy 76.2 238.76) (xy 83.82 238.76))
     (stroke (width 0) (type default))
@@
     (stroke (width 0) (type default))
   )
-  (wire (pts (xy 354.33 61.595) (xy 354.33 73.66))
-    (stroke (width 0) (type default))
-  )
   (wire (pts (xy 194.31 223.52) (xy 200.66 223.52))
     (stroke (width 0) (type default))
@@
     (stroke (width 0) (type default))
   )
+  (wire (pts (xy 354.33 73.66) (xy 354.33 78.74))
+    (stroke (width 0) (type default))
+  )
   (wire (pts (xy 165.735 140.335) (xy 165.735 135.255))
     (stroke (width 0) (type default))
@@
     (stroke (width 0) (type default))
   )
-  (wire (pts (xy 354.33 73.66) (xy 354.33 78.74))
-    (stroke (width 0) (type default))
-  )
   (wire (pts (xy 306.07 58.42) (xy 306.07 49.53))
     (stroke (width 0) (type default))
@@
     )
   )
-  (symbol (lib_id "sixteen-bit-computer:74HC08") (at 361.95 59.055 0) (unit 2)
+  (symbol (lib_id "sixteen-bit-computer:74HC08") (at 4.445 87.63 0) (unit 2)
     (in_bom yes) (on_board yes) (dnp no) (fields_autoplaced)
-    (property "Reference" "U13" (at 361.9417 50.8 0)
+    (property "Reference" "U13" (at 4.4367 79.375 0)
       (effects (font (size 1.27 1.27)))
     )
-    (property "Value" "74HC08" (at 361.9417 53.34 0)
+    (property "Value" "74HC08" (at 4.4367 81.915 0)
       (effects (font (size 1.27 1.27)))
     )
-    (property "Footprint" "Package_DIP:DIP-14_W7.62mm_Socket" (at 361.95 59.055 0)
+    (property "Footprint" "Package_DIP:DIP-14_W7.62mm_Socket" (at 4.445 87.63 0)
       (effects (font (size 1.27 1.27)) hide)
     )
-    (property "Datasheet" "https://www.ti.com/lit/ds/symlink/sn74hc08.pdf" (at 361.95 59.055 0)
+    (property "Datasheet" "https://www.ti.com/lit/ds/symlink/sn74hc08.pdf" (at 4.445 87.63 0)
       (effects (font (size 1.27 1.27)) hide)
     )
@@
     )
   )
-  (symbol (lib_id "Connector:Conn_01x03_Pin") (at 365.76 219.71 180) (unit 1)
-    (in_bom yes) (on_board yes) (dnp no) (fields_autoplaced)
-    (property "Reference" "J4" (at 367.03 219.075 0)
+  (symbol (lib_id "Connector:Conn_01x03_Pin") (at 365.76 219.71 0) (mirror y) (unit 1)
+    (in_bom yes) (on_board yes) (dnp no)
+    (property "Reference" "J4" (at 367.03 220.345 0)
       (effects (font (size 1.27 1.27)) (justify right))
     )
-    (property "Value" "Conn_01x03_Pin" (at 367.03 221.615 0)
+    (property "Value" "Conn_01x03_Pin" (at 367.03 217.805 0)
       (effects (font (size 1.27 1.27)) (justify right))
     )
@@
     )
   )
-  (symbol (lib_id "sixteen-bit-computer:74HC08") (at 93.345 137.795 0) (unit 4)
+  (symbol (lib_id "sixteen-bit-computer:74HC08") (at 361.95 76.2 0) (unit 4)
     (in_bom yes) (on_board yes) (dnp no) (fields_autoplaced)
-    (property "Reference" "U13" (at 93.3367 129.54 0)
+    (property "Reference" "U13" (at 361.9417 67.945 0)
       (effects (font (size 1.27 1.27)))
     )
-    (property "Value" "74HC08" (at 93.3367 132.08 0)
+    (property "Value" "74HC08" (at 361.9417 70.485 0)
       (effects (font (size 1.27 1.27)))
     )
-    (property "Footprint" "Package_DIP:DIP-14_W7.62mm_Socket" (at 93.345 137.795 0)
+    (property "Footprint" "Package_DIP:DIP-14_W7.62mm_Socket" (at 361.95 76.2 0)
       (effects (font (size 1.27 1.27)) hide)
     )
-    (property "Datasheet" "https://www.ti.com/lit/ds/symlink/sn74hc08.pdf" (at 93.345 137.795 0)
+    (property "Datasheet" "https://www.ti.com/lit/ds/symlink/sn74hc08.pdf" (at 361.95 76.2 0)
       (effects (font (size 1.27 1.27)) hide)
     )
@@
     )
   )
-  (symbol (lib_id "sixteen-bit-computer:74HC08") (at 361.95 76.2 0) (unit 3)
+  (symbol (lib_id "sixteen-bit-computer:74HC08") (at 361.95 59.055 0) (unit 3)
     (in_bom yes) (on_board yes) (dnp no) (fields_autoplaced)
-    (property "Reference" "U13" (at 361.9417 68.58 0)
+    (property "Reference" "U13" (at 361.9417 51.435 0)
       (effects (font (size 1.27 1.27)))
     )
-    (property "Value" "74HC08" (at 361.9417 71.12 0)
+    (property "Value" "74HC08" (at 361.9417 53.975 0)
       (effects (font (size 1.27 1.27)))
     )
-    (property "Footprint" "Package_DIP:DIP-14_W7.62mm_Socket" (at 361.95 76.2 0)
+    (property "Footprint" "Package_DIP:DIP-14_W7.62mm_Socket" (at 361.95 59.055 0)
       (effects (font (size 1.27 1.27)) hide)
     )
-    (property "Datasheet" "https://www.ti.com/lit/ds/symlink/sn74hc08.pdf" (at 361.95 76.2 0)
+    (property "Datasheet" "https://www.ti.com/lit/ds/symlink/sn74hc08.pdf" (at 361.95 59.055 0)
       (effects (font (size 1.27 1.27)) hide)
     )
@@
     )
   )
-  (symbol (lib_id "sixteen-bit-computer:74HC08") (at 4.445 87.63 0) (unit 1)
+  (symbol (lib_id "sixteen-bit-computer:74HC08") (at 93.345 137.795 0) (unit 1)
     (in_bom yes) (on_board yes) (dnp no) (fields_autoplaced)
-    (property "Reference" "U13" (at 4.4367 79.375 0)
+    (property "Reference" "U13" (at 93.3367 129.54 0)
       (effects (font (size 1.27 1.27)))
     )
-    (property "Value" "74HC08" (at 4.4367 81.915 0)
+    (property "Value" "74HC08" (at 93.3367 132.08 0)
       (effects (font (size 1.27 1.27)))
     )
-    (property "Footprint" "Package_DIP:DIP-14_W7.62mm_Socket" (at 4.445 87.63 0)
+    (property "Footprint" "Package_DIP:DIP-14_W7.62mm_Socket" (at 93.345 137.795 0)
       (effects (font (size 1.27 1.27)) hide)
     )
-    (property "Datasheet" "https://www.ti.com/lit/ds/symlink/sn74hc08.pdf" (at 4.445 87.63 0)
+    (property "Datasheet" "https://www.ti.com/lit/ds/symlink/sn74hc08.pdf" (at 93.345 137.795 0)
       (effects (font (size 1.27 1.27)) hide)
     )

Commit message: Shift rot pretty much done. Final tidy ups on offset preset counter.
Parts:
- C10, C11, C12: value C_Polarized -> 33uF
- RN1, RN2: value 10K -> VAR
Connections:
- net CTNT_MOD_00: now also J6.1 (Pin_1); no longer J6.16 (Pin_16)
- net CTNT_MOD_01: now also J6.2 (Pin_2); no longer J6.15 (Pin_15)
- net CTNT_MOD_02: now also J6.3 (Pin_3); no longer J6.14 (Pin_14)
- net CTNT_MOD_03: now also J6.4 (Pin_4); no longer J6.13 (Pin_13)
- net CTNT_MOD_04: now also J6.5 (Pin_5); no longer J6.12 (Pin_12)
- net CTNT_MOD_05: now also J6.6 (Pin_6); no longer J6.11 (Pin_11)
- net CTNT_MOD_06: now also J6.7 (Pin_7); no longer J6.10 (Pin_10)
- net CTNT_MOD_07: now also J6.8 (Pin_8); no longer J6.9 (Pin_9)
- net CTNT_MOD_08: now also J6.9 (Pin_9); no longer J6.8 (Pin_8)
- net CTNT_MOD_09: now also J6.10 (Pin_10); no longer J6.7 (Pin_7)
- net CTNT_MOD_10: now also J6.11 (Pin_11); no longer J6.6 (Pin_6)
- net CTNT_MOD_11: now also J6.12 (Pin_12); no longer J6.5 (Pin_5)
- net CTNT_MOD_12: now also J6.13 (Pin_13); no longer J6.4 (Pin_4)
- net CTNT_MOD_13: now also J6.14 (Pin_14); no longer J6.3 (Pin_3)
- net CTNT_MOD_14: now also J6.15 (Pin_15); no longer J6.2 (Pin_2)
- net CTNT_MOD_15: now also J6.16 (Pin_16); no longer J6.1 (Pin_1)
Other:
- moved on the sheet: J6
Changed lines of the file:
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@@
       (effects (font (size 1.27 1.27)))
     )
-    (property "Value" "10K" (at 233.68 225.3996 90)
+    (property "Value" "VAR" (at 233.68 225.3996 90)
       (effects (font (size 1.27 1.27)))
     )
@@
       (effects (font (size 1.27 1.27)))
     )
-    (property "Value" "10K" (at 119.38 225.3996 90)
+    (property "Value" "VAR" (at 119.38 225.3996 90)
       (effects (font (size 1.27 1.27)))
     )
@@
       (effects (font (size 1.27 1.27)) (justify left))
     )
-    (property "Value" "C_Polarized" (at 347.345 209.296 0)
+    (property "Value" "33uF" (at 347.345 209.296 0)
       (effects (font (size 1.27 1.27)) (justify left))
     )
@@
     )
   )
-  (symbol (lib_id "Connector:Conn_01x16_Socket") (at 386.08 116.205 90) (unit 1)
-    (in_bom yes) (on_board yes) (dnp no) (fields_autoplaced)
+  (symbol (lib_id "Connector:Conn_01x16_Socket") (at 388.62 116.205 270) (mirror x) (unit 1)
+    (in_bom yes) (on_board yes) (dnp no)
     (property "Reference" "J6" (at 387.35 112.395 90)
       (effects (font (size 1.27 1.27)))
@@
       (effects (font (size 1.27 1.27)))
     )
-    (property "Footprint" "Connector_PinSocket_2.54mm:PinSocket_1x16_P2.54mm_Horizontal" (at 386.08 116.205 0)
-      (effects (font (size 1.27 1.27)) hide)
-    )
-    (property "Datasheet" "~" (at 386.08 116.205 0)
+    (property "Footprint" "Connector_PinSocket_2.54mm:PinSocket_1x16_P2.54mm_Horizontal" (at 388.62 116.205 0)
+      (effects (font (size 1.27 1.27)) hide)
+    )
+    (property "Datasheet" "~" (at 388.62 116.205 0)
       (effects (font (size 1.27 1.27)) hide)
     )
@@
       (effects (font (size 1.27 1.27)) (justify left))
     )
-    (property "Value" "C_Polarized" (at 330.2 209.296 0)
+    (property "Value" "33uF" (at 330.2 209.296 0)
       (effects (font (size 1.27 1.27)) (justify left))
     )
@@
       (effects (font (size 1.27 1.27)) (justify left))
     )
-    (property "Value" "C_Polarized" (at 363.22 209.296 0)
-      (effects (font (size 1.27 1.27)) (justify left))
-    )
+    (property "Value" "33uF" (at 363.22 209.296 0)
+      (effects (font (size 1.27 1.27)) (justify left))
+    )

Commit message: Tech checks and BOMs complete
Parts:
- removed R2: 10K, Resistor_THT:R_Axial_DIN0207_L6.3mm_D2.5mm_P10.16mm_Horizontal, symbol Device:R
- added R2: 10K, Resistor_THT:R_Axial_DIN0207_L6.3mm_D2.5mm_P10.16mm_Horizontal, symbol Device:R_US
Connections:
- net VCC: now also R2.2
- net ~{EITHER_OUT}: now also R2.1
- net LED_CONTROL renamed LED_~{OE}
Other:
- note added: "Content and counter"
- note added: "Content to bus"
- note added: "Ctl sig decode"
- note added: "LED Output"
- note added: "Time offset the content"
- moved on the sheet: C1, C10, C11, C12, C13, C14, C15, C16, C2, C3, C4, C5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
