File: kicad/projects/offest_preset_counter/offset_preset_counter.kicad_pcb (KiCad board)
At the start: 2 copper layers, 203.2 x 97.8 mm, 47 parts, among them J1 Conn_01x16_Female, J2 Control_signal_backplane, J3 Bus_connection, J4 Aux_connection, J5 LED_CONTROL, J6 TOP_POWER, U1 74HC04, U2 74HC245, U3 74HC161, U4 74HC245, U5 74HC161, U6 74HC245, U7 74HC161, U8 74HC245, U9 74HC161

Commit message: More work on presettable counter with offset PCB.
Parts:
- added C13: 0.1uF, Capacitor_THT:C_Disc_D5.0mm_W2.5mm_P5.00mm, F.Cu at (53.3, 96.5)
- added C14: 0.1uF, Capacitor_THT:C_Disc_D5.0mm_W2.5mm_P5.00mm, F.Cu at (124.5, 58.3)
- added C15: 0.1uF, Capacitor_THT:C_Disc_D5.0mm_W2.5mm_P5.00mm, F.Cu at (86.4, 96.4)
- added C16: 0.1uF, Capacitor_THT:C_Disc_D5.0mm_W2.5mm_P5.00mm, F.Cu at (101.6, 71.0)
- added J10: HIGH, Connector_Wire:SolderWire-0.5sqmm_1x01_D0.9mm_OD2.3mm, F.Cu at (248.9, 116.8)
- added J11: LOW, Connector_Wire:SolderWire-0.5sqmm_1x01_D0.9mm_OD2.3mm, F.Cu at (238.8, 121.9)
- added J12: HIGH, Connector_Wire:SolderWire-0.5sqmm_1x01_D0.9mm_OD2.3mm, F.Cu at (248.9, 127.0)
- added J13: LOW, Connector_Wire:SolderWire-0.5sqmm_1x01_D0.9mm_OD2.3mm, F.Cu at (238.8, 116.8)
- added J14: HIGH, Connector_Wire:SolderWire-0.5sqmm_1x01_D0.9mm_OD2.3mm, F.Cu at (248.9, 121.9)
- added J15: LOW, Connector_Wire:SolderWire-0.5sqmm_1x01_D0.9mm_OD2.3mm, F.Cu at (238.8, 127.0)
- added J7: CS_0, Connector_Wire:SolderWire-0.5sqmm_1x01_D0.9mm_OD2.3mm, F.Cu at (243.8, 116.8)
- added J8: CS_1, Connector_Wire:SolderWire-0.5sqmm_1x01_D0.9mm_OD2.3mm, F.Cu at (243.8, 121.9)
- added J9: CS_2, Connector_Wire:SolderWire-0.5sqmm_1x01_D0.9mm_OD2.3mm, F.Cu at (243.8, 127.0)
- added U10: 74HC138, Package_DIP:DIP-16_W7.62mm_Socket, F.Cu at (129.5, 61.0)
- added U11: 74HC574, Package_DIP:DIP-20_W7.62mm_Socket, F.Cu at (91.4, 99.1)
- added U12: 74HC574, Package_DIP:DIP-20_W7.62mm_Socket, F.Cu at (58.4, 99.1)
- added U13: 74HC08, Package_DIP:DIP-14_W7.62mm_Socket, F.Cu at (106.7, 73.7)
- C10, C11, C12: value 33uF -> C_Polarized
- J1: value Conn_01x16_Female -> Control_signal_backplane; footprint Connector_PinSocket_2.54mm:PinSocket_1x16_P2.54mm_Horizontal -> sixteen-bit-computer:backplane-connector-annotated
- J2: value Control_signal_backplane -> Aux_connection; footprint sixteen-bit-computer:backplane-connector-single-row-annotated -> sixteen-bit-computer:aux-connection
- J3: value Bus_connection -> Conn_01x16_Pin
- J4: value Aux_connection -> Conn_01x03_Pin; footprint sixteen-bit-computer:aux-connection -> Connector_PinHeader_2.54mm:PinHeader_1x03_P2.54mm_Horizontal
- J5: value LED_CONTROL -> Conn_01x02_Socket; footprint Connector_PinHeader_2.54mm:PinHeader_1x03_P2.54mm_Horizontal -> Connector_PinSocket_2.54mm:PinSocket_1x02_P2.54mm_Horizontal
- J6: value TOP_POWER -> Conn_01x16_Socket; footprint Connector_PinSocket_2.54mm:PinSocket_1x02_P2.54mm_Horizontal -> Connector_PinSocket_2.54mm:PinSocket_1x16_P2.54mm_Horizontal
- U4, U6: value 74HC245 -> 74HC161; footprint Package_DIP:DIP-20_W7.62mm_Socket -> Package_DIP:DIP-16_W7.62mm_Socket
- U7, U9: value 74HC161 -> 74HC245; footprint Package_DIP:DIP-16_W7.62mm_Socket -> Package_DIP:DIP-20_W7.62mm_Socket
- moved C12 201.2 mm to (-48.2, 89.2), turned to 0 degrees
- moved J1 171.7 mm to (241.3, 144.8)
- moved J4 168.4 mm to (241.3, 78.8), turned to 0 degrees
- moved U6 157.6 mm to (58.4, 125.7)
- moved J2 154.9 mm to (86.4, 144.8)
- moved J5 143.3 mm to (99.1, 61.0), turned to -90 degrees
- moved U9 139.8 mm to (203.2, 125.7)
- moved C11 137.3 mm to (96.5, 33.0), turned to 90 degrees
- moved U7 123.9 mm to (210.8, 86.4)
- moved U4 61.3 mm to (114.3, 125.7)
- moved U2 56.5 mm to (170.2, 125.7)
- moved C10 42.5 mm to (37.1, 165.8)
- moved U5 33.6 mm to (86.4, 125.7)
- moved C4 14.2 mm to (198.1, 118.0)
- moved C9 13.8 mm to (127.0, 71.0)
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Connections:
- D1 pad 2: Net-(D1-Pad2) -> Net-(D1-A)
- D2 pad 2: Net-(D2-Pad2) -> Net-(D2-A)
- D3 pad 2: Net-(D3-Pad2) -> Net-(D3-A)
- D4 pad 2: Net-(D4-Pad2) -> Net-(D4-A)
- D5 pad 2: Net-(D5-Pad2) -> Net-(D5-A)
- D6 pad 2: Net-(D6-Pad2) -> Net-(D6-A)
- D7 pad 2: Net-(D7-Pad2) -> Net-(D7-A)
- D8 pad 2: Net-(D8-Pad2) -> Net-(D8-A)
- J1 pad 1: /CTNT_00 -> unconnected-(J1-ACC_IN-Pad1)
- J1 pad 10: /CTNT_09 -> unconnected-(J1-ALU_ST_FL-Pad10)
- J1 pad 11: /CTNT_10 -> unconnected-(J1-ALU_OUT-Pad11)
- J1 pad 12: /CTNT_11 -> unconnected-(J1-ALU_A_BUS-Pad12)
- J1 pad 13: /CTNT_12 -> unconnected-(J1-ALU_S0-Pad13)
- J1 pad 14: /CTNT_13 -> unconnected-(J1-ALU_S1-Pad14)
- J1 pad 15: /CTNT_14 -> unconnected-(J1-ALU_S2-Pad15)
- J1 pad 16: /CTNT_15 -> unconnected-(J1-ALU_S3-Pad16)
- J1 pad 2: /CTNT_01 -> unconnected-(J1-ACC_OUT-Pad2)
- J1 pad 3: /CTNT_02 -> unconnected-(J1-MR_IN0-Pad3)
- J1 pad 4: /CTNT_03 -> unconnected-(J1-MR_IN1-Pad4)
- J1 pad 5: /CTNT_04 -> unconnected-(J1-MR_IN2-Pad5)
- J1 pad 6: /CTNT_05 -> unconnected-(J1-MR_OUT0-Pad6)
- J1 pad 7: /CTNT_06 -> unconnected-(J1-MR_OUT1-Pad7)
- J1 pad 8: /CTNT_07 -> unconnected-(J1-MR_OUT2-Pad8)
- J1 pad 9: /CTNT_08 -> unconnected-(J1-ALU_ST_RS-Pad9)
- J2 pad 1: Net-(J2-Pad1) -> VCC
- J2 pad 10: Net-(J2-Pad10) -> /RESET
- J2 pad 2: Net-(J2-Pad2) -> VCC
- J2 pad 3: Net-(J2-Pad3) -> GND
- J2 pad 4: Net-(J2-Pad4) -> GND
- J2 pad 5: Net-(J2-Pad5) -> unconnected-(J2-NC-Pad5)
- J2 pad 6: Net-(J2-Pad6) -> /DATA_CLK
- J2 pad 7: Net-(J2-Pad7) -> unconnected-(J2-NC-Pad7)
- J2 pad 8: Net-(J2-Pad8) -> /CTL_CLK
- J2 pad 9: Net-(J2-Pad9) -> unconnected-(J2-NC-Pad9)
- J4 pad 1: VCC -> GND
- J4 pad 2: VCC -> /LED_CONTROL
- J4 pad 3: GND -> VCC
- J5 pad 2: /LED_CONTROL -> GND
- J6 pad 1: VCC -> /CTNT_MOD_15
- J6 pad 2: GND -> /CTNT_MOD_14
- R2 pad 1: /~PC_OUT -> /~{EITHER_OUT}
- U1 pad 1: /PC_IN -> VCC
- U1 pad 10: Net-(U1-Pad10) -> unconnected-(U1-Pad10)
- U1 pad 11: GND -> VCC
- U1 pad 12: Net-(U1-Pad12) -> unconnected-(U1-Pad12)
- U1 pad 13: GND -> VCC
- U1 pad 2: /~PC_IN -> unconnected-(U1-Pad2)
- U1 pad 4: /~RESET -> /~{RESET}
- U1 pad 5: /PC_OUT -> /~{EITHER_COUNT}
- U1 pad 6: /~PC_OUT -> /EITHER_COUNT
- U1 pad 8: Net-(U1-Pad8) -> unconnected-(U1-Pad8)
- U1 pad 9: GND -> VCC
- U2 pad 1: VCC -> GND
- U2 pad 11: Net-(D1-Pad2) -> /CTNT_MOD_08
- U2 pad 12: Net-(D2-Pad2) -> /CTNT_MOD_09
- U2 pad 13: Net-(D3-Pad2) -> /CTNT_MOD_10
- U2 pad 14: Net-(D4-Pad2) -> /CTNT_MOD_11
- U2 pad 15: Net-(D5-Pad2) -> /CTNT_MOD_12
- U2 pad 16: Net-(D6-Pad2) -> /CTNT_MOD_13
- U2 pad 17: Net-(D7-Pad2) -> /CTNT_MOD_14
- U2 pad 18: Net-(D8-Pad2) -> /CTNT_MOD_15
- U2 pad 19: /LED_CONTROL -> /~{EITHER_OUT}
- U2 pad 2: /CTNT_07 -> /BUS_15
- U2 pad 3: /CTNT_06 -> /BUS_14
- U2 pad 4: /CTNT_05 -> /BUS_13
- U2 pad 5: /CTNT_04 -> /BUS_12
- U2 pad 6: /CTNT_03 -> /BUS_11
- U2 pad 7: /CTNT_02 -> /BUS_10
- U2 pad 8: /CTNT_01 -> /BUS_09
- U2 pad 9: /CTNT_00 -> /BUS_08
- U3 pad 1: /~RESET -> /~{RESET}
- U3 pad 15: Net-(U3-Pad15) -> Net-(U3-TC)
- U3 pad 7: /PC_COUNT -> /EITHER_COUNT
- U3 pad 9: /~PC_IN -> /~{IN}
- U4 pad 1: GND -> /~{RESET}
- U4 pad 10: GND -> Net-(U3-TC)
- U4 pad 11: /CTNT_08 -> /CTNT_07
- U4 pad 12: /CTNT_09 -> /CTNT_06
- U4 pad 13: /CTNT_10 -> /CTNT_05
- U4 pad 14: /CTNT_11 -> /CTNT_04
- U4 pad 15: /CTNT_12 -> Net-(U4-TC)
- U4 pad 16: /CTNT_13 -> VCC
- U4 pad 2: /BUS_15 -> /DATA_CLK
- U4 pad 3: /BUS_14 -> /BUS_04
- U4 pad 4: /BUS_13 -> /BUS_05
- U4 pad 5: /BUS_12 -> /BUS_06
- U4 pad 6: /BUS_11 -> /BUS_07
- U4 pad 7: /BUS_10 -> /EITHER_COUNT
- U4 pad 8: /BUS_09 -> GND
- U4 pad 9: /BUS_08 -> /~{IN}
- U5 pad 1: /~RESET -> /~{RESET}
- U5 pad 10: Net-(U3-Pad15) -> Net-(U4-TC)
- U5 pad 11: /CTNT_07 -> /CTNT_11
- U5 pad 12: /CTNT_06 -> /CTNT_10
- U5 pad 13: /CTNT_05 -> /CTNT_09
- U5 pad 14: /CTNT_04 -> /CTNT_08
- U5 pad 15: Net-(U5-Pad15) -> Net-(U5-TC)
- U5 pad 3: /BUS_04 -> /BUS_08
- U5 pad 4: /BUS_05 -> /BUS_09
- U5 pad 5: /BUS_06 -> /BUS_10
- U5 pad 6: /BUS_07 -> /BUS_11
- U5 pad 7: /PC_COUNT -> /EITHER_COUNT
- U5 pad 9: /~PC_IN -> /~{IN}
- U6 pad 1: GND -> /~{RESET}
- U6 pad 10: GND -> Net-(U5-TC)
- U6 pad 11: /CTNT_00 -> /CTNT_15
- U6 pad 12: /CTNT_01 -> /CTNT_14
- U6 pad 13: /CTNT_02 -> /CTNT_13
- U6 pad 14: /CTNT_03 -> /CTNT_12
- U6 pad 15: /CTNT_04 -> unconnected-(U6-TC-Pad15)
- U6 pad 16: /CTNT_05 -> VCC
- U6 pad 2: /BUS_07 -> /DATA_CLK
- U6 pad 3: /BUS_06 -> /BUS_12
- U6 pad 4: /BUS_05 -> /BUS_13
- U6 pad 5: /BUS_04 -> /BUS_14
- U6 pad 6: /BUS_03 -> /BUS_15
- U6 pad 7: /BUS_02 -> /EITHER_COUNT
- U6 pad 8: /BUS_01 -> GND
- U6 pad 9: /BUS_00 -> /~{IN}
- U7 pad 1: /~RESET -> VCC
- U7 pad 10: Net-(U5-Pad15) -> GND
- U7 pad 11: /CTNT_11 -> Net-(D1-A)
- U7 pad 12: /CTNT_10 -> Net-(D2-A)
- U7 pad 13: /CTNT_09 -> Net-(D3-A)
- U7 pad 14: /CTNT_08 -> Net-(D4-A)
- U7 pad 15: Net-(U7-Pad15) -> Net-(D5-A)
- U7 pad 16: VCC -> Net-(D6-A)
- U7 pad 2: /DATA_CLK -> /CTNT_MOD_07
- U7 pad 3: /BUS_08 -> /CTNT_MOD_06
- U7 pad 4: /BUS_09 -> /CTNT_MOD_05
- U7 pad 5: /BUS_10 -> /CTNT_MOD_04
- U7 pad 6: /BUS_11 -> /CTNT_MOD_03
- U7 pad 7: /PC_COUNT -> /CTNT_MOD_02
- U7 pad 8: GND -> /CTNT_MOD_01
- U7 pad 9: /~PC_IN -> /CTNT_MOD_00
- U8 pad 2: /CTNT_15 -> /CTNT_MOD_15
- U8 pad 3: /CTNT_14 -> /CTNT_MOD_14
- U8 pad 4: /CTNT_13 -> /CTNT_MOD_13
- U8 pad 5: /CTNT_12 -> /CTNT_MOD_12
- U8 pad 6: /CTNT_11 -> /CTNT_MOD_11
- U8 pad 7: /CTNT_10 -> /CTNT_MOD_10
- U8 pad 8: /CTNT_09 -> /CTNT_MOD_09
- U8 pad 9: /CTNT_08 -> /CTNT_MOD_08
- U9 pad 1: /~RESET -> GND
- U9 pad 10: Net-(U7-Pad15) -> GND
- U9 pad 11: /CTNT_15 -> /CTNT_MOD_00
- U9 pad 12: /CTNT_14 -> /CTNT_MOD_01
- U9 pad 13: /CTNT_13 -> /CTNT_MOD_02
- U9 pad 14: /CTNT_12 -> /CTNT_MOD_03
- U9 pad 15: Net-(U9-Pad15) -> /CTNT_MOD_04
- U9 pad 16: VCC -> /CTNT_MOD_05
- U9 pad 2: /DATA_CLK -> /BUS_07
- U9 pad 3: /BUS_12 -> /BUS_06
- U9 pad 4: /BUS_13 -> /BUS_05
- U9 pad 5: /BUS_14 -> /BUS_04
- U9 pad 6: /BUS_15 -> /BUS_03
- U9 pad 7: /PC_COUNT -> /BUS_02
- U9 pad 8: GND -> /BUS_01
- U9 pad 9: /~PC_IN -> /BUS_00
Routing:
- net /PC_IN: track 239.1 -> 0.00 mm
- net /PC_OUT: track 223.8 -> 0.00 mm
- net /CTNT_05: track 223.9 -> 4.83 mm, vias 6 -> 0
- net /CTNT_07: track 223.6 -> 4.83 mm, vias 6 -> 0
- net /CTNT_04: track 223.6 -> 4.83 mm, vias 6 -> 0
- net /CTNT_06: track 223.6 -> 4.83 mm, vias 6 -> 0
- net /CTNT_13: track 204.8 -> 5.08 mm, vias 6 -> 0
- net /CTNT_14: track 204.8 -> 5.08 mm, vias 6 -> 0
- net /CTNT_12: track 204.8 -> 5.08 mm, vias 6 -> 0
- net /CTNT_15: track 204.6 -> 5.08 mm, vias 4 -> 0
- net /CTNT_10: track 204.3 -> 5.08 mm, vias 6 -> 0
- net /CTNT_09: track 204.3 -> 5.08 mm, vias 6 -> 0
- net /CTNT_08: track 204.3 -> 5.08 mm, vias 6 -> 0
- net /CTNT_11: track 204.3 -> 5.08 mm, vias 6 -> 0
- net /CTNT_00: track 224.4 -> 43.2 mm, vias 4 -> 0
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Other:
- net class Default removed
- board text added: "LED ~{OE}"
- board text removed: "LED ~OE"
- board text removed: "PROGRAM COUNTER"
- board text removed: "V.2"

Commit message: Almost done on counter reg PCB.
Parts:
- moved R2 83.1 mm to (238.8, 111.5)
- moved C14 12.8 mm to (124.5, 71.1)
- moved C9 12.7 mm to (127.0, 58.3)
- moved U1 12.7 mm to (132.1, 61.0)
- moved U10 12.7 mm to (129.5, 73.7)
- moved C6 11.5 mm to (158.8, 78.7)
- moved U8 11.4 mm to (163.8, 86.4)
- moved R1 10.2 mm to (241.3, 73.7), turned to 0 degrees
- moved RN2 7.62 mm to (167.6, 73.7)
- moved U13 2.54 mm to (104.1, 73.7)
- moved U7 1.27 mm to (212.1, 86.4)
- moved C16 1.27 mm to (100.3, 71.0)
- moved C13 0.08 mm to (53.3, 96.4)
- moved C4 0.08 mm to (198.1, 118.1)
- moved U2 0.08 mm to (170.2, 125.7)
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Connections:
- J4 pad 1: GND -> VCC
- J4 pad 3: VCC -> GND
- U13 pad 1: /~{COUNT} -> /~{OUT}
- U13 pad 11: /~{EITHER_OUT} -> unconnected-(U13-Pad11)
- U13 pad 12: /~{OUT} -> VCC
- U13 pad 13: /~{OUT_AND_COUNT} -> VCC
- U13 pad 3: /~{EITHER_COUNT} -> /~{EITHER_OUT}
- U13 pad 4: VCC -> /~{COUNT}
- U13 pad 5: VCC -> /~{OUT_AND_COUNT}
- U13 pad 6: unconnected-(U13-Pad6) -> /~{EITHER_COUNT}
Routing:
- net VCC: track 376.2 -> 666.0 mm, vias 24 -> 9
- net /CTNT_MOD_01: track 34.7 -> 251.0 mm, vias 0 -> 5
- net /CTNT_MOD_02: track 35.9 -> 244.7 mm, vias 0 -> 5
- net /CTNT_MOD_03: track 37.1 -> 239.5 mm, vias 0 -> 5
- net /CTNT_MOD_04: track 38.3 -> 234.5 mm, vias 0 -> 5
- net /CTNT_MOD_05: track 39.6 -> 229.5 mm, vias 0 -> 5
- net /CTNT_MOD_06: track 40.8 -> 224.3 mm, vias 0 -> 5
- net /RESET: track 0.00 -> 182.8 mm, vias 0 -> 2
- net /CTNT_MOD_07: track 42.1 -> 219.3 mm, vias 0 -> 5
- net /CTNT_MOD_00: track 82.6 -> 254.4 mm, vias 0 -> 2
- net /CS_02: track 0.00 -> 157.9 mm
- net /CTNT_MOD_08: track 38.2 -> 195.4 mm, vias 0 -> 5
- net /CS_01: track 0.00 -> 153.1 mm
- net /CTNT_MOD_09: track 39.4 -> 190.3 mm, vias 0 -> 5
- net /CS_0: track 0.00 -> 148.2 mm
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
Commit message: Shift rot pretty much done. Final tidy ups on offset preset counter.
Parts:
- C10, C11, C12: value C_Polarized -> 33uF
- RN1, RN2: value 10K -> VAR
- moved C12 243.8 mm to (195.6, 86.4)
- moved C10 50.0 mm to (76.2, 134.6)
- moved C11 27.4 mm to (106.7, 58.4), turned to -90 degrees
- moved J7 10.2 mm to (243.8, 127.0)
- moved J9 10.2 mm to (243.8, 116.8)
- moved C16 1.27 mm to (99.1, 71.0)
Connections:
- J6 pad 1: /CTNT_MOD_15 -> /CTNT_MOD_00
- J6 pad 10: /CTNT_MOD_06 -> /CTNT_MOD_09
- J6 pad 11: /CTNT_MOD_05 -> /CTNT_MOD_10
- J6 pad 12: /CTNT_MOD_04 -> /CTNT_MOD_11
- J6 pad 13: /CTNT_MOD_03 -> /CTNT_MOD_12
- J6 pad 14: /CTNT_MOD_02 -> /CTNT_MOD_13
- J6 pad 15: /CTNT_MOD_01 -> /CTNT_MOD_14
- J6 pad 16: /CTNT_MOD_00 -> /CTNT_MOD_15
- J6 pad 2: /CTNT_MOD_14 -> /CTNT_MOD_01
- J6 pad 3: /CTNT_MOD_13 -> /CTNT_MOD_02
- J6 pad 4: /CTNT_MOD_12 -> /CTNT_MOD_03
- J6 pad 5: /CTNT_MOD_11 -> /CTNT_MOD_04
- J6 pad 6: /CTNT_MOD_10 -> /CTNT_MOD_05
- J6 pad 7: /CTNT_MOD_09 -> /CTNT_MOD_06
- J6 pad 8: /CTNT_MOD_08 -> /CTNT_MOD_07
- J6 pad 9: /CTNT_MOD_07 -> /CTNT_MOD_08
Routing:
- net VCC: track 666.0 -> 741.9 mm, vias 9 -> 15
- net /~{IN}: track 92.9 -> 164.6 mm, vias 3 -> 6
- net /CTNT_MOD_15: track 159.6 -> 198.0 mm
- net /CTNT_MOD_14: track 164.9 -> 198.3 mm, vias 5 -> 7
- net /CTNT_MOD_13: track 170.0 -> 198.3 mm, vias 5 -> 7
- net /CTNT_MOD_12: track 175.1 -> 198.3 mm, vias 5 -> 7
- net /CTNT_MOD_11: track 180.2 -> 198.3 mm, vias 5 -> 7
- net /CTNT_MOD_10: track 185.3 -> 198.3 mm, vias 5 -> 7
- net /CS_0: track 148.2 -> 160.8 mm
- net /~{RESET}: track 178.8 -> 188.4 mm, vias 4 -> 6
- net /CTNT_MOD_01: track 251.0 -> 242.4 mm, vias 5 -> 7
- net /CTNT_MOD_09: track 190.3 -> 198.3 mm, vias 5 -> 7
- net /CS_02: track 157.9 -> 150.3 mm
- net /CTNT_MOD_04: track 234.5 -> 227.2 mm, vias 5 -> 7
- net /CTNT_MOD_02: track 244.7 -> 237.3 mm, vias 5 -> 7
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Other:
- board text added: "1"
- board text added: "10"
- board text added: "11"
- board text added: "12"
- board text added: "13"
- board text added: "14"
- board text added: "2"
- board text added: "3"
- board text added: "4"
- board text added: "5"
- board text added: "6"
- board text added: "7"
- board text added: "8"
- board text added: "9"
- board text added: "HIGH"
- board text added: "LOW"
- board text added: "OFFSET PRESET COUNTER"
- board text added: "v. 1.0"

Commit message: Tech checks and BOMs complete
Parts:
- moved C11 16.3 mm to (94.0, 68.6)
- moved C12 3.05 mm to (192.5, 86.4), turned to -90 degrees
Connections:
- net /LED_CONTROL renamed /LED_~{OE}
Routing:
- net /BUS_03: track 109.5 -> 105.9 mm
- net /CTNT_MOD_06: track 217.0 -> 213.6 mm
- net /CTNT_MOD_00: track 247.5 -> 244.1 mm
- net /CTNT_MOD_07: track 217.0 -> 213.6 mm
- net /CTNT_MOD_03: track 232.2 -> 228.8 mm
- net /CTNT_MOD_02: track 237.3 -> 233.9 mm
- net /CTNT_MOD_01: track 242.4 -> 239.0 mm
- net /CTNT_MOD_05: track 222.7 -> 219.2 mm
- net /CTNT_MOD_04: track 227.2 -> 223.7 mm
- net /BUS_02: track 109.8 -> 106.7 mm
- net /BUS_01: track 110.1 -> 107.5 mm
- net /BUS_00: track 110.5 -> 108.2 mm
- net Net-(D1-A): track 23.9 -> 25.8 mm
- net VCC: track 741.9 -> 740.1 mm
- net Net-(D3-K): track 13.3 -> 15.1 mm
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Other:
- board text added: "HC574 = Content offset to control clock Short marked pins = Content not offfset"
- board text added: "OFFSET PRESET COUNTER REG"
- board text removed: "OFFSET PRESET COUNTER"

Commit message: Gerbers generated
Other:
- rule pad_to_mask_clearance: 0.051 -> 0
Changed lines of the file:
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@@
       (dielectric_constraints no)
     )
-    (pad_to_mask_clearance 0.051)
-    (solder_mask_min_width 0.25)
+    (pad_to_mask_clearance 0)
     (pcbplotparams
       (layerselection 0x00010fc_ffffffff)
@@
       (drillshape 0)
       (scaleselection 1)
-      (outputdirectory "gerber_v2/")
+      (outputdirectory "gerbers_v1/")
     )
   )
@@
     (fp_circle (center 0 0) (end 1.15 0)
       (stroke (width 0.1) (type solid)) (fill none) (layer "F.Fab"))
-    (pad "1" thru_hole roundrect (at 0 0) (size 2.3 2.3) (drill 1.1) (layers "*.Cu" "*.Mask") (roundrect_rratio 0.108696)
+    (pad "1" thru_hole roundrect (at 0 0) (size 2.3 2.3) (drill 1.1) (layers "*.Cu" "*.Mask") (roundrect_rratio 0.108696087)
       (net 1 "GND") (pinfunction "Pin_1") (pintype "passive"))
     (model "${KICAD6_3DMODEL_DIR}/Connector_Wire.3dshapes/SolderWire-0.5sqmm_1x01_D0.9mm_OD2.3mm.wrl"
@@
     (fp_circle (center 0 0) (end 1.15 0)
       (stroke (width 0.1) (type solid)) (fill none) (layer "F.Fab"))
-    (pad "1" thru_hole roundrect (at 0 0) (size 2.3 2.3) (drill 1.1) (layers "*.Cu" "*.Mask") (roundrect_rratio 0.108696)
+    (pad "1" thru_hole roundrect (at 0 0) (size 2.3 2.3) (drill 1.1) (layers "*.Cu" "*.Mask") (roundrect_rratio 0.108696087)
       (net 2 "VCC") (pinfunction "Pin_1") (pintype "passive"))
     (model "${KICAD6_3DMODEL_DIR}/Connector_Wire.3dshapes/SolderWire-0.5sqmm_1x01_D0.9mm_OD2.3mm.wrl"
@@
     (fp_circle (center 0 0) (end 1.15 0)
       (stroke (width 0.1) (type solid)) (fill none) (layer "F.Fab"))
-    (pad "1" thru_hole roundrect (at 0 0) (size 2.3 2.3) (drill 1.1) (layers "*.Cu" "*.Mask") (roundrect_rratio 0.108696)
+    (pad "1" thru_hole roundrect (at 0 0) (size 2.3 2.3) (drill 1.1) (layers "*.Cu" "*.Mask") (roundrect_rratio 0.108696087)
       (net 2 "VCC") (pinfunction "Pin_1") (pintype "passive"))
     (model "${KICAD6_3DMODEL_DIR}/Connector_Wire.3dshapes/SolderWire-0.5sqmm_1x01_D0.9mm_OD2.3mm.wrl"
@@
     (fp_circle (center 0 0) (end 1.15 0)
       (stroke (width 0.1) (type solid)) (fill none) (layer "F.Fab"))
-    (pad "1" thru_hole roundrect (at 0 0) (size 2.3 2.3) (drill 1.1) (layers "*.Cu" "*.Mask") (roundrect_rratio 0.108696)
+    (pad "1" thru_hole roundrect (at 0 0) (size 2.3 2.3) (drill 1.1) (layers "*.Cu" "*.Mask") (roundrect_rratio 0.108696087)
       (net 1 "GND") (pinfunction "Pin_1") (pintype "passive"))
     (model "${KICAD6_3DMODEL_DIR}/Connector_Wire.3dshapes/SolderWire-0.5sqmm_1x01_D0.9mm_OD2.3mm.wrl"
@@
     (fp_circle (center 0 0) (end 1.15 0)
       (stroke (width 0.1) (type solid)) (fill none) (layer "F.Fab"))
-    (pad "1" thru_hole roundrect (at 0 0) (size 2.3 2.3) (drill 1.1) (layers "*.Cu" "*.Mask") (roundrect_rratio 0.108696)
+    (pad "1" thru_hole roundrect (at 0 0) (size 2.3 2.3) (drill 1.1) (layers "*.Cu" "*.Mask") (roundrect_rratio 0.108696087)
       (net 1 "GND") (pinfunction "Pin_1") (pintype "passive"))
     (model "${KICAD6_3DMODEL_DIR}/Connector_Wire.3dshapes/SolderWire-0.5sqmm_1x01_D0.9mm_OD2.3mm.wrl"
@@
     (fp_circle (center 0 0) (end 1.15 0)
       (stroke (width 0.1) (type solid)) (fill none) (layer "F.Fab"))
-    (pad "1" thru_hole roundrect (at 0 0) (size 2.3 2.3) (drill 1.1) (layers "*.Cu" "*.Mask") (roundrect_rratio 0.108696)
+    (pad "1" thru_hole roundrect (at 0 0) (size 2.3 2.3) (drill 1.1) (layers "*.Cu" "*.Mask") (roundrect_rratio 0.108696087)
       (net 125 "/CS_02") (pinfunction "Pin_1") (pintype "passive"))
     (model "${KICAD6_3DMODEL_DIR}/Connector_Wire.3dshapes/SolderWire-0.5sqmm_1x01_D0.9mm_OD2.3mm.wrl"
@@
     (fp_circle (center 0 0) (end 1.15 0)
       (stroke (width 0.1) (type solid)) (fill none) (layer "F.Fab"))
-    (pad "1" thru_hole roundrect (at 0 0) (size 2.3 2.3) (drill 1.1) (layers "*.Cu" "*.Mask") (roundrect_rratio 0.108696)
+    (pad "1" thru_hole roundrect (at 0 0) (size 2.3 2.3) (drill 1.1) (layers "*.Cu" "*.Mask") (roundrect_rratio 0.108696087)
       (net 2 "VCC") (pinfunction "Pin_1") (pintype "passive"))
     (model "${KICAD6_3DMODEL_DIR}/Connector_Wire.3dshapes/SolderWire-0.5sqmm_1x01_D0.9mm_OD2.3mm.wrl"
@@
     (fp_circle (center 0 0) (end 1.15 0)
       (stroke (width 0.1) (type solid)) (fill none) (layer "F.Fab"))
-    (pad "1" thru_hole roundrect (at 0 0) (size 2.3 2.3) (drill 1.1) (layers "*.Cu" "*.Mask") (roundrect_rratio 0.108696)
+    (pad "1" thru_hole roundrect (at 0 0) (size 2.3 2.3) (drill 1.1) (layers "*.Cu" "*.Mask") (roundrect_rratio 0.108696087)
       (net 124 "/CS_01") (pinfunction "Pin_1") (pintype "passive"))
     (model "${KICAD6_3DMODEL_DIR}/Connector_Wire.3dshapes/SolderWire-0.5sqmm_1x01_D0.9mm_OD2.3mm.wrl"
@@
     (fp_circle (center 0 0) (end 1.15 0)
       (stroke (width 0.1) (type solid)) (fill none) (layer "F.Fab"))
-    (pad "1" thru_hole roundrect (at 0 0) (size 2.3 2.3) (drill 1.1) (layers "*.Cu" "*.Mask") (roundrect_rratio 0.108696)
+    (pad "1" thru_hole roundrect (at 0 0) (size 2.3 2.3) (drill 1.1) (layers "*.Cu" "*.Mask") (roundrect_rratio 0.108696087)
       (net 123 "/CS_0") (pinfunction "Pin_1") (pintype "passive"))
     (model "${KICAD6_3DMODEL_DIR}/Connector_Wire.3dshapes/SolderWire-0.5sqmm_1x01_D0.9mm_OD2.3mm.wrl"
